File: 12x8 Led Array 9mm pitch/12x8 Led Array 9mm pitch.kicad_sch (KiCad schematic)
At the start: 0 parts

Commit message: Generate both schematics: all parts placed with verified pinouts
- 310 parts LED board (96 LED/NTC/R clusters, 6 muxes, 5 IDC)
- 627 parts control board (96 PT4115 channels, 6 PCA9685, 5V rail,
  ESP32 socket, UI buttons/LEDs, fan driver)
- design_data.py is the single source of truth incl. full netlist
- pin numbers cross-validated against KiCad + EasyEDA symbol libraries

Co-Authored-By: Claude Fable 5 <noreply@anthropic.com>
Claude-Session: https://claude.ai/code/session_017oD54uh7Tvu54u9NPQNcZB
Parts:
- added C1, C2, C3, C4, C5, C6: 100nF, Capacitor_SMD:C_0603_1608Metric, symbol Device:C
- added J1: LED ch 1-24, Connector_IDC:IDC-Header_2x25_P2.54mm_Vertical, symbol Connector_Generic:Conn_02x25_Odd_Even
- added J2: LED ch 25-48, Connector_IDC:IDC-Header_2x25_P2.54mm_Vertical, symbol Connector_Generic:Conn_02x25_Odd_Even
- added J3: LED ch 49-72, Connector_IDC:IDC-Header_2x25_P2.54mm_Vertical, symbol Connector_Generic:Conn_02x25_Odd_Even
- added J4: LED ch 73-96, Connector_IDC:IDC-Header_2x25_P2.54mm_Vertical, symbol Connector_Generic:Conn_02x25_Odd_Even
- added J5: logic/analog, Connector_IDC:IDC-Header_2x10_P2.54mm_Vertical, symbol Connector_Generic:Conn_02x10_Odd_Even
- added LED1, LED10, LED11, LED12, LED13, LED14, LED15, LED16, LED17, LED18, LED19, LED2, LED20, LED21, LED22, LED23, LED24, LED25, LED26, LED27, LED28, LED29, LED3, LED30, LED31, LED32, LED33, LED34, LED35, LED36, LED37, LED38, LED39, LED4, LED40, LED41, LED42, LED43, LED44, LED45, LED46, LED47, LED48, LED49, LED5, LED50, LED51, LED52, LED53, LED54, LED55, LED56, LED57, LED58, LED59, LED6, LED60, LED61, LED62, LED63, LED64, LED65, LED66, LED67, LED68, LED69, LED7, LED70, LED71, LED72, LED73, LED74, LED75, LED76, LED77, LED78, LED79, LED8, LED80, LED81, LED82, LED83, LED84, LED85, LED86, LED87, LED88, LED89, LED9, LED90, LED91, LED92, LED93, LED94, LED95, LED96: HL-C3535F15R3GA-ZW 660nm, jlc_parts:LED-SMD_3P-L3.5-W3.5_NLW3535AV2, symbol jlc_parts:HL-C3535F15R3GA-ZW
- added R1, R10, R11, R12, R13, R14, R15, R16, R17, R18, R19, R2, R20, R21, R22, R23, R24, R25, R26, R27, R28, R29, R3, R30, R31, R32, R33, R34, R35, R36, R37, R38, R39, R4, R40, R41, R42, R43, R44, R45, R46, R47, R48, R49, R5, R50, R51, R52, R53, R54, R55, R56, R57, R58, R59, R6, R60, R61, R62, R63, R64, R65, R66, R67, R68, R69, R7, R70, R71, R72, R73, R74, R75, R76, R77, R78, R79, R8, R80, R81, R82, R83, R84, R85, R86, R87, R88, R89, R9, R90, R91, R92, R93, R94, R95, R96: 10k 1%, Resistor_SMD:R_0603_1608Metric, symbol Device:R
- added TH1, TH10, TH11, TH12, TH13, TH14, TH15, TH16, TH17, TH18, TH19, TH2, TH20, TH21, TH22, TH23, TH24, TH25, TH26, TH27, TH28, TH29, TH3, TH30, TH31, TH32, TH33, TH34, TH35, TH36, TH37, TH38, TH39, TH4, TH40, TH41, TH42, TH43, TH44, TH45, TH46, TH47, TH48, TH49, TH5, TH50, TH51, TH52, TH53, TH54, TH55, TH56, TH57, TH58, TH59, TH6, TH60, TH61, TH62, TH63, TH64, TH65, TH66, TH67, TH68, TH69, TH7, TH70, TH71, TH72, TH73, TH74, TH75, TH76, TH77, TH78, TH79, TH8, TH80, TH81, TH82, TH83, TH84, TH85, TH86, TH87, TH88, TH89, TH9, TH90, TH91, TH92, TH93, TH94, TH95, TH96: NTC 10k B3434, Resistor_SMD:R_0603_1608Metric, symbol Device:Thermistor_NTC
- added U1, U2, U3, U4, U5, U6: CD74HC4067M96, jlc_parts:SOIC-24_L15.4-W7.5-P1.27-LS10.3-BL, symbol jlc_parts:CD74HC4067M96
Other:
- note added: "CH1"
- note added: "CH10"
- note added: "CH11"
- note added: "CH12"
- note added: "CH13"
- note added: "CH14"
- note added: "CH15"
- note added: "CH16"
- note added: "CH17"
- note added: "CH18"
- note added: "CH19"
- note added: "CH2"
- note added: "CH20"
- note added: "CH21"
- note added: "CH22"
- note added: "CH23"
- note added: "CH24"
- note added: "CH25"
- note added: "CH26"
- note added: "CH27"
- note added: "CH28"
- note added: "CH29"
- note added: "CH3"
- note added: "CH30"
- note added: "CH31"
- note added: "CH32"
- note added: "CH33"
- note added: "CH34"
- note added: "CH35"
- note added: "CH36"
- note added: "CH37"
- note added: "CH38"
- note added: "CH39"
- note added: "CH4"
- note added: "CH40"
- note added: "CH41"
- note added: "CH42"
- note added: "CH43"
- note added: "CH44"
- note added: "CH45"
- note added: "CH46"
- note added: "CH47"
- note added: "CH48"
- note added: "CH49"
- note added: "CH5"
- note added: "CH50"
- note added: "CH51"
- note added: "CH52"
- note added: "CH53"
- note added: "CH54"
- note added: "CH55"
- note added: "CH56"
- note added: "CH57"
- note added: "CH58"
- note added: "CH59"
- note added: "CH6"
- note added: "CH60"
- note added: "CH61"
- note added: "CH62"
- note added: "CH63"
- note added: "CH64"
- note added: "CH65"
- note added: "CH66"
- note added: "CH67"
- note added: "CH68"
- note added: "CH69"
- note added: "CH7"
- note added: "CH70"
- note added: "CH71"
- note added: "CH72"
- note added: "CH73"
- note added: "CH74"
- note added: "CH75"
- note added: "CH76"
- note added: "CH77"
- note added: "CH78"
- note added: "CH79"
- note added: "CH8"
- note added: "CH80"
- note added: "CH81"
- note added: "CH82"
- note added: "CH83"
- note added: "CH84"
- note added: "CH85"
- note added: "CH86"
- note added: "CH87"
- note added: "CH88"
- note added: "CH89"
- note added: "CH9"
- note added: "CH90"
- note added: "CH91"
- note added: "CH92"
- note added: "CH93"
- note added: "CH94"
- note added: "CH95"
- note added: "CH96"
- note added: "NTC MUXES (U1..U6 = channels 1-16 / 17-32 / 33-48 / 49-64 / 65-80 / 81-96)"
- note added: "RIBBONS TO CONTROL BOARD"
- note added: "Wire per CONNECTIONS.md - LED pin1=A(+), pin2=K(-), pin3=thermal: tie to pin2"
- title: (none) -> 12x8 660nm LED Array - LED Board

Commit message: Hierarchical schematics: fully wired, netlist-verified, ERC clean
- Root + well.kicad_sch / channel.kicad_sch instantiated 96x each;
  refs preserved (LED1-96, U1-96...) via instance paths
- Sub-sheets pre-wired; root connected via net labels; no_connects
  on unused ESP32 socket pins; PWR_FLAGs per rail
- verify_netlist.py: KiCad netlist export matches design_data on all
  300 (LED) + 412 (control) intended nets; ERC clean / 3 benign warns
- LCSC corrections from verification agent applied (C125847, C134514,
  C286136, C134820, C36414); datasheets for all parts in reference/
- jlc_parts pins normalized to passive

Co-Authored-By: Claude Fable 5 <noreply@anthropic.com>
Claude-Session: https://claude.ai/code/session_017oD54uh7Tvu54u9NPQNcZB
Parts:
- removed LED1, LED10, LED11, LED12, LED13, LED14, LED15, LED16, LED17, LED18, LED19, LED2, LED20, LED21, LED22, LED23, LED24, LED25, LED26, LED27, LED28, LED29, LED3, LED30, LED31, LED32, LED33, LED34, LED35, LED36, LED37, LED38, LED39, LED4, LED40, LED41, LED42, LED43, LED44, LED45, LED46, LED47, LED48, LED49, LED5, LED50, LED51, LED52, LED53, LED54, LED55, LED56, LED57, LED58, LED59, LED6, LED60, LED61, LED62, LED63, LED64, LED65, LED66, LED67, LED68, LED69, LED7, LED70, LED71, LED72, LED73, LED74, LED75, LED76, LED77, LED78, LED79, LED8, LED80, LED81, LED82, LED83, LED84, LED85, LED86, LED87, LED88, LED89, LED9, LED90, LED91, LED92, LED93, LED94, LED95, LED96: HL-C3535F15R3GA-ZW 660nm, jlc_parts:LED-SMD_3P-L3.5-W3.5_NLW3535AV2, symbol jlc_parts:HL-C3535F15R3GA-ZW
- removed R1, R10, R11, R12, R13, R14, R15, R16, R17, R18, R19, R2, R20, R21, R22, R23, R24, R25, R26, R27, R28, R29, R3, R30, R31, R32, R33, R34, R35, R36, R37, R38, R39, R4, R40, R41, R42, R43, R44, R45, R46, R47, R48, R49, R5, R50, R51, R52, R53, R54, R55, R56, R57, R58, R59, R6, R60, R61, R62, R63, R64, R65, R66, R67, R68, R69, R7, R70, R71, R72, R73, R74, R75, R76, R77, R78, R79, R8, R80, R81, R82, R83, R84, R85, R86, R87, R88, R89, R9, R90, R91, R92, R93, R94, R95, R96: 10k 1%, Resistor_SMD:R_0603_1608Metric, symbol Device:R
- removed TH1, TH10, TH11, TH12, TH13, TH14, TH15, TH16, TH17, TH18, TH19, TH2, TH20, TH21, TH22, TH23, TH24, TH25, TH26, TH27, TH28, TH29, TH3, TH30, TH31, TH32, TH33, TH34, TH35, TH36, TH37, TH38, TH39, TH4, TH40, TH41, TH42, TH43, TH44, TH45, TH46, TH47, TH48, TH49, TH5, TH50, TH51, TH52, TH53, TH54, TH55, TH56, TH57, TH58, TH59, TH6, TH60, TH61, TH62, TH63, TH64, TH65, TH66, TH67, TH68, TH69, TH7, TH70, TH71, TH72, TH73, TH74, TH75, TH76, TH77, TH78, TH79, TH8, TH80, TH81, TH82, TH83, TH84, TH85, TH86, TH87, TH88, TH89, TH9, TH90, TH91, TH92, TH93, TH94, TH95, TH96: NTC 10k B3434, Resistor_SMD:R_0603_1608Metric, symbol Device:Thermistor_NTC
- J5: footprint Connector_IDC:IDC-Header_2x10_P2.54mm_Vertical -> Connector_IDC:IDC-Header_2x10_P2.54mm_Horizontal
Connections:
- net NTC_SIG4: now reaches U4.1 (COMMONINPUT/OUTPUT)
- net NTC_SIG4: now also J5.9 (Pin_9)
- net MUX_A0: now reaches U4.10 (S0)
- net MUX_A0: now also J5.15 (Pin_15), U1.10 (S0), U2.10 (S0), U3.10 (S0), U5.10 (S0), U6.10 (S0)
- net MUX_A1: now reaches U4.11 (S1)
- net MUX_A1: now also J5.16 (Pin_16), U1.11 (S1), U2.11 (S1), U3.11 (S1), U5.11 (S1), U6.11 (S1)
- net GND: now reaches U4.12 (GND)
- net GND: now also C1.2, C2.2, C3.2, C4.2, C5.2, C6.2, J1.49 (Pin_49), J1.50 (Pin_50), J2.49 (Pin_49), J2.50 (Pin_50), J3.49 (Pin_49), J3.50 (Pin_50), J4.49 (Pin_49), J4.50 (Pin_50), J5.10 (Pin_10), J5.12 (Pin_12), J5.14 (Pin_14), J5.19 (Pin_19), J5.2 (Pin_2), J5.20 (Pin_20), J5.4 (Pin_4), J5.6 (Pin_6), J5.8 (Pin_8), U1.12 (GND), U1.15 (~{E}), U2.12 (GND), U2.15 (~{E}), U3.12 (GND), U3.15 (~{E}), U4.15 (~{E}), U5.12 (GND), U5.15 (~{E}), U6.12 (GND), U6.15 (~{E})
- net MUX_A3: now reaches U4.13 (S3)
- net MUX_A3: now also J5.18 (Pin_18), U1.13 (S3), U2.13 (S3), U3.13 (S3), U5.13 (S3), U6.13 (S3)
- net MUX_A2: now reaches U4.14 (S2)
- net MUX_A2: now also J5.17 (Pin_17), U1.14 (S2), U2.14 (S2), U3.14 (S2), U5.14 (S2), U6.14 (S2)
- net NTC64: now reaches U4.16 (I15)
- net NTC63: now reaches U4.17 (I14)
- net NTC62: now reaches U4.18 (I13)
- net NTC61: now reaches U4.19 (I12)
- net NTC56: now reaches U4.2 (I7)
- net NTC60: now reaches U4.20 (I11)
- net NTC59: now reaches U4.21 (I10)
- net NTC58: now reaches U4.22 (I9)
- net NTC57: now reaches U4.23 (I8)
- net +3V3: now reaches U4.24 (VCC)
- net +3V3: now also C1.1, C2.1, C3.1, C4.1, C5.1, C6.1, J5.1 (Pin_1), U1.24 (VCC), U2.24 (VCC), U3.24 (VCC), U5.24 (VCC), U6.24 (VCC)
- net NTC55: now reaches U4.3 (I6)
- net NTC54: now reaches U4.4 (I5)
- net NTC53: now reaches U4.5 (I4)
- net NTC52: now reaches U4.6 (I3)
- net NTC51: now reaches U4.7 (I2)
- net NTC50: now reaches U4.8 (I1)
- net NTC49: now reaches U4.9 (I0)
- net NTC_SIG5: now reaches U5.1 (COMMONINPUT/OUTPUT)
- net NTC_SIG5: now also J5.11 (Pin_11)
- net NTC80: now reaches U5.16 (I15)
- net NTC79: now reaches U5.17 (I14)
- net NTC78: now reaches U5.18 (I13)
- net NTC77: now reaches U5.19 (I12)
- net NTC72: now reaches U5.2 (I7)
- net NTC76: now reaches U5.20 (I11)
- net NTC75: now reaches U5.21 (I10)
- net NTC74: now reaches U5.22 (I9)
- net NTC73: now reaches U5.23 (I8)
- net NTC71: now reaches U5.3 (I6)
- net NTC70: now reaches U5.4 (I5)
- net NTC69: now reaches U5.5 (I4)
- net NTC68: now reaches U5.6 (I3)
- net NTC67: now reaches U5.7 (I2)
- net NTC66: now reaches U5.8 (I1)
- net NTC65: now reaches U5.9 (I0)
- net LED_A25: now reaches J2.1 (Pin_1)
- net LED_K29: now reaches J2.10 (Pin_10)
- net LED_A30: now reaches J2.11 (Pin_11)
- net LED_K30: now reaches J2.12 (Pin_12)
- net LED_A31: now reaches J2.13 (Pin_13)
- net LED_K31: now reaches J2.14 (Pin_14)
- net LED_A32: now reaches J2.15 (Pin_15)
- net LED_K32: now reaches J2.16 (Pin_16)
- net LED_A33: now reaches J2.17 (Pin_17)
- net LED_K33: now reaches J2.18 (Pin_18)
- net LED_A34: now reaches J2.19 (Pin_19)
- net LED_K25: now reaches J2.2 (Pin_2)
- net LED_K34: now reaches J2.20 (Pin_20)
- net LED_A35: now reaches J2.21 (Pin_21)
- net LED_K35: now reaches J2.22 (Pin_22)
- net LED_A36: now reaches J2.23 (Pin_23)
- net LED_K36: now reaches J2.24 (Pin_24)
- net LED_A37: now reaches J2.25 (Pin_25)
- net LED_K37: now reaches J2.26 (Pin_26)
- net LED_A38: now reaches J2.27 (Pin_27)
- net LED_K38: now reaches J2.28 (Pin_28)
- net LED_A39: now reaches J2.29 (Pin_29)
- net LED_A26: now reaches J2.3 (Pin_3)
- net LED_K39: now reaches J2.30 (Pin_30)
- net LED_A40: now reaches J2.31 (Pin_31)
- net LED_K40: now reaches J2.32 (Pin_32)
- net LED_A41: now reaches J2.33 (Pin_33)
- net LED_K41: now reaches J2.34 (Pin_34)
- net LED_A42: now reaches J2.35 (Pin_35)
- net LED_K42: now reaches J2.36 (Pin_36)
- net LED_A43: now reaches J2.37 (Pin_37)
- net LED_K43: now reaches J2.38 (Pin_38)
- net LED_A44: now reaches J2.39 (Pin_39)
- net LED_K26: now reaches J2.4 (Pin_4)
- net LED_K44: now reaches J2.40 (Pin_40)
- net LED_A45: now reaches J2.41 (Pin_41)
- net LED_K45: now reaches J2.42 (Pin_42)
- net LED_A46: now reaches J2.43 (Pin_43)
- net LED_K46: now reaches J2.44 (Pin_44)
- net LED_A47: now reaches J2.45 (Pin_45)
- net LED_K47: now reaches J2.46 (Pin_46)
- net LED_A48: now reaches J2.47 (Pin_47)
- net LED_K48: now reaches J2.48 (Pin_48)
- net LED_A27: now reaches J2.5 (Pin_5)
- net LED_K27: now reaches J2.6 (Pin_6)
- net LED_A28: now reaches J2.7 (Pin_7)
- net LED_K28: now reaches J2.8 (Pin_8)
- net LED_A29: now reaches J2.9 (Pin_9)
- net NTC_SIG1: now reaches U1.1 (COMMONINPUT/OUTPUT)
- net NTC_SIG1: now also J5.3 (Pin_3)
- net NTC16: now reaches U1.16 (I15)
- net NTC15: now reaches U1.17 (I14)
- net NTC14: now reaches U1.18 (I13)
- net NTC13: now reaches U1.19 (I12)
- net NTC8: now reaches U1.2 (I7)
- net NTC12: now reaches U1.20 (I11)
- net NTC11: now reaches U1.21 (I10)
- net NTC10: now reaches U1.22 (I9)
- net NTC9: now reaches U1.23 (I8)
- net NTC7: now reaches U1.3 (I6)
- net NTC6: now reaches U1.4 (I5)
- net NTC5: now reaches U1.5 (I4)
- net NTC4: now reaches U1.6 (I3)
- net NTC3: now reaches U1.7 (I2)
- net NTC2: now reaches U1.8 (I1)
- net NTC1: now reaches U1.9 (I0)
- net LED_A73: now reaches J4.1 (Pin_1)
- net LED_K77: now reaches J4.10 (Pin_10)
- net LED_A78: now reaches J4.11 (Pin_11)
- net LED_K78: now reaches J4.12 (Pin_12)
- net LED_A79: now reaches J4.13 (Pin_13)
- net LED_K79: now reaches J4.14 (Pin_14)
- net LED_A80: now reaches J4.15 (Pin_15)
- net LED_K80: now reaches J4.16 (Pin_16)
- net LED_A81: now reaches J4.17 (Pin_17)
- net LED_K81: now reaches J4.18 (Pin_18)
- net LED_A82: now reaches J4.19 (Pin_19)
- net LED_K73: now reaches J4.2 (Pin_2)
- net LED_K82: now reaches J4.20 (Pin_20)
- net LED_A83: now reaches J4.21 (Pin_21)
- net LED_K83: now reaches J4.22 (Pin_22)
- net LED_A84: now reaches J4.23 (Pin_23)
- net LED_K84: now reaches J4.24 (Pin_24)
- net LED_A85: now reaches J4.25 (Pin_25)
- net LED_K85: now reaches J4.26 (Pin_26)
- net LED_A86: now reaches J4.27 (Pin_27)
- net LED_K86: now reaches J4.28 (Pin_28)
- net LED_A87: now reaches J4.29 (Pin_29)
- net LED_A74: now reaches J4.3 (Pin_3)
- net LED_K87: now reaches J4.30 (Pin_30)
- net LED_A88: now reaches J4.31 (Pin_31)
- net LED_K88: now reaches J4.32 (Pin_32)
- net LED_A89: now reaches J4.33 (Pin_33)
- net LED_K89: now reaches J4.34 (Pin_34)
- net LED_A90: now reaches J4.35 (Pin_35)
- net LED_K90: now reaches J4.36 (Pin_36)
- net LED_A91: now reaches J4.37 (Pin_37)
- net LED_K91: now reaches J4.38 (Pin_38)
- net LED_A92: now reaches J4.39 (Pin_39)
- net LED_K74: now reaches J4.4 (Pin_4)
- net LED_K92: now reaches J4.40 (Pin_40)
- net LED_A93: now reaches J4.41 (Pin_41)
- net LED_K93: now reaches J4.42 (Pin_42)
- net LED_A94: now reaches J4.43 (Pin_43)
- net LED_K94: now reaches J4.44 (Pin_44)
- net LED_A95: now reaches J4.45 (Pin_45)
- net LED_K95: now reaches J4.46 (Pin_46)
- net LED_A96: now reaches J4.47 (Pin_47)
- net LED_K96: now reaches J4.48 (Pin_48)
- net LED_A75: now reaches J4.5 (Pin_5)
- net LED_K75: now reaches J4.6 (Pin_6)
- net LED_A76: now reaches J4.7 (Pin_7)
- net LED_K76: now reaches J4.8 (Pin_8)
- net LED_A77: now reaches J4.9 (Pin_9)
- net NTC_SIG3: now reaches U3.1 (COMMONINPUT/OUTPUT)
- net NTC_SIG3: now also J5.7 (Pin_7)
- net NTC48: now reaches U3.16 (I15)
- net NTC47: now reaches U3.17 (I14)
- net NTC46: now reaches U3.18 (I13)
- net NTC45: now reaches U3.19 (I12)
- net NTC40: now reaches U3.2 (I7)
- net NTC44: now reaches U3.20 (I11)
- net NTC43: now reaches U3.21 (I10)
- net NTC42: now reaches U3.22 (I9)
- net NTC41: now reaches U3.23 (I8)
- net NTC39: now reaches U3.3 (I6)
- net NTC38: now reaches U3.4 (I5)
- net NTC37: now reaches U3.5 (I4)
- net NTC36: now reaches U3.6 (I3)
- net NTC35: now reaches U3.7 (I2)
- net NTC34: now reaches U3.8 (I1)
- net NTC33: now reaches U3.9 (I0)
- net NTC_SIG2: now reaches U2.1 (COMMONINPUT/OUTPUT)
- net NTC_SIG2: now also J5.5 (Pin_5)
- net NTC32: now reaches U2.16 (I15)
- net NTC31: now reaches U2.17 (I14)
- net NTC30: now reaches U2.18 (I13)
- net NTC29: now reaches U2.19 (I12)
- net NTC24: now reaches U2.2 (I7)
- net NTC28: now reaches U2.20 (I11)
- net NTC27: now reaches U2.21 (I10)
- net NTC26: now reaches U2.22 (I9)
- net NTC25: now reaches U2.23 (I8)
- net NTC23: now reaches U2.3 (I6)
- net NTC22: now reaches U2.4 (I5)
- net NTC21: now reaches U2.5 (I4)
- net NTC20: now reaches U2.6 (I3)
- net NTC19: now reaches U2.7 (I2)
- net NTC18: now reaches U2.8 (I1)
- net NTC17: now reaches U2.9 (I0)
- net LED_A1: now reaches J1.1 (Pin_1)
- net LED_K5: now reaches J1.10 (Pin_10)
- net LED_A6: now reaches J1.11 (Pin_11)
- net LED_K6: now reaches J1.12 (Pin_12)
- net LED_A7: now reaches J1.13 (Pin_13)
- net LED_K7: now reaches J1.14 (Pin_14)
- net LED_A8: now reaches J1.15 (Pin_15)
- net LED_K8: now reaches J1.16 (Pin_16)
- net LED_A9: now reaches J1.17 (Pin_17)
- net LED_K9: now reaches J1.18 (Pin_18)
- net LED_A10: now reaches J1.19 (Pin_19)
- net LED_K1: now reaches J1.2 (Pin_2)
- net LED_K10: now reaches J1.20 (Pin_20)
- net LED_A11: now reaches J1.21 (Pin_21)
- net LED_K11: now reaches J1.22 (Pin_22)
- net LED_A12: now reaches J1.23 (Pin_23)
- net LED_K12: now reaches J1.24 (Pin_24)
- net LED_A13: now reaches J1.25 (Pin_25)
- net LED_K13: now reaches J1.26 (Pin_26)
- net LED_A14: now reaches J1.27 (Pin_27)
- net LED_K14: now reaches J1.28 (Pin_28)
- net LED_A15: now reaches J1.29 (Pin_29)
- net LED_A2: now reaches J1.3 (Pin_3)
- net LED_K15: now reaches J1.30 (Pin_30)
- net LED_A16: now reaches J1.31 (Pin_31)
- net LED_K16: now reaches J1.32 (Pin_32)
- net LED_A17: now reaches J1.33 (Pin_33)
- net LED_K17: now reaches J1.34 (Pin_34)
- net LED_A18: now reaches J1.35 (Pin_35)
- net LED_K18: now reaches J1.36 (Pin_36)
- net LED_A19: now reaches J1.37 (Pin_37)
- net LED_K19: now reaches J1.38 (Pin_38)
- net LED_A20: now reaches J1.39 (Pin_39)
- net LED_K2: now reaches J1.4 (Pin_4)
- net LED_K20: now reaches J1.40 (Pin_40)
- net LED_A21: now reaches J1.41 (Pin_41)
- net LED_K21: now reaches J1.42 (Pin_42)
- net LED_A22: now reaches J1.43 (Pin_43)
- net LED_K22: now reaches J1.44 (Pin_44)
- net LED_A23: now reaches J1.45 (Pin_45)
- net LED_K23: now reaches J1.46 (Pin_46)
- net LED_A24: now reaches J1.47 (Pin_47)
- net LED_K24: now reaches J1.48 (Pin_48)
- net LED_A3: now reaches J1.5 (Pin_5)
- net LED_K3: now reaches J1.6 (Pin_6)
- net LED_A4: now reaches J1.7 (Pin_7)
- net LED_K4: now reaches J1.8 (Pin_8)
- net LED_A5: now reaches J1.9 (Pin_9)
- net NTC_SIG6: now reaches U6.1 (COMMONINPUT/OUTPUT)
- net NTC_SIG6: now also J5.13 (Pin_13)
- net NTC96: now reaches U6.16 (I15)
- net NTC95: now reaches U6.17 (I14)
- net NTC94: now reaches U6.18 (I13)
- net NTC93: now reaches U6.19 (I12)
- net NTC88: now reaches U6.2 (I7)
- net NTC92: now reaches U6.20 (I11)
- net NTC91: now reaches U6.21 (I10)
- net NTC90: now reaches U6.22 (I9)
- net NTC89: now reaches U6.23 (I8)
- net NTC87: now reaches U6.3 (I6)
- net NTC86: now reaches U6.4 (I5)
- net NTC85: now reaches U6.5 (I4)
- net NTC84: now reaches U6.6 (I3)
- net NTC83: now reaches U6.7 (I2)
- net NTC82: now reaches U6.8 (I1)
- net NTC81: now reaches U6.9 (I0)
- net LED_A49: now reaches J3.1 (Pin_1)
- net LED_K53: now reaches J3.10 (Pin_10)
- net LED_A54: now reaches J3.11 (Pin_11)
- net LED_K54: now reaches J3.12 (Pin_12)
- net LED_A55: now reaches J3.13 (Pin_13)
- net LED_K55: now reaches J3.14 (Pin_14)
- net LED_A56: now reaches J3.15 (Pin_15)
- net LED_K56: now reaches J3.16 (Pin_16)
- net LED_A57: now reaches J3.17 (Pin_17)
- net LED_K57: now reaches J3.18 (Pin_18)
- net LED_A58: now reaches J3.19 (Pin_19)
- net LED_K49: now reaches J3.2 (Pin_2)
- net LED_K58: now reaches J3.20 (Pin_20)
- net LED_A59: now reaches J3.21 (Pin_21)
- net LED_K59: now reaches J3.22 (Pin_22)
- net LED_A60: now reaches J3.23 (Pin_23)
- net LED_K60: now reaches J3.24 (Pin_24)
- net LED_A61: now reaches J3.25 (Pin_25)
- net LED_K61: now reaches J3.26 (Pin_26)
- net LED_A62: now reaches J3.27 (Pin_27)
- net LED_K62: now reaches J3.28 (Pin_28)
- net LED_A63: now reaches J3.29 (Pin_29)
- net LED_A50: now reaches J3.3 (Pin_3)
- net LED_K63: now reaches J3.30 (Pin_30)
- net LED_A64: now reaches J3.31 (Pin_31)
- net LED_K64: now reaches J3.32 (Pin_32)
- net LED_A65: now reaches J3.33 (Pin_33)
- net LED_K65: now reaches J3.34 (Pin_34)
- net LED_A66: now reaches J3.35 (Pin_35)
- net LED_K66: now reaches J3.36 (Pin_36)
- net LED_A67: now reaches J3.37 (Pin_37)
- net LED_K67: now reaches J3.38 (Pin_38)
- net LED_A68: now reaches J3.39 (Pin_39)
- net LED_K50: now reaches J3.4 (Pin_4)
- net LED_K68: now reaches J3.40 (Pin_40)
- net LED_A69: now reaches J3.41 (Pin_41)
- net LED_K69: now reaches J3.42 (Pin_42)
- net LED_A70: now reaches J3.43 (Pin_43)
- net LED_K70: now reaches J3.44 (Pin_44)
- net LED_A71: now reaches J3.45 (Pin_45)
- net LED_K71: now reaches J3.46 (Pin_46)
- net LED_A72: now reaches J3.47 (Pin_47)
- net LED_K72: now reaches J3.48 (Pin_48)
- net LED_A51: now reaches J3.5 (Pin_5)
- net LED_K51: now reaches J3.6 (Pin_6)
- net LED_A52: now reaches J3.7 (Pin_7)
- net LED_K52: now reaches J3.8 (Pin_8)
- net LED_A53: now reaches J3.9 (Pin_9)
Other:
- added sheet CH01 (well.kicad_sch)
- added sheet CH02 (well.kicad_sch)
- added sheet CH03 (well.kicad_sch)
- added sheet CH04 (well.kicad_sch)
- added sheet CH05 (well.kicad_sch)
- added sheet CH06 (well.kicad_sch)
- added sheet CH07 (well.kicad_sch)
- added sheet CH08 (well.kicad_sch)
- added sheet CH09 (well.kicad_sch)
- added sheet CH10 (well.kicad_sch)
- added sheet CH11 (well.kicad_sch)
- added sheet CH12 (well.kicad_sch)
- added sheet CH13 (well.kicad_sch)
- added sheet CH14 (well.kicad_sch)
- added sheet CH15 (well.kicad_sch)
- added sheet CH16 (well.kicad_sch)
- added sheet CH17 (well.kicad_sch)
- added sheet CH18 (well.kicad_sch)
- added sheet CH19 (well.kicad_sch)
- added sheet CH20 (well.kicad_sch)
- added sheet CH21 (well.kicad_sch)
- added sheet CH22 (well.kicad_sch)
- added sheet CH23 (well.kicad_sch)
- added sheet CH24 (well.kicad_sch)
- added sheet CH25 (well.kicad_sch)
- added sheet CH26 (well.kicad_sch)
- added sheet CH27 (well.kicad_sch)
- added sheet CH28 (well.kicad_sch)
- added sheet CH29 (well.kicad_sch)
- added sheet CH30 (well.kicad_sch)
- added sheet CH31 (well.kicad_sch)
- added sheet CH32 (well.kicad_sch)
- added sheet CH33 (well.kicad_sch)
- added sheet CH34 (well.kicad_sch)
- added sheet CH35 (well.kicad_sch)
- added sheet CH36 (well.kicad_sch)
- added sheet CH37 (well.kicad_sch)
- added sheet CH38 (well.kicad_sch)
- added sheet CH39 (well.kicad_sch)
- added sheet CH40 (well.kicad_sch)
- added sheet CH41 (well.kicad_sch)
- added sheet CH42 (well.kicad_sch)
- added sheet CH43 (well.kicad_sch)
- added sheet CH44 (well.kicad_sch)
- added sheet CH45 (well.kicad_sch)
- added sheet CH46 (well.kicad_sch)
- added sheet CH47 (well.kicad_sch)
- added sheet CH48 (well.kicad_sch)
- added sheet CH49 (well.kicad_sch)
- added sheet CH50 (well.kicad_sch)
- added sheet CH51 (well.kicad_sch)
- added sheet CH52 (well.kicad_sch)
- added sheet CH53 (well.kicad_sch)
- added sheet CH54 (well.kicad_sch)
- added sheet CH55 (well.kicad_sch)
- added sheet CH56 (well.kicad_sch)
- added sheet CH57 (well.kicad_sch)
- added sheet CH58 (well.kicad_sch)
- added sheet CH59 (well.kicad_sch)
- added sheet CH60 (well.kicad_sch)
- added sheet CH61 (well.kicad_sch)
- added sheet CH62 (well.kicad_sch)
- added sheet CH63 (well.kicad_sch)
- added sheet CH64 (well.kicad_sch)
- added sheet CH65 (well.kicad_sch)
- added sheet CH66 (well.kicad_sch)
- added sheet CH67 (well.kicad_sch)
- added sheet CH68 (well.kicad_sch)
- added sheet CH69 (well.kicad_sch)
- added sheet CH70 (well.kicad_sch)
- added sheet CH71 (well.kicad_sch)
- added sheet CH72 (well.kicad_sch)
- added sheet CH73 (well.kicad_sch)
- added sheet CH74 (well.kicad_sch)
- added sheet CH75 (well.kicad_sch)
- added sheet CH76 (well.kicad_sch)
- added sheet CH77 (well.kicad_sch)
- added sheet CH78 (well.kicad_sch)
- added sheet CH79 (well.kicad_sch)
- added sheet CH80 (well.kicad_sch)
- added sheet CH81 (well.kicad_sch)
- added sheet CH82 (well.kicad_sch)
- added sheet CH83 (well.kicad_sch)
- added sheet CH84 (well.kicad_sch)
- added sheet CH85 (well.kicad_sch)
- added sheet CH86 (well.kicad_sch)
- added sheet CH87 (well.kicad_sch)
- added sheet CH88 (well.kicad_sch)
- added sheet CH89 (well.kicad_sch)
- added sheet CH90 (well.kicad_sch)
- added sheet CH91 (well.kicad_sch)
- added sheet CH92 (well.kicad_sch)
- added sheet CH93 (well.kicad_sch)
- added sheet CH94 (well.kicad_sch)
- added sheet CH95 (well.kicad_sch)
- added sheet CH96 (well.kicad_sch)
- note added: "96 WELLS (CH01..CH96) - see well.kicad_sch"
- note added: "NTC MUXES U1-U6 (ch 1-16 / 17-32 / 33-48 / 49-64 / 65-80 / 81-96)"
- note removed: "CH1"
- note removed: "CH10"
- note removed: "CH11"
- note removed: "CH12"
- note removed: "CH13"
- note removed: "CH14"
- note removed: "CH15"
- note removed: "CH16"
- note removed: "CH17"
- note removed: "CH18"
- note removed: "CH19"
- note removed: "CH2"
- note removed: "CH20"
- note removed: "CH21"
- note removed: "CH22"
- note removed: "CH23"
- note removed: "CH24"
- note removed: "CH25"
- note removed: "CH26"
- note removed: "CH27"
- note removed: "CH28"
- note removed: "CH29"
- note removed: "CH3"
- note removed: "CH30"
- note removed: "CH31"
- note removed: "CH32"
- note removed: "CH33"
- note removed: "CH34"
- note removed: "CH35"
- note removed: "CH36"
- note removed: "CH37"
- note removed: "CH38"
- note removed: "CH39"
- note removed: "CH4"
- note removed: "CH40"
- note removed: "CH41"
- note removed: "CH42"
- note removed: "CH43"
- note removed: "CH44"
- note removed: "CH45"
- note removed: "CH46"
- note removed: "CH47"
- note removed: "CH48"
- note removed: "CH49"
- note removed: "CH5"
- note removed: "CH50"
- note removed: "CH51"
- note removed: "CH52"
- note removed: "CH53"
- note removed: "CH54"
- note removed: "CH55"
- note removed: "CH56"
- note removed: "CH57"
- note removed: "CH58"
- note removed: "CH59"
- note removed: "CH6"
- note removed: "CH60"
- note removed: "CH61"
- note removed: "CH62"
- note removed: "CH63"
- note removed: "CH64"
- note removed: "CH65"
- note removed: "CH66"
- note removed: "CH67"
- note removed: "CH68"
- note removed: "CH69"
- note removed: "CH7"
- note removed: "CH70"
- note removed: "CH71"
- note removed: "CH72"
- note removed: "CH73"
- note removed: "CH74"
- note removed: "CH75"
- note removed: "CH76"
- note removed: "CH77"
- note removed: "CH78"
- note removed: "CH79"
- note removed: "CH8"
- note removed: "CH80"
- note removed: "CH81"
- note removed: "CH82"
- note removed: "CH83"
- note removed: "CH84"
- note removed: "CH85"
- note removed: "CH86"
- note removed: "CH87"
- note removed: "CH88"
- note removed: "CH89"
- note removed: "CH9"
- note removed: "CH90"
- note removed: "CH91"
- note removed: "CH92"
- note removed: "CH93"
- note removed: "CH94"
- note removed: "CH95"
- note removed: "CH96"
- note removed: "NTC MUXES (U1..U6 = channels 1-16 / 17-32 / 33-48 / 49-64 / 65-80 / 81-96)"
- note removed: "Wire per CONNECTIONS.md - LED pin1=A(+), pin2=K(-), pin3=thermal: tie to pin2"

Commit message: Add test points and mounting holes to schematics
- LED board: TP1-TP3 (+3V3, GND x2); H1-H5 as Mechanical:MountingHole
- Control board: TP1-TP12 (rails, SW_5V, I2C, FAN_SW, CH1 debug set
  DIM1/LED_A1/LED_K1); H1-H4
- 1.5mm bare-pad TestPoint footprints (no BOM cost)
- Netlist re-verified: all nets match; ERC still clean

Co-Authored-By: Claude Fable 5 <noreply@anthropic.com>
Claude-Session: https://claude.ai/code/session_017oD54uh7Tvu54u9NPQNcZB
Parts:
- added H1, H2, H3, H4, H5: M3, MountingHole:MountingHole_3.2mm_M3, symbol Mechanical:MountingHole
- added TP1: +3V3, TestPoint:TestPoint_Pad_1.5x1.5mm, symbol Connector:TestPoint
- added TP2, TP3: GND, TestPoint:TestPoint_Pad_1.5x1.5mm, symbol Connector:TestPoint
Connections:
- net +3V3: now also TP1.1
- net GND: now also TP2.1, TP3.1
