File: 12x8 Led Array 9mm pitch/12x8 Led Array 9mm pitch.kicad_sch (KiCad schematic)
At the start: 25 parts, among them J1 LED ch 1-24, J2 LED ch 25-48, J3 LED ch 49-72, J4 LED ch 73-96, J5 logic/analog, U1 CD74HC4067M96, U2 CD74HC4067M96, U3 CD74HC4067M96, U4 CD74HC4067M96, U5 CD74HC4067M96, U6 CD74HC4067M96

Commit message: Apply user's label cleanup style to control board
- All generated labels now carry explicit justification (left/right
  per rotation, bottom-anchored) matching the hand-cleaned LED board
- gen_schematics_hier.py takes led|ctl|all arg; LED board excluded
  from regeneration by default (hand-edited in KiCad)
- Control board netlist re-verified: all 412 nets match

Co-Authored-By: Claude Fable 5 <noreply@anthropic.com>
Claude-Session: https://claude.ai/code/session_017oD54uh7Tvu54u9NPQNcZB
Connections:
- net +3V3: no longer C1.1, C1.2, C2.1, C2.2, C3.1, C3.2, C4.1, C4.2, C5.1, C5.2, C6.1, C6.2, J1.49 (Pin_49), J1.50 (Pin_50), J2.49 (Pin_49), J2.50 (Pin_50), J3.49 (Pin_49), J3.50 (Pin_50), J4.49 (Pin_49), J4.50 (Pin_50), J5.1 (Pin_1), J5.10 (Pin_10), J5.12 (Pin_12), J5.14 (Pin_14), J5.19 (Pin_19), J5.2 (Pin_2), J5.20 (Pin_20), J5.4 (Pin_4), J5.6 (Pin_6), J5.8 (Pin_8), TP2.1, TP3.1, U1.12 (GND), U1.15 (~{E}), U1.24 (VCC), U2.12 (GND), U2.15 (~{E}), U2.24 (VCC), U3.12 (GND), U3.15 (~{E}), U3.24 (VCC), U4.12 (GND), U4.15 (~{E}), U4.24 (VCC), U5.12 (GND), U5.15 (~{E}), U5.24 (VCC), U6.12 (GND), U6.15 (~{E}), U6.24 (VCC)
- new net +3.3V: C1.1, C1.2, C2.1, C2.2, C3.1, C3.2, C4.1, C4.2, C5.1, C5.2, C6.1, C6.2, J1.49 (Pin_49), J1.50 (Pin_50), J2.49 (Pin_49), J2.50 (Pin_50), J3.49 (Pin_49), J3.50 (Pin_50), J4.49 (Pin_49), J4.50 (Pin_50), J5.1 (Pin_1), J5.10 (Pin_10), J5.12 (Pin_12), J5.14 (Pin_14), J5.19 (Pin_19), J5.2 (Pin_2), J5.20 (Pin_20), J5.4 (Pin_4), J5.6 (Pin_6), J5.8 (Pin_8), TP2.1, TP3.1, U1.12 (GND), U1.15 (~{E}), U1.24 (VCC), U2.12 (GND), U2.15 (~{E}), U2.24 (VCC), U3.12 (GND), U3.15 (~{E}), U3.24 (VCC), U4.12 (GND), U4.15 (~{E}), U4.24 (VCC), U5.12 (GND), U5.15 (~{E}), U5.24 (VCC), U6.12 (GND), U6.15 (~{E}), U6.24 (VCC)
Other:
- moved on the sheet: C1, H1, H2, H3, H4, H5, J2, J3, J4, J5, TP1, TP2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

Commit message: Fix 3.3V/GND bridge, adopt +3.3V naming, power symbols at rail pins
- Removed 6 wire segments that tied each mux VCC run into its
  decoupling cap's GND pin (merged the rails through all six caps)
- Renamed +3V3 -> +3.3V everywhere (user convention), incl. well
  sub-sheet power symbols and docs
- Control board root now uses real power symbols on wire stubs
  instead of text labels for GND/+3.3V/+5V/+24V (user style)
- Verified: netlists match design intent on all 300+412 nets; LED
  board ERC 0 violations; I2C addresses confirmed from netlist
  (PCA9685 0x40-0x45, ADS1115 0x48, no conflicts)

Co-Authored-By: Claude Fable 5 <noreply@anthropic.com>
Claude-Session: https://claude.ai/code/session_017oD54uh7Tvu54u9NPQNcZB
Parts:
- TP1: value +3V3 -> +3.3V
Connections:
- net +3V3 is gone; now on net +3.3V: TP1.1
- net +3.3V: no longer C1.2, C2.2, C3.2, C4.2, C5.2, C6.2, J1.49 (Pin_49), J1.50 (Pin_50), J2.49 (Pin_49), J2.50 (Pin_50), J3.49 (Pin_49), J3.50 (Pin_50), J4.49 (Pin_49), J4.50 (Pin_50), J5.10 (Pin_10), J5.12 (Pin_12), J5.14 (Pin_14), J5.19 (Pin_19), J5.2 (Pin_2), J5.20 (Pin_20), J5.4 (Pin_4), J5.6 (Pin_6), J5.8 (Pin_8), TP2.1, TP3.1, U1.12 (GND), U1.15 (~{E}), U2.12 (GND), U2.15 (~{E}), U3.12 (GND), U3.15 (~{E}), U4.12 (GND), U4.15 (~{E}), U5.12 (GND), U5.15 (~{E}), U6.12 (GND), U6.15 (~{E})
- new net GND: C1.2, C2.2, C3.2, C4.2, C5.2, C6.2, J1.49 (Pin_49), J1.50 (Pin_50), J2.49 (Pin_49), J2.50 (Pin_50), J3.49 (Pin_49), J3.50 (Pin_50), J4.49 (Pin_49), J4.50 (Pin_50), J5.10 (Pin_10), J5.12 (Pin_12), J5.14 (Pin_14), J5.19 (Pin_19), J5.2 (Pin_2), J5.20 (Pin_20), J5.4 (Pin_4), J5.6 (Pin_6), J5.8 (Pin_8), TP2.1, TP3.1, U1.12 (GND), U1.15 (~{E}), U2.12 (GND), U2.15 (~{E}), U3.12 (GND), U3.15 (~{E}), U4.12 (GND), U4.15 (~{E}), U5.12 (GND), U5.15 (~{E}), U6.12 (GND), U6.15 (~{E})
Changed lines of the file:
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@@
 	(wire
 		(pts
-			(xy 342.9 293.37) (xy 355.6 293.37)
-		)
-		(stroke
-			(width 0)
-			(type default)
-		)
-	)
-	(wire
-		(pts
 			(xy 327.66 224.79) (xy 331.47 224.79)
 		)
@@
 	(wire
 		(pts
-			(xy 212.09 347.98) (xy 224.79 347.98)
-		)
-		(stroke
-			(width 0)
-			(type default)
-		)
-	)
-	(wire
-		(pts
 			(xy 43.18 113.03) (xy 46.99 113.03)
 		)
@@
 	(wire
 		(pts
-			(xy 342.9 353.06) (xy 355.6 353.06)
-		)
-		(stroke
-			(width 0)
-			(type default)
-		)
-	)
-	(wire
-		(pts
 			(xy 562.61 140.97) (xy 556.26 140.97)
 		)
@@
 	(wire
 		(pts
-			(xy 87.63 346.71) (xy 100.33 346.71)
-		)
-		(stroke
-			(width 0)
-			(type default)
-		)
-	)
-	(wire
-		(pts
 			(xy 292.1 87.63) (xy 295.91 87.63)
 		)
@@
 	(wire
 		(pts
-			(xy 88.9 293.37) (xy 101.6 293.37)
-		)
-		(stroke
-			(width 0)
-			(type default)
-		)
-	)
-	(wire
-		(pts
 			(xy 288.29 311.15) (xy 292.1 311.15)
 		)
@@
 	(wire
 		(pts
-			(xy 213.36 292.1) (xy 226.06 292.1)
-		)
-		(stroke
-			(width 0)
-			(type default)
-		)
-	)
-	(wire
-		(pts
 			(xy 477.52 48.26) (xy 482.6 48.26)
 		)
@@
 		)
 	)
-	(label "+3V3"
+	(label "+3.3V"
 		(at 431.8 270.51 90)
 		(effects
@@
 			)
 		)
-		(property "Value" "+3V3"
+		(property "Value" "+3.3V"
 			(at 434.34 267.97 0)
 			(show_name no)
@@
 	)
 	(symbol
-		(lib_id "power:+3V3")
+		(lib_id "power:+3.3V")
 		(at 386.08 270.51 0)
 		(unit 1)
@@
 			)
 		)
-		(property "Value" "+3V3"
+		(property "Value" "+3.3V"
 			(at 389.636 273.558 0)
 			(show_name no)

Commit message: Optimize ribbon/mux pin assignments to match user's PCB placement
- Quadrant mapping from actual footprint positions (via pcbnew API):
  J1 left-back = cols1-6/rows1-4, J2 right-back = cols7-12/rows1-4,
  J4 left-front = cols1-6/rows5-8, J3 right-front = cols7-12/rows5-8;
  pin pairs column-major in physical pin-1 direction (nested fan-out,
  no crossings)
- NTC->mux side-matched: U1-U3 serve cols 1-6, U6/U5/U4 cols 7-12
- pin_maps.py generated by optimize_pins.py; design_data now table-driven
- 274 labels renamed in the hand-edited LED sch (proximity-matched,
  0 misses); control board regenerated; CONNECTIONS.md updated
- Both netlists verify (300+412 nets), LED ERC still 0 errors

Co-Authored-By: Claude Fable 5 <noreply@anthropic.com>
Claude-Session: https://claude.ai/code/session_017oD54uh7Tvu54u9NPQNcZB
Connections:
- net LED_A10: now also J2.25 (Pin_25); no longer J1.19 (Pin_19)
- net LED_A11: now also J2.33 (Pin_33); no longer J1.21 (Pin_21)
- net LED_A12: now also J2.41 (Pin_41); no longer J1.23 (Pin_23)
- net LED_A13: now also J1.3 (Pin_3); no longer J1.25 (Pin_25)
- net LED_A14: now also J1.11 (Pin_11); no longer J1.27 (Pin_27)
- net LED_A15: now also J1.19 (Pin_19); no longer J1.29 (Pin_29)
- net LED_A16: now also J1.27 (Pin_27); no longer J1.31 (Pin_31)
- net LED_A17: now also J1.35 (Pin_35); no longer J1.33 (Pin_33)
- net LED_A18: now also J1.43 (Pin_43); no longer J1.35 (Pin_35)
- net LED_A19: now also J2.3 (Pin_3); no longer J1.37 (Pin_37)
- net LED_A2: now also J1.9 (Pin_9); no longer J1.3 (Pin_3)
- net LED_A20: now also J2.11 (Pin_11); no longer J1.39 (Pin_39)
- net LED_A21: now also J2.19 (Pin_19); no longer J1.41 (Pin_41)
- net LED_A22: now also J2.27 (Pin_27); no longer J1.43 (Pin_43)
- net LED_A23: now also J2.35 (Pin_35); no longer J1.45 (Pin_45)
- net LED_A24: now also J2.43 (Pin_43); no longer J1.47 (Pin_47)
- net LED_A25: now also J1.5 (Pin_5); no longer J2.1 (Pin_1)
- net LED_A26: now also J1.13 (Pin_13); no longer J2.3 (Pin_3)
- net LED_A27: now also J1.21 (Pin_21); no longer J2.5 (Pin_5)
- net LED_A28: now also J1.29 (Pin_29); no longer J2.7 (Pin_7)
- net LED_A29: now also J1.37 (Pin_37); no longer J2.9 (Pin_9)
- net LED_A3: now also J1.17 (Pin_17); no longer J1.5 (Pin_5)
- net LED_A30: now also J1.45 (Pin_45); no longer J2.11 (Pin_11)
- net LED_A31: now also J2.5 (Pin_5); no longer J2.13 (Pin_13)
- net LED_A32: now also J2.13 (Pin_13); no longer J2.15 (Pin_15)
- net LED_A33: now also J2.21 (Pin_21); no longer J2.17 (Pin_17)
- net LED_A34: now also J2.29 (Pin_29); no longer J2.19 (Pin_19)
- net LED_A35: now also J2.37 (Pin_37); no longer J2.21 (Pin_21)
- net LED_A36: now also J2.45 (Pin_45); no longer J2.23 (Pin_23)
- net LED_A37: now also J1.7 (Pin_7); no longer J2.25 (Pin_25)
- net LED_A38: now also J1.15 (Pin_15); no longer J2.27 (Pin_27)
- net LED_A39: now also J1.23 (Pin_23); no longer J2.29 (Pin_29)
- net LED_A4: now also J1.25 (Pin_25); no longer J1.7 (Pin_7)
- net LED_A40: now also J1.31 (Pin_31); no longer J2.31 (Pin_31)
- net LED_A41: now also J1.39 (Pin_39); no longer J2.33 (Pin_33)
- net LED_A42: now also J1.47 (Pin_47); no longer J2.35 (Pin_35)
- net LED_A43: now also J2.7 (Pin_7); no longer J2.37 (Pin_37)
- net LED_A44: now also J2.15 (Pin_15); no longer J2.39 (Pin_39)
- net LED_A45: now also J2.23 (Pin_23); no longer J2.41 (Pin_41)
- net LED_A46: now also J2.31 (Pin_31); no longer J2.43 (Pin_43)
- net LED_A47: now also J2.39 (Pin_39); no longer J2.45 (Pin_45)
- net LED_A49: now also J4.1 (Pin_1); no longer J3.1 (Pin_1)
- net LED_A5: now also J1.33 (Pin_33); no longer J1.9 (Pin_9)
- net LED_A50: now also J4.9 (Pin_9); no longer J3.3 (Pin_3)
- net LED_A51: now also J4.17 (Pin_17); no longer J3.5 (Pin_5)
- net LED_A52: now also J4.25 (Pin_25); no longer J3.7 (Pin_7)
- net LED_A53: now also J4.33 (Pin_33); no longer J3.9 (Pin_9)
- net LED_A54: now also J4.41 (Pin_41); no longer J3.11 (Pin_11)
- net LED_A55: now also J3.1 (Pin_1); no longer J3.13 (Pin_13)
- net LED_A56: now also J3.9 (Pin_9); no longer J3.15 (Pin_15)
- net LED_A58: now also J3.25 (Pin_25); no longer J3.19 (Pin_19)
- net LED_A59: now also J3.33 (Pin_33); no longer J3.21 (Pin_21)
- net LED_A6: now also J1.41 (Pin_41); no longer J1.11 (Pin_11)
- net LED_A60: now also J3.41 (Pin_41); no longer J3.23 (Pin_23)
- net LED_A61: now also J4.3 (Pin_3); no longer J3.25 (Pin_25)
- net LED_A62: now also J4.11 (Pin_11); no longer J3.27 (Pin_27)
- net LED_A63: now also J4.19 (Pin_19); no longer J3.29 (Pin_29)
- net LED_A64: now also J4.27 (Pin_27); no longer J3.31 (Pin_31)
- net LED_A65: now also J4.35 (Pin_35); no longer J3.33 (Pin_33)
- net LED_A66: now also J4.43 (Pin_43); no longer J3.35 (Pin_35)
- net LED_A67: now also J3.3 (Pin_3); no longer J3.37 (Pin_37)
- net LED_A68: now also J3.11 (Pin_11); no longer J3.39 (Pin_39)
- net LED_A69: now also J3.19 (Pin_19); no longer J3.41 (Pin_41)
- net LED_A7: now also J2.1 (Pin_1); no longer J1.13 (Pin_13)
- net LED_A70: now also J3.27 (Pin_27); no longer J3.43 (Pin_43)
- net LED_A71: now also J3.35 (Pin_35); no longer J3.45 (Pin_45)
- net LED_A72: now also J3.43 (Pin_43); no longer J3.47 (Pin_47)
- net LED_A73: now also J4.5 (Pin_5); no longer J4.1 (Pin_1)
- net LED_A74: now also J4.13 (Pin_13); no longer J4.3 (Pin_3)
- net LED_A75: now also J4.21 (Pin_21); no longer J4.5 (Pin_5)
- net LED_A76: now also J4.29 (Pin_29); no longer J4.7 (Pin_7)
- net LED_A77: now also J4.37 (Pin_37); no longer J4.9 (Pin_9)
- net LED_A78: now also J4.45 (Pin_45); no longer J4.11 (Pin_11)
- net LED_A79: now also J3.5 (Pin_5); no longer J4.13 (Pin_13)
- net LED_A8: now also J2.9 (Pin_9); no longer J1.15 (Pin_15)
- net LED_A80: now also J3.13 (Pin_13); no longer J4.15 (Pin_15)
- net LED_A81: now also J3.21 (Pin_21); no longer J4.17 (Pin_17)
- net LED_A82: now also J3.29 (Pin_29); no longer J4.19 (Pin_19)
- net LED_A83: now also J3.37 (Pin_37); no longer J4.21 (Pin_21)
- net LED_A84: now also J3.45 (Pin_45); no longer J4.23 (Pin_23)
- net LED_A85: now also J4.7 (Pin_7); no longer J4.25 (Pin_25)
- net LED_A86: now also J4.15 (Pin_15); no longer J4.27 (Pin_27)
- net LED_A87: now also J4.23 (Pin_23); no longer J4.29 (Pin_29)
- net LED_A89: now also J4.39 (Pin_39); no longer J4.33 (Pin_33)
- net LED_A9: now also J2.17 (Pin_17); no longer J1.17 (Pin_17)
- net LED_A90: now also J4.47 (Pin_47); no longer J4.35 (Pin_35)
- net LED_A91: now also J3.7 (Pin_7); no longer J4.37 (Pin_37)
- net LED_A92: now also J3.15 (Pin_15); no longer J4.39 (Pin_39)
- net LED_A93: now also J3.23 (Pin_23); no longer J4.41 (Pin_41)
- net LED_A94: now also J3.31 (Pin_31); no longer J4.43 (Pin_43)
- net LED_A95: now also J3.39 (Pin_39); no longer J4.45 (Pin_45)
- net LED_A96: now also J3.47 (Pin_47); no longer J4.47 (Pin_47)
- net LED_K10: now also J2.26 (Pin_26); no longer J1.20 (Pin_20)
- net LED_K11: now also J2.34 (Pin_34); no longer J1.22 (Pin_22)
- net LED_K12: now also J2.42 (Pin_42); no longer J1.24 (Pin_24)
- net LED_K13: now also J1.4 (Pin_4); no longer J1.26 (Pin_26)
- net LED_K14: now also J1.12 (Pin_12); no longer J1.28 (Pin_28)
- net LED_K15: now also J1.20 (Pin_20); no longer J1.30 (Pin_30)
- net LED_K16: now also J1.28 (Pin_28); no longer J1.32 (Pin_32)
- net LED_K17: now also J1.36 (Pin_36); no longer J1.34 (Pin_34)
- net LED_K18: now also J1.44 (Pin_44); no longer J1.36 (Pin_36)
- net LED_K19: now also J2.4 (Pin_4); no longer J1.38 (Pin_38)
- net LED_K2: now also J1.10 (Pin_10); no longer J1.4 (Pin_4)
- net LED_K20: now also J2.12 (Pin_12); no longer J1.40 (Pin_40)
- net LED_K21: now also J2.20 (Pin_20); no longer J1.42 (Pin_42)
- net LED_K22: now also J2.28 (Pin_28); no longer J1.44 (Pin_44)
- net LED_K23: now also J2.36 (Pin_36); no longer J1.46 (Pin_46)
- net LED_K24: now also J2.44 (Pin_44); no longer J1.48 (Pin_48)
- net LED_K25: now also J1.6 (Pin_6); no longer J2.2 (Pin_2)
- net LED_K26: now also J1.14 (Pin_14); no longer J2.4 (Pin_4)
- net LED_K27: now also J1.22 (Pin_22); no longer J2.6 (Pin_6)
- net LED_K28: now also J1.30 (Pin_30); no longer J2.8 (Pin_8)
- net LED_K29: now also J1.38 (Pin_38); no longer J2.10 (Pin_10)
- net LED_K3: now also J1.18 (Pin_18); no longer J1.6 (Pin_6)
- net LED_K30: now also J1.46 (Pin_46); no longer J2.12 (Pin_12)
- net LED_K31: now also J2.6 (Pin_6); no longer J2.14 (Pin_14)
- net LED_K32: now also J2.14 (Pin_14); no longer J2.16 (Pin_16)
- net LED_K33: now also J2.22 (Pin_22); no longer J2.18 (Pin_18)
- net LED_K34: now also J2.30 (Pin_30); no longer J2.20 (Pin_20)
- net LED_K35: now also J2.38 (Pin_38); no longer J2.22 (Pin_22)
- net LED_K36: now also J2.46 (Pin_46); no longer J2.24 (Pin_24)
- net LED_K37: now also J1.8 (Pin_8); no longer J2.26 (Pin_26)
- net LED_K38: now also J1.16 (Pin_16); no longer J2.28 (Pin_28)
- net LED_K39: now also J1.24 (Pin_24); no longer J2.30 (Pin_30)
- net LED_K4: now also J1.26 (Pin_26); no longer J1.8 (Pin_8)
- net LED_K40: now also J1.32 (Pin_32); no longer J2.32 (Pin_32)
- net LED_K41: now also J1.40 (Pin_40); no longer J2.34 (Pin_34)
- net LED_K42: now also J1.48 (Pin_48); no longer J2.36 (Pin_36)
- net LED_K43: now also J2.8 (Pin_8); no longer J2.38 (Pin_38)
- net LED_K44: now also J2.16 (Pin_16); no longer J2.40 (Pin_40)
- net LED_K45: now also J2.24 (Pin_24); no longer J2.42 (Pin_42)
- net LED_K46: now also J2.32 (Pin_32); no longer J2.44 (Pin_44)
- net LED_K47: now also J2.40 (Pin_40); no longer J2.46 (Pin_46)
- net LED_K49: now also J4.2 (Pin_2); no longer J3.2 (Pin_2)
- net LED_K5: now also J1.34 (Pin_34); no longer J1.10 (Pin_10)
- net LED_K50: now also J4.10 (Pin_10); no longer J3.4 (Pin_4)
- net LED_K51: now also J4.18 (Pin_18); no longer J3.6 (Pin_6)
- net LED_K52: now also J4.26 (Pin_26); no longer J3.8 (Pin_8)
- net LED_K53: now also J4.34 (Pin_34); no longer J3.10 (Pin_10)
- net LED_K54: now also J4.42 (Pin_42); no longer J3.12 (Pin_12)
- net LED_K55: now also J3.2 (Pin_2); no longer J3.14 (Pin_14)
- net LED_K56: now also J3.10 (Pin_10); no longer J3.16 (Pin_16)
- net LED_K58: now also J3.26 (Pin_26); no longer J3.20 (Pin_20)
- net LED_K59: now also J3.34 (Pin_34); no longer J3.22 (Pin_22)
- net LED_K6: now also J1.42 (Pin_42); no longer J1.12 (Pin_12)
- net LED_K60: now also J3.42 (Pin_42); no longer J3.24 (Pin_24)
- net LED_K61: now also J4.4 (Pin_4); no longer J3.26 (Pin_26)
- net LED_K62: now also J4.12 (Pin_12); no longer J3.28 (Pin_28)
- net LED_K63: now also J4.20 (Pin_20); no longer J3.30 (Pin_30)
- net LED_K64: now also J4.28 (Pin_28); no longer J3.32 (Pin_32)
- net LED_K65: now also J4.36 (Pin_36); no longer J3.34 (Pin_34)
- net LED_K66: now also J4.44 (Pin_44); no longer J3.36 (Pin_36)
- net LED_K67: now also J3.4 (Pin_4); no longer J3.38 (Pin_38)
- net LED_K68: now also J3.12 (Pin_12); no longer J3.40 (Pin_40)
- net LED_K69: now also J3.20 (Pin_20); no longer J3.42 (Pin_42)
- net LED_K7: now also J2.2 (Pin_2); no longer J1.14 (Pin_14)
- net LED_K70: now also J3.28 (Pin_28); no longer J3.44 (Pin_44)
- net LED_K71: now also J3.36 (Pin_36); no longer J3.46 (Pin_46)
- net LED_K72: now also J3.44 (Pin_44); no longer J3.48 (Pin_48)
- net LED_K73: now also J4.6 (Pin_6); no longer J4.2 (Pin_2)
- net LED_K74: now also J4.14 (Pin_14); no longer J4.4 (Pin_4)
- net LED_K75: now also J4.22 (Pin_22); no longer J4.6 (Pin_6)
- net LED_K76: now also J4.30 (Pin_30); no longer J4.8 (Pin_8)
- net LED_K77: now also J4.38 (Pin_38); no longer J4.10 (Pin_10)
- net LED_K78: now also J4.46 (Pin_46); no longer J4.12 (Pin_12)
- net LED_K79: now also J3.6 (Pin_6); no longer J4.14 (Pin_14)
- net LED_K8: now also J2.10 (Pin_10); no longer J1.16 (Pin_16)
- net LED_K80: now also J3.14 (Pin_14); no longer J4.16 (Pin_16)
- net LED_K81: now also J3.22 (Pin_22); no longer J4.18 (Pin_18)
- net LED_K82: now also J3.30 (Pin_30); no longer J4.20 (Pin_20)
- net LED_K83: now also J3.38 (Pin_38); no longer J4.22 (Pin_22)
- net LED_K84: now also J3.46 (Pin_46); no longer J4.24 (Pin_24)
- net LED_K85: now also J4.8 (Pin_8); no longer J4.26 (Pin_26)
- net LED_K86: now also J4.16 (Pin_16); no longer J4.28 (Pin_28)
- net LED_K87: now also J4.24 (Pin_24); no longer J4.30 (Pin_30)
- net LED_K89: now also J4.40 (Pin_40); no longer J4.34 (Pin_34)
- net LED_K9: now also J2.18 (Pin_18); no longer J1.18 (Pin_18)
- net LED_K90: now also J4.48 (Pin_48); no longer J4.36 (Pin_36)
- net LED_K91: now also J3.8 (Pin_8); no longer J4.38 (Pin_38)
- net LED_K92: now also J3.16 (Pin_16); no longer J4.40 (Pin_40)
- net LED_K93: now also J3.24 (Pin_24); no longer J4.42 (Pin_42)
- net LED_K94: now also J3.32 (Pin_32); no longer J4.44 (Pin_44)
- net LED_K95: now also J3.40 (Pin_40); no longer J4.46 (Pin_46)
- net LED_K96: now also J3.48 (Pin_48); no longer J4.48 (Pin_48)
- net NTC10: now also U6.6 (I3); no longer U1.22 (I9)
- net NTC11: now also U6.5 (I4); no longer U1.21 (I10)
- net NTC12: now also U6.4 (I5); no longer U1.20 (I11)
- net NTC13: now also U1.3 (I6); no longer U1.19 (I12)
- net NTC14: now also U1.2 (I7); no longer U1.18 (I13)
- net NTC15: now also U1.23 (I8); no longer U1.17 (I14)
- net NTC16: now also U1.22 (I9); no longer U1.16 (I15)
- net NTC17: now also U1.21 (I10); no longer U2.9 (I0)
- net NTC18: now also U1.20 (I11); no longer U2.8 (I1)
- net NTC19: now also U6.3 (I6); no longer U2.7 (I2)
- net NTC20: now also U6.2 (I7); no longer U2.6 (I3)
- net NTC21: now also U6.23 (I8); no longer U2.5 (I4)
- net NTC22: now also U6.22 (I9); no longer U2.4 (I5)
- net NTC23: now also U6.21 (I10); no longer U2.3 (I6)
- net NTC24: now also U6.20 (I11); no longer U2.2 (I7)
- net NTC25: now also U1.19 (I12); no longer U2.23 (I8)
- net NTC26: now also U1.18 (I13); no longer U2.22 (I9)
- net NTC27: now also U1.17 (I14); no longer U2.21 (I10)
- net NTC28: now also U1.16 (I15); no longer U2.20 (I11)
- net NTC29: now also U2.9 (I0); no longer U2.19 (I12)
- net NTC30: now also U2.8 (I1); no longer U2.18 (I13)
- net NTC31: now also U6.19 (I12); no longer U2.17 (I14)
- net NTC32: now also U6.18 (I13); no longer U2.16 (I15)
- net NTC33: now also U6.17 (I14); no longer U3.9 (I0)
- net NTC34: now also U6.16 (I15); no longer U3.8 (I1)
- net NTC35: now also U5.9 (I0); no longer U3.7 (I2)
- net NTC36: now also U5.8 (I1); no longer U3.6 (I3)
- net NTC37: now also U2.7 (I2); no longer U3.5 (I4)
- net NTC38: now also U2.6 (I3); no longer U3.4 (I5)
- net NTC39: now also U2.5 (I4); no longer U3.3 (I6)
- net NTC40: now also U2.4 (I5); no longer U3.2 (I7)
- net NTC41: now also U2.3 (I6); no longer U3.23 (I8)
- net NTC42: now also U2.2 (I7); no longer U3.22 (I9)
- net NTC43: now also U5.7 (I2); no longer U3.21 (I10)
- net NTC44: now also U5.6 (I3); no longer U3.20 (I11)
- net NTC45: now also U5.5 (I4); no longer U3.19 (I12)
- net NTC46: now also U5.4 (I5); no longer U3.18 (I13)
- net NTC47: now also U5.3 (I6); no longer U3.17 (I14)
- net NTC48: now also U5.2 (I7); no longer U3.16 (I15)
- net NTC49: now also U2.23 (I8); no longer U4.9 (I0)
- net NTC50: now also U2.22 (I9); no longer U4.8 (I1)
- net NTC51: now also U2.21 (I10); no longer U4.7 (I2)
- net NTC52: now also U2.20 (I11); no longer U4.6 (I3)
- net NTC53: now also U2.19 (I12); no longer U4.5 (I4)
- net NTC54: now also U2.18 (I13); no longer U4.4 (I5)
- net NTC55: now also U5.23 (I8); no longer U4.3 (I6)
- net NTC56: now also U5.22 (I9); no longer U4.2 (I7)
- net NTC57: now also U5.21 (I10); no longer U4.23 (I8)
- net NTC58: now also U5.20 (I11); no longer U4.22 (I9)
- net NTC59: now also U5.19 (I12); no longer U4.21 (I10)
- net NTC60: now also U5.18 (I13); no longer U4.20 (I11)
- net NTC61: now also U2.17 (I14); no longer U4.19 (I12)
- net NTC62: now also U2.16 (I15); no longer U4.18 (I13)
- net NTC63: now also U3.9 (I0); no longer U4.17 (I14)
- net NTC64: now also U3.8 (I1); no longer U4.16 (I15)
- net NTC65: now also U3.7 (I2); no longer U5.9 (I0)
- net NTC66: now also U3.6 (I3); no longer U5.8 (I1)
- net NTC67: now also U5.17 (I14); no longer U5.7 (I2)
- net NTC68: now also U5.16 (I15); no longer U5.6 (I3)
- net NTC69: now also U4.9 (I0); no longer U5.5 (I4)
- net NTC7: now also U6.9 (I0); no longer U1.3 (I6)
- net NTC70: now also U4.8 (I1); no longer U5.4 (I5)
- net NTC71: now also U4.7 (I2); no longer U5.3 (I6)
- net NTC72: now also U4.6 (I3); no longer U5.2 (I7)
- net NTC73: now also U3.5 (I4); no longer U5.23 (I8)
- net NTC74: now also U3.4 (I5); no longer U5.22 (I9)
- net NTC75: now also U3.3 (I6); no longer U5.21 (I10)
- net NTC76: now also U3.2 (I7); no longer U5.20 (I11)
- net NTC77: now also U3.23 (I8); no longer U5.19 (I12)
- net NTC78: now also U3.22 (I9); no longer U5.18 (I13)
- net NTC79: now also U4.5 (I4); no longer U5.17 (I14)
- net NTC8: now also U6.8 (I1); no longer U1.2 (I7)
- net NTC80: now also U4.4 (I5); no longer U5.16 (I15)
- net NTC81: now also U4.3 (I6); no longer U6.9 (I0)
- net NTC82: now also U4.2 (I7); no longer U6.8 (I1)
- net NTC83: now also U4.23 (I8); no longer U6.7 (I2)
- net NTC84: now also U4.22 (I9); no longer U6.6 (I3)
- net NTC85: now also U3.21 (I10); no longer U6.5 (I4)
- net NTC86: now also U3.20 (I11); no longer U6.4 (I5)
- net NTC87: now also U3.19 (I12); no longer U6.3 (I6)
- net NTC88: now also U3.18 (I13); no longer U6.2 (I7)
- net NTC89: now also U3.17 (I14); no longer U6.23 (I8)
- net NTC9: now also U6.7 (I2); no longer U1.23 (I8)
- net NTC90: now also U3.16 (I15); no longer U6.22 (I9)
- net NTC91: now also U4.21 (I10); no longer U6.21 (I10)
- net NTC92: now also U4.20 (I11); no longer U6.20 (I11)
- net NTC93: now also U4.19 (I12); no longer U6.19 (I12)
- net NTC94: now also U4.18 (I13); no longer U6.18 (I13)
- net NTC95: now also U4.17 (I14); no longer U6.17 (I14)
- net NTC96: now also U4.16 (I15); no longer U6.16 (I15)

Commit message: Mux split 4 left / 2 right, column-pair NTC mapping
- U1-U4 left stack, U5/U6 right beside J5 (user layout request)
- Each mux owns 2 columns; 94 NTC labels remapped; netlists verify
- Old stubs swept, GND re-stitched, placement DRC clean

Co-Authored-By: Claude Fable 5 <noreply@anthropic.com>
Claude-Session: https://claude.ai/code/session_017oD54uh7Tvu54u9NPQNcZB
Connections:
- net NTC10: now also U5.23 (I8); no longer U6.6 (I3)
- net NTC11: now also U6.9 (I0); no longer U6.5 (I4)
- net NTC12: now also U6.23 (I8); no longer U6.4 (I5)
- net NTC13: now also U1.8 (I1); no longer U1.3 (I6)
- net NTC14: now also U1.22 (I9); no longer U1.2 (I7)
- net NTC15: now also U2.8 (I1); no longer U1.23 (I8)
- net NTC16: now also U2.22 (I9); no longer U1.22 (I9)
- net NTC17: now also U3.8 (I1); no longer U1.21 (I10)
- net NTC18: now also U3.22 (I9); no longer U1.20 (I11)
- net NTC19: now also U4.8 (I1); no longer U6.3 (I6)
- net NTC2: now also U1.23 (I8); no longer U1.8 (I1)
- net NTC20: now also U4.22 (I9); no longer U6.2 (I7)
- net NTC21: now also U5.8 (I1); no longer U6.23 (I8)
- net NTC22: now also U5.22 (I9); no longer U6.22 (I9)
- net NTC23: now also U6.8 (I1); no longer U6.21 (I10)
- net NTC24: now also U6.22 (I9); no longer U6.20 (I11)
- net NTC25: now also U1.7 (I2); no longer U1.19 (I12)
- net NTC26: now also U1.21 (I10); no longer U1.18 (I13)
- net NTC27: now also U2.7 (I2); no longer U1.17 (I14)
- net NTC28: now also U2.21 (I10); no longer U1.16 (I15)
- net NTC29: now also U3.7 (I2); no longer U2.9 (I0)
- net NTC3: now also U2.9 (I0); no longer U1.7 (I2)
- net NTC30: now also U3.21 (I10); no longer U2.8 (I1)
- net NTC31: now also U4.7 (I2); no longer U6.19 (I12)
- net NTC32: now also U4.21 (I10); no longer U6.18 (I13)
- net NTC33: now also U5.7 (I2); no longer U6.17 (I14)
- net NTC34: now also U5.21 (I10); no longer U6.16 (I15)
- net NTC35: now also U6.7 (I2); no longer U5.9 (I0)
- net NTC36: now also U6.21 (I10); no longer U5.8 (I1)
- net NTC37: now also U1.6 (I3); no longer U2.7 (I2)
- net NTC38: now also U1.20 (I11); no longer U2.6 (I3)
- net NTC39: now also U2.6 (I3); no longer U2.5 (I4)
- net NTC4: now also U2.23 (I8); no longer U1.6 (I3)
- net NTC40: now also U2.20 (I11); no longer U2.4 (I5)
- net NTC41: now also U3.6 (I3); no longer U2.3 (I6)
- net NTC42: now also U3.20 (I11); no longer U2.2 (I7)
- net NTC43: now also U4.6 (I3); no longer U5.7 (I2)
- net NTC44: now also U4.20 (I11); no longer U5.6 (I3)
- net NTC45: now also U5.6 (I3); no longer U5.5 (I4)
- net NTC46: now also U5.20 (I11); no longer U5.4 (I5)
- net NTC47: now also U6.6 (I3); no longer U5.3 (I6)
- net NTC48: now also U6.20 (I11); no longer U5.2 (I7)
- net NTC49: now also U1.5 (I4); no longer U2.23 (I8)
- net NTC5: now also U3.9 (I0); no longer U1.5 (I4)
- net NTC50: now also U1.19 (I12); no longer U2.22 (I9)
- net NTC51: now also U2.5 (I4); no longer U2.21 (I10)
- net NTC52: now also U2.19 (I12); no longer U2.20 (I11)
- net NTC53: now also U3.5 (I4); no longer U2.19 (I12)
- net NTC54: now also U3.19 (I12); no longer U2.18 (I13)
- net NTC55: now also U4.5 (I4); no longer U5.23 (I8)
- net NTC56: now also U4.19 (I12); no longer U5.22 (I9)
- net NTC57: now also U5.5 (I4); no longer U5.21 (I10)
- net NTC58: now also U5.19 (I12); no longer U5.20 (I11)
- net NTC59: now also U6.5 (I4); no longer U5.19 (I12)
- net NTC6: now also U3.23 (I8); no longer U1.4 (I5)
- net NTC60: now also U6.19 (I12); no longer U5.18 (I13)
- net NTC61: now also U1.4 (I5); no longer U2.17 (I14)
- net NTC62: now also U1.18 (I13); no longer U2.16 (I15)
- net NTC63: now also U2.4 (I5); no longer U3.9 (I0)
- net NTC64: now also U2.18 (I13); no longer U3.8 (I1)
- net NTC65: now also U3.4 (I5); no longer U3.7 (I2)
- net NTC66: now also U3.18 (I13); no longer U3.6 (I3)
- net NTC67: now also U4.4 (I5); no longer U5.17 (I14)
- net NTC68: now also U4.18 (I13); no longer U5.16 (I15)
- net NTC69: now also U5.4 (I5); no longer U4.9 (I0)
- net NTC7: now also U4.9 (I0); no longer U6.9 (I0)
- net NTC70: now also U5.18 (I13); no longer U4.8 (I1)
- net NTC71: now also U6.4 (I5); no longer U4.7 (I2)
- net NTC72: now also U6.18 (I13); no longer U4.6 (I3)
- net NTC73: now also U1.3 (I6); no longer U3.5 (I4)
- net NTC74: now also U1.17 (I14); no longer U3.4 (I5)
- net NTC75: now also U2.3 (I6); no longer U3.3 (I6)
- net NTC76: now also U2.17 (I14); no longer U3.2 (I7)
- net NTC77: now also U3.3 (I6); no longer U3.23 (I8)
- net NTC78: now also U3.17 (I14); no longer U3.22 (I9)
- net NTC79: now also U4.3 (I6); no longer U4.5 (I4)
- net NTC8: now also U4.23 (I8); no longer U6.8 (I1)
- net NTC80: now also U4.17 (I14); no longer U4.4 (I5)
- net NTC81: now also U5.3 (I6); no longer U4.3 (I6)
- net NTC82: now also U5.17 (I14); no longer U4.2 (I7)
- net NTC83: now also U6.3 (I6); no longer U4.23 (I8)
- net NTC84: now also U6.17 (I14); no longer U4.22 (I9)
- net NTC85: now also U1.2 (I7); no longer U3.21 (I10)
- net NTC86: now also U1.16 (I15); no longer U3.20 (I11)
- net NTC87: now also U2.2 (I7); no longer U3.19 (I12)
- net NTC88: now also U2.16 (I15); no longer U3.18 (I13)
- net NTC89: now also U3.2 (I7); no longer U3.17 (I14)
- net NTC9: now also U5.9 (I0); no longer U6.7 (I2)
- net NTC91: now also U4.2 (I7); no longer U4.21 (I10)
- net NTC92: now also U4.16 (I15); no longer U4.20 (I11)
- net NTC93: now also U5.2 (I7); no longer U4.19 (I12)
- net NTC94: now also U5.16 (I15); no longer U4.18 (I13)
- net NTC95: now also U6.2 (I7); no longer U4.17 (I14)
- net NTC96: now also U6.16 (I15); no longer U4.16 (I15)

Commit message: Geometric mux input assignment (crossing-free fan-in), 88 labels remapped
Co-Authored-By: Claude Fable 5 <noreply@anthropic.com>
Claude-Session: https://claude.ai/code/session_017oD54uh7Tvu54u9NPQNcZB
Connections:
- net NTC1: now also U1.23 (I8); no longer U1.9 (I0)
- net NTC10: now also U5.9 (I0); no longer U5.23 (I8)
- net NTC11: now also U6.16 (I15); no longer U6.9 (I0)
- net NTC12: now also U6.9 (I0); no longer U6.23 (I8)
- net NTC13: now also U1.22 (I9); no longer U1.8 (I1)
- net NTC14: now also U1.3 (I6); no longer U1.22 (I9)
- net NTC15: now also U2.22 (I9); no longer U2.8 (I1)
- net NTC16: now also U2.3 (I6); no longer U2.22 (I9)
- net NTC17: now also U3.22 (I9); no longer U3.8 (I1)
- net NTC18: now also U3.3 (I6); no longer U3.22 (I9)
- net NTC2: now also U1.2 (I7); no longer U1.23 (I8)
- net NTC20: now also U4.17 (I14); no longer U4.22 (I9)
- net NTC21: now also U5.17 (I14); no longer U5.8 (I1)
- net NTC22: now also U5.8 (I1); no longer U5.22 (I9)
- net NTC23: now also U6.17 (I14); no longer U6.8 (I1)
- net NTC24: now also U6.8 (I1); no longer U6.22 (I9)
- net NTC25: now also U1.21 (I10); no longer U1.7 (I2)
- net NTC26: now also U1.4 (I5); no longer U1.21 (I10)
- net NTC27: now also U2.21 (I10); no longer U2.7 (I2)
- net NTC28: now also U2.4 (I5); no longer U2.21 (I10)
- net NTC29: now also U3.21 (I10); no longer U3.7 (I2)
- net NTC3: now also U2.23 (I8); no longer U2.9 (I0)
- net NTC30: now also U3.4 (I5); no longer U3.21 (I10)
- net NTC32: now also U4.18 (I13); no longer U4.21 (I10)
- net NTC33: now also U5.18 (I13); no longer U5.7 (I2)
- net NTC34: now also U5.7 (I2); no longer U5.21 (I10)
- net NTC35: now also U6.18 (I13); no longer U6.7 (I2)
- net NTC36: now also U6.7 (I2); no longer U6.21 (I10)
- net NTC37: now also U1.20 (I11); no longer U1.6 (I3)
- net NTC38: now also U1.5 (I4); no longer U1.20 (I11)
- net NTC39: now also U2.20 (I11); no longer U2.6 (I3)
- net NTC4: now also U2.2 (I7); no longer U2.23 (I8)
- net NTC40: now also U2.5 (I4); no longer U2.20 (I11)
- net NTC41: now also U3.20 (I11); no longer U3.6 (I3)
- net NTC42: now also U3.5 (I4); no longer U3.20 (I11)
- net NTC44: now also U4.19 (I12); no longer U4.20 (I11)
- net NTC45: now also U5.19 (I12); no longer U5.6 (I3)
- net NTC46: now also U5.6 (I3); no longer U5.20 (I11)
- net NTC47: now also U6.19 (I12); no longer U6.6 (I3)
- net NTC48: now also U6.6 (I3); no longer U6.20 (I11)
- net NTC49: now also U1.19 (I12); no longer U1.5 (I4)
- net NTC5: now also U3.23 (I8); no longer U3.9 (I0)
- net NTC50: now also U1.6 (I3); no longer U1.19 (I12)
- net NTC51: now also U2.19 (I12); no longer U2.5 (I4)
- net NTC52: now also U2.6 (I3); no longer U2.19 (I12)
- net NTC53: now also U3.19 (I12); no longer U3.5 (I4)
- net NTC54: now also U3.6 (I3); no longer U3.19 (I12)
- net NTC56: now also U4.20 (I11); no longer U4.19 (I12)
- net NTC57: now also U5.20 (I11); no longer U5.5 (I4)
- net NTC58: now also U5.5 (I4); no longer U5.19 (I12)
- net NTC59: now also U6.20 (I11); no longer U6.5 (I4)
- net NTC6: now also U3.2 (I7); no longer U3.23 (I8)
- net NTC60: now also U6.5 (I4); no longer U6.19 (I12)
- net NTC61: now also U1.18 (I13); no longer U1.4 (I5)
- net NTC62: now also U1.7 (I2); no longer U1.18 (I13)
- net NTC63: now also U2.18 (I13); no longer U2.4 (I5)
- net NTC64: now also U2.7 (I2); no longer U2.18 (I13)
- net NTC65: now also U3.18 (I13); no longer U3.4 (I5)
- net NTC66: now also U3.7 (I2); no longer U3.18 (I13)
- net NTC68: now also U4.21 (I10); no longer U4.18 (I13)
- net NTC69: now also U5.21 (I10); no longer U5.4 (I5)
- net NTC70: now also U5.4 (I5); no longer U5.18 (I13)
- net NTC71: now also U6.21 (I10); no longer U6.4 (I5)
- net NTC72: now also U6.4 (I5); no longer U6.18 (I13)
- net NTC73: now also U1.17 (I14); no longer U1.3 (I6)
- net NTC74: now also U1.8 (I1); no longer U1.17 (I14)
- net NTC75: now also U2.17 (I14); no longer U2.3 (I6)
- net NTC76: now also U2.8 (I1); no longer U2.17 (I14)
- net NTC77: now also U3.17 (I14); no longer U3.3 (I6)
- net NTC78: now also U3.8 (I1); no longer U3.17 (I14)
- net NTC8: now also U4.16 (I15); no longer U4.23 (I8)
- net NTC80: now also U4.22 (I9); no longer U4.17 (I14)
- net NTC81: now also U5.22 (I9); no longer U5.3 (I6)
- net NTC82: now also U5.3 (I6); no longer U5.17 (I14)
- net NTC83: now also U6.22 (I9); no longer U6.3 (I6)
- net NTC84: now also U6.3 (I6); no longer U6.17 (I14)
- net NTC85: now also U1.16 (I15); no longer U1.2 (I7)
- net NTC86: now also U1.9 (I0); no longer U1.16 (I15)
- net NTC87: now also U2.16 (I15); no longer U2.2 (I7)
- net NTC88: now also U2.9 (I0); no longer U2.16 (I15)
- net NTC89: now also U3.16 (I15); no longer U3.2 (I7)
- net NTC9: now also U5.16 (I15); no longer U5.9 (I0)
- net NTC90: now also U3.9 (I0); no longer U3.16 (I15)
- net NTC92: now also U4.23 (I8); no longer U4.16 (I15)
- net NTC93: now also U5.23 (I8); no longer U5.2 (I7)
- net NTC94: now also U5.2 (I7); no longer U5.16 (I15)
- net NTC95: now also U6.23 (I8); no longer U6.2 (I7)
- net NTC96: now also U6.2 (I7); no longer U6.16 (I15)
