File: 12x8 Led Array 9mm pitch/12x8 Led Array 9mm pitch.kicad_sch (KiCad schematic)
At the start: 27 parts, among them J1 LED ch 1-16, J2 LED ch 17-32, J3 LED ch 33-48, J4 LED ch 49-64, J5 LED ch 65-80, J6 LED ch 81-96, J9 logic/analog, U1 CD74HC4067M96, U2 CD74HC4067M96, U3 CD74HC4067M96, U4 CD74HC4067M96, U5 CD74HC4067M96, U6 CD74HC4067M96

Commit message: LED board support parts copied to control-board topology (15mm border kept)
J1/J4 vertical on left edge, J2/J3 top, J5/J6 bottom, mux stack +
J9 on right strip; pin_maps v6 (CONN_MAP re-optimized, NTC_MAP
re-derived for right-strip muxes); schematics regenerated, netlists
verified, pads re-netted, zones refilled. New scripts:
layout_led_support.py, apply_netlist.py.

Co-Authored-By: Claude Fable 5 <noreply@anthropic.com>
Claude-Session: https://claude.ai/code/session_017oD54uh7Tvu54u9NPQNcZB
Connections:
- net LED_A10: now also J1.21 (Pin_21); no longer J1.27 (Pin_27)
- net LED_A11: now also J1.23 (Pin_23); no longer J1.31 (Pin_31)
- net LED_A12: now also J1.25 (Pin_25); no longer J1.33 (Pin_33)
- net LED_A13: now also J1.27 (Pin_27); no longer J1.11 (Pin_11)
- net LED_A14: now also J1.29 (Pin_29); no longer J1.17 (Pin_17)
- net LED_A15: now also J1.31 (Pin_31); no longer J1.23 (Pin_23)
- net LED_A16: now also J1.33 (Pin_33); no longer J1.29 (Pin_29)
- net LED_A54: now also J4.11 (Pin_11); no longer J4.13 (Pin_13)
- net LED_A55: now also J4.13 (Pin_13); no longer J4.15 (Pin_15)
- net LED_A56: now also J4.15 (Pin_15); no longer J4.21 (Pin_21)
- net LED_A57: now also J4.17 (Pin_17); no longer J4.25 (Pin_25)
- net LED_A58: now also J4.21 (Pin_21); no longer J4.27 (Pin_27)
- net LED_A59: now also J4.23 (Pin_23); no longer J4.31 (Pin_31)
- net LED_A6: now also J1.11 (Pin_11); no longer J1.13 (Pin_13)
- net LED_A60: now also J4.25 (Pin_25); no longer J4.33 (Pin_33)
- net LED_A61: now also J4.27 (Pin_27); no longer J4.11 (Pin_11)
- net LED_A62: now also J4.29 (Pin_29); no longer J4.17 (Pin_17)
- net LED_A63: now also J4.31 (Pin_31); no longer J4.23 (Pin_23)
- net LED_A64: now also J4.33 (Pin_33); no longer J4.29 (Pin_29)
- net LED_A7: now also J1.13 (Pin_13); no longer J1.15 (Pin_15)
- net LED_A8: now also J1.15 (Pin_15); no longer J1.21 (Pin_21)
- net LED_A9: now also J1.17 (Pin_17); no longer J1.25 (Pin_25)
- net LED_K10: now also J1.22 (Pin_22); no longer J1.28 (Pin_28)
- net LED_K11: now also J1.24 (Pin_24); no longer J1.32 (Pin_32)
- net LED_K12: now also J1.26 (Pin_26); no longer J1.34 (Pin_34)
- net LED_K13: now also J1.28 (Pin_28); no longer J1.12 (Pin_12)
- net LED_K14: now also J1.30 (Pin_30); no longer J1.18 (Pin_18)
- net LED_K15: now also J1.32 (Pin_32); no longer J1.24 (Pin_24)
- net LED_K16: now also J1.34 (Pin_34); no longer J1.30 (Pin_30)
- net LED_K54: now also J4.12 (Pin_12); no longer J4.14 (Pin_14)
- net LED_K55: now also J4.14 (Pin_14); no longer J4.16 (Pin_16)
- net LED_K56: now also J4.16 (Pin_16); no longer J4.22 (Pin_22)
- net LED_K57: now also J4.18 (Pin_18); no longer J4.26 (Pin_26)
- net LED_K58: now also J4.22 (Pin_22); no longer J4.28 (Pin_28)
- net LED_K59: now also J4.24 (Pin_24); no longer J4.32 (Pin_32)
- net LED_K6: now also J1.12 (Pin_12); no longer J1.14 (Pin_14)
- net LED_K60: now also J4.26 (Pin_26); no longer J4.34 (Pin_34)
- net LED_K61: now also J4.28 (Pin_28); no longer J4.12 (Pin_12)
- net LED_K62: now also J4.30 (Pin_30); no longer J4.18 (Pin_18)
- net LED_K63: now also J4.32 (Pin_32); no longer J4.24 (Pin_24)
- net LED_K64: now also J4.34 (Pin_34); no longer J4.30 (Pin_30)
- net LED_K7: now also J1.14 (Pin_14); no longer J1.16 (Pin_16)
- net LED_K8: now also J1.16 (Pin_16); no longer J1.22 (Pin_22)
- net LED_K9: now also J1.18 (Pin_18); no longer J1.26 (Pin_26)
- net NTC10: now also U5.22 (I9); no longer U5.9 (I0)
- net NTC11: now also U6.23 (I8); no longer U6.16 (I15)
- net NTC12: now also U6.22 (I9); no longer U6.9 (I0)
- net NTC13: now also U1.21 (I10); no longer U1.22 (I9)
- net NTC14: now also U1.20 (I11); no longer U1.3 (I6)
- net NTC15: now also U2.21 (I10); no longer U2.22 (I9)
- net NTC16: now also U2.20 (I11); no longer U2.3 (I6)
- net NTC17: now also U3.21 (I10); no longer U3.22 (I9)
- net NTC18: now also U3.20 (I11); no longer U3.3 (I6)
- net NTC19: now also U4.21 (I10); no longer U4.8 (I1)
- net NTC2: now also U1.22 (I9); no longer U1.2 (I7)
- net NTC20: now also U4.20 (I11); no longer U4.17 (I14)
- net NTC21: now also U5.21 (I10); no longer U5.17 (I14)
- net NTC22: now also U5.20 (I11); no longer U5.8 (I1)
- net NTC23: now also U6.21 (I10); no longer U6.17 (I14)
- net NTC24: now also U6.20 (I11); no longer U6.8 (I1)
- net NTC25: now also U1.19 (I12); no longer U1.21 (I10)
- net NTC26: now also U1.18 (I13); no longer U1.4 (I5)
- net NTC27: now also U2.19 (I12); no longer U2.21 (I10)
- net NTC28: now also U2.18 (I13); no longer U2.4 (I5)
- net NTC29: now also U3.19 (I12); no longer U3.21 (I10)
- net NTC30: now also U3.18 (I13); no longer U3.4 (I5)
- net NTC31: now also U4.19 (I12); no longer U4.7 (I2)
- net NTC33: now also U5.19 (I12); no longer U5.18 (I13)
- net NTC34: now also U5.18 (I13); no longer U5.7 (I2)
- net NTC35: now also U6.19 (I12); no longer U6.18 (I13)
- net NTC36: now also U6.18 (I13); no longer U6.7 (I2)
- net NTC37: now also U1.17 (I14); no longer U1.20 (I11)
- net NTC38: now also U1.16 (I15); no longer U1.5 (I4)
- net NTC39: now also U2.17 (I14); no longer U2.20 (I11)
- net NTC4: now also U2.22 (I9); no longer U2.2 (I7)
- net NTC40: now also U2.16 (I15); no longer U2.5 (I4)
- net NTC41: now also U3.17 (I14); no longer U3.20 (I11)
- net NTC42: now also U3.16 (I15); no longer U3.5 (I4)
- net NTC43: now also U4.17 (I14); no longer U4.6 (I3)
- net NTC44: now also U4.16 (I15); no longer U4.19 (I12)
- net NTC45: now also U5.17 (I14); no longer U5.19 (I12)
- net NTC46: now also U5.16 (I15); no longer U5.6 (I3)
- net NTC47: now also U6.17 (I14); no longer U6.19 (I12)
- net NTC48: now also U6.16 (I15); no longer U6.6 (I3)
- net NTC49: now also U1.2 (I7); no longer U1.19 (I12)
- net NTC50: now also U1.3 (I6); no longer U1.6 (I3)
- net NTC51: now also U2.2 (I7); no longer U2.19 (I12)
- net NTC52: now also U2.3 (I6); no longer U2.6 (I3)
- net NTC53: now also U3.2 (I7); no longer U3.19 (I12)
- net NTC54: now also U3.3 (I6); no longer U3.6 (I3)
- net NTC55: now also U4.2 (I7); no longer U4.5 (I4)
- net NTC56: now also U4.3 (I6); no longer U4.20 (I11)
- net NTC57: now also U5.2 (I7); no longer U5.20 (I11)
- net NTC58: now also U5.3 (I6); no longer U5.5 (I4)
- net NTC59: now also U6.2 (I7); no longer U6.20 (I11)
- net NTC6: now also U3.22 (I9); no longer U3.2 (I7)
- net NTC60: now also U6.3 (I6); no longer U6.5 (I4)
- net NTC61: now also U1.4 (I5); no longer U1.18 (I13)
- net NTC62: now also U1.5 (I4); no longer U1.7 (I2)
- net NTC63: now also U2.4 (I5); no longer U2.18 (I13)
- net NTC64: now also U2.5 (I4); no longer U2.7 (I2)
- net NTC65: now also U3.4 (I5); no longer U3.18 (I13)
- net NTC66: now also U3.5 (I4); no longer U3.7 (I2)
- net NTC68: now also U4.5 (I4); no longer U4.21 (I10)
- net NTC69: now also U5.4 (I5); no longer U5.21 (I10)
- net NTC7: now also U4.23 (I8); no longer U4.9 (I0)
- net NTC70: now also U5.5 (I4); no longer U5.4 (I5)
- net NTC71: now also U6.4 (I5); no longer U6.21 (I10)
- net NTC72: now also U6.5 (I4); no longer U6.4 (I5)
- net NTC73: now also U1.6 (I3); no longer U1.17 (I14)
- net NTC74: now also U1.7 (I2); no longer U1.8 (I1)
- net NTC75: now also U2.6 (I3); no longer U2.17 (I14)
- net NTC76: now also U2.7 (I2); no longer U2.8 (I1)
- net NTC77: now also U3.6 (I3); no longer U3.17 (I14)
- net NTC78: now also U3.7 (I2); no longer U3.8 (I1)
- net NTC79: now also U4.6 (I3); no longer U4.3 (I6)
- net NTC8: now also U4.22 (I9); no longer U4.16 (I15)
- net NTC80: now also U4.7 (I2); no longer U4.22 (I9)
- net NTC81: now also U5.6 (I3); no longer U5.22 (I9)
- net NTC82: now also U5.7 (I2); no longer U5.3 (I6)
- net NTC83: now also U6.6 (I3); no longer U6.22 (I9)
- net NTC84: now also U6.7 (I2); no longer U6.3 (I6)
- net NTC85: now also U1.8 (I1); no longer U1.16 (I15)
- net NTC87: now also U2.8 (I1); no longer U2.16 (I15)
- net NTC89: now also U3.8 (I1); no longer U3.16 (I15)
- net NTC9: now also U5.23 (I8); no longer U5.16 (I15)
- net NTC91: now also U4.8 (I1); no longer U4.2 (I7)
- net NTC92: now also U4.9 (I0); no longer U4.23 (I8)
- net NTC93: now also U5.8 (I1); no longer U5.23 (I8)
- net NTC94: now also U5.9 (I0); no longer U5.2 (I7)
- net NTC95: now also U6.8 (I1); no longer U6.23 (I8)
- net NTC96: now also U6.9 (I0); no longer U6.2 (I7)
