File: 12x8 Led Array 9mm pitch/12x8 Led Array 9mm pitch.kicad_sch (KiCad schematic)
At the start: 27 parts, among them J1 LED ch 1-16, J2 LED ch 17-32, J3 LED ch 33-48, J4 LED ch 49-64, J5 LED ch 65-80, J6 LED ch 81-96, J9 logic/analog, U1 CD74HC4067M96, U2 CD74HC4067M96, U3 CD74HC4067M96, U4 CD74HC4067M96, U5 CD74HC4067M96, U6 CD74HC4067M96

Commit message: LED-array pinout optimization: zero ribbon fan-out crossings + proximity NTC muxing
CONN_MAP -> LED-board-optimal nested pin order: fan-out crossings on the
LED board 536->0 across all six ribbons; control board near-Pareto
(440->464 inversions, J1/J4 improved to 0). Shared 1:1 cable respected.
NTC_MAP -> each mux takes its 16 nearest NTCs (proximity row-bands for the
right-edge stack): analog trace length -11% (8107->7222mm), horizontal
fan-in. PCA_MAP carried through unchanged (control-internal).

pin_maps v7; schematics regenerated; netlists ALL MATCH + cross-board OK;
286/192 pads re-netted; zones refilled. New: optimize_led_pins.py.

Co-Authored-By: Claude Fable 5 <noreply@anthropic.com>
Claude-Session: https://claude.ai/code/session_017oD54uh7Tvu54u9NPQNcZB
Connections:
- net LED_A1: now also J1.33 (Pin_33); no longer J1.1 (Pin_1)
- net LED_A10: now also J1.13 (Pin_13); no longer J1.21 (Pin_21)
- net LED_A11: now also J1.11 (Pin_11); no longer J1.23 (Pin_23)
- net LED_A12: now also J1.9 (Pin_9); no longer J1.25 (Pin_25)
- net LED_A13: now also J1.7 (Pin_7); no longer J1.27 (Pin_27)
- net LED_A14: now also J1.5 (Pin_5); no longer J1.29 (Pin_29)
- net LED_A15: now also J1.3 (Pin_3); no longer J1.31 (Pin_31)
- net LED_A16: now also J1.1 (Pin_1); no longer J1.33 (Pin_33)
- net LED_A17: now also J2.9 (Pin_9); no longer J2.33 (Pin_33)
- net LED_A18: now also J2.13 (Pin_13); no longer J2.31 (Pin_31)
- net LED_A19: now also J2.17 (Pin_17); no longer J2.29 (Pin_29)
- net LED_A2: now also J1.31 (Pin_31); no longer J1.3 (Pin_3)
- net LED_A20: now also J2.23 (Pin_23); no longer J2.27 (Pin_27)
- net LED_A21: now also J2.27 (Pin_27); no longer J2.25 (Pin_25)
- net LED_A22: now also J2.29 (Pin_29); no longer J2.23 (Pin_23)
- net LED_A23: now also J2.31 (Pin_31); no longer J2.21 (Pin_21)
- net LED_A24: now also J2.33 (Pin_33); no longer J2.17 (Pin_17)
- net LED_A25: now also J2.1 (Pin_1); no longer J2.15 (Pin_15)
- net LED_A26: now also J2.3 (Pin_3); no longer J2.13 (Pin_13)
- net LED_A27: now also J2.5 (Pin_5); no longer J2.11 (Pin_11)
- net LED_A28: now also J2.7 (Pin_7); no longer J2.9 (Pin_9)
- net LED_A29: now also J2.11 (Pin_11); no longer J2.7 (Pin_7)
- net LED_A3: now also J1.29 (Pin_29); no longer J1.5 (Pin_5)
- net LED_A30: now also J2.15 (Pin_15); no longer J2.5 (Pin_5)
- net LED_A31: now also J2.21 (Pin_21); no longer J2.3 (Pin_3)
- net LED_A32: now also J2.25 (Pin_25); no longer J2.1 (Pin_1)
- net LED_A33: now also J3.17 (Pin_17); no longer J3.33 (Pin_33)
- net LED_A34: now also J3.23 (Pin_23); no longer J3.31 (Pin_31)
- net LED_A35: now also J3.27 (Pin_27); no longer J3.29 (Pin_29)
- net LED_A36: now also J3.31 (Pin_31); no longer J3.27 (Pin_27)
- net LED_A37: now also J3.1 (Pin_1); no longer J3.25 (Pin_25)
- net LED_A38: now also J3.3 (Pin_3); no longer J3.23 (Pin_23)
- net LED_A39: now also J3.5 (Pin_5); no longer J3.21 (Pin_21)
- net LED_A4: now also J1.27 (Pin_27); no longer J1.7 (Pin_7)
- net LED_A40: now also J3.7 (Pin_7); no longer J3.17 (Pin_17)
- net LED_A41: now also J3.9 (Pin_9); no longer J3.15 (Pin_15)
- net LED_A42: now also J3.11 (Pin_11); no longer J3.13 (Pin_13)
- net LED_A43: now also J3.13 (Pin_13); no longer J3.11 (Pin_11)
- net LED_A44: now also J3.15 (Pin_15); no longer J3.9 (Pin_9)
- net LED_A45: now also J3.21 (Pin_21); no longer J3.7 (Pin_7)
- net LED_A46: now also J3.25 (Pin_25); no longer J3.5 (Pin_5)
- net LED_A47: now also J3.29 (Pin_29); no longer J3.3 (Pin_3)
- net LED_A48: now also J3.33 (Pin_33); no longer J3.1 (Pin_1)
- net LED_A49: now also J4.33 (Pin_33); no longer J4.1 (Pin_1)
- net LED_A5: now also J1.25 (Pin_25); no longer J1.9 (Pin_9)
- net LED_A50: now also J4.31 (Pin_31); no longer J4.3 (Pin_3)
- net LED_A51: now also J4.29 (Pin_29); no longer J4.5 (Pin_5)
- net LED_A52: now also J4.27 (Pin_27); no longer J4.7 (Pin_7)
- net LED_A53: now also J4.25 (Pin_25); no longer J4.9 (Pin_9)
- net LED_A54: now also J4.23 (Pin_23); no longer J4.11 (Pin_11)
- net LED_A55: now also J4.21 (Pin_21); no longer J4.13 (Pin_13)
- net LED_A56: now also J4.17 (Pin_17); no longer J4.15 (Pin_15)
- net LED_A57: now also J4.15 (Pin_15); no longer J4.17 (Pin_17)
- net LED_A58: now also J4.13 (Pin_13); no longer J4.21 (Pin_21)
- net LED_A59: now also J4.11 (Pin_11); no longer J4.23 (Pin_23)
- net LED_A6: now also J1.23 (Pin_23); no longer J1.11 (Pin_11)
- net LED_A60: now also J4.9 (Pin_9); no longer J4.25 (Pin_25)
- net LED_A61: now also J4.7 (Pin_7); no longer J4.27 (Pin_27)
- net LED_A62: now also J4.5 (Pin_5); no longer J4.29 (Pin_29)
- net LED_A63: now also J4.3 (Pin_3); no longer J4.31 (Pin_31)
- net LED_A64: now also J4.1 (Pin_1); no longer J4.33 (Pin_33)
- net LED_A65: now also J5.9 (Pin_9); no longer J5.33 (Pin_33)
- net LED_A66: now also J5.13 (Pin_13); no longer J5.31 (Pin_31)
- net LED_A67: now also J5.17 (Pin_17); no longer J5.29 (Pin_29)
- net LED_A68: now also J5.23 (Pin_23); no longer J5.27 (Pin_27)
- net LED_A69: now also J5.27 (Pin_27); no longer J5.25 (Pin_25)
- net LED_A7: now also J1.21 (Pin_21); no longer J1.13 (Pin_13)
- net LED_A70: now also J5.29 (Pin_29); no longer J5.23 (Pin_23)
- net LED_A71: now also J5.31 (Pin_31); no longer J5.21 (Pin_21)
- net LED_A72: now also J5.33 (Pin_33); no longer J5.17 (Pin_17)
- net LED_A73: now also J5.1 (Pin_1); no longer J5.15 (Pin_15)
- net LED_A74: now also J5.3 (Pin_3); no longer J5.13 (Pin_13)
- net LED_A75: now also J5.5 (Pin_5); no longer J5.11 (Pin_11)
- net LED_A76: now also J5.7 (Pin_7); no longer J5.9 (Pin_9)
- net LED_A77: now also J5.11 (Pin_11); no longer J5.7 (Pin_7)
- net LED_A78: now also J5.15 (Pin_15); no longer J5.5 (Pin_5)
- net LED_A79: now also J5.21 (Pin_21); no longer J5.3 (Pin_3)
- net LED_A8: now also J1.17 (Pin_17); no longer J1.15 (Pin_15)
- net LED_A80: now also J5.25 (Pin_25); no longer J5.1 (Pin_1)
- net LED_A81: now also J6.17 (Pin_17); no longer J6.33 (Pin_33)
- net LED_A82: now also J6.23 (Pin_23); no longer J6.31 (Pin_31)
- net LED_A83: now also J6.27 (Pin_27); no longer J6.29 (Pin_29)
- net LED_A84: now also J6.31 (Pin_31); no longer J6.27 (Pin_27)
- net LED_A85: now also J6.1 (Pin_1); no longer J6.25 (Pin_25)
- net LED_A86: now also J6.3 (Pin_3); no longer J6.23 (Pin_23)
- net LED_A87: now also J6.5 (Pin_5); no longer J6.21 (Pin_21)
- net LED_A88: now also J6.7 (Pin_7); no longer J6.17 (Pin_17)
- net LED_A89: now also J6.9 (Pin_9); no longer J6.15 (Pin_15)
- net LED_A9: now also J1.15 (Pin_15); no longer J1.17 (Pin_17)
- net LED_A90: now also J6.11 (Pin_11); no longer J6.13 (Pin_13)
- net LED_A91: now also J6.13 (Pin_13); no longer J6.11 (Pin_11)
- net LED_A92: now also J6.15 (Pin_15); no longer J6.9 (Pin_9)
- net LED_A93: now also J6.21 (Pin_21); no longer J6.7 (Pin_7)
- net LED_A94: now also J6.25 (Pin_25); no longer J6.5 (Pin_5)
- net LED_A95: now also J6.29 (Pin_29); no longer J6.3 (Pin_3)
- net LED_A96: now also J6.33 (Pin_33); no longer J6.1 (Pin_1)
- net LED_K1: now also J1.34 (Pin_34); no longer J1.2 (Pin_2)
- net LED_K10: now also J1.14 (Pin_14); no longer J1.22 (Pin_22)
- net LED_K11: now also J1.12 (Pin_12); no longer J1.24 (Pin_24)
- net LED_K12: now also J1.10 (Pin_10); no longer J1.26 (Pin_26)
- net LED_K13: now also J1.8 (Pin_8); no longer J1.28 (Pin_28)
- net LED_K14: now also J1.6 (Pin_6); no longer J1.30 (Pin_30)
- net LED_K15: now also J1.4 (Pin_4); no longer J1.32 (Pin_32)
- net LED_K16: now also J1.2 (Pin_2); no longer J1.34 (Pin_34)
- net LED_K17: now also J2.10 (Pin_10); no longer J2.34 (Pin_34)
- net LED_K18: now also J2.14 (Pin_14); no longer J2.32 (Pin_32)
- net LED_K19: now also J2.18 (Pin_18); no longer J2.30 (Pin_30)
- net LED_K2: now also J1.32 (Pin_32); no longer J1.4 (Pin_4)
- net LED_K20: now also J2.24 (Pin_24); no longer J2.28 (Pin_28)
- net LED_K21: now also J2.28 (Pin_28); no longer J2.26 (Pin_26)
- net LED_K22: now also J2.30 (Pin_30); no longer J2.24 (Pin_24)
- net LED_K23: now also J2.32 (Pin_32); no longer J2.22 (Pin_22)
- net LED_K24: now also J2.34 (Pin_34); no longer J2.18 (Pin_18)
- net LED_K25: now also J2.2 (Pin_2); no longer J2.16 (Pin_16)
- net LED_K26: now also J2.4 (Pin_4); no longer J2.14 (Pin_14)
- net LED_K27: now also J2.6 (Pin_6); no longer J2.12 (Pin_12)
- net LED_K28: now also J2.8 (Pin_8); no longer J2.10 (Pin_10)
- net LED_K29: now also J2.12 (Pin_12); no longer J2.8 (Pin_8)
- net LED_K3: now also J1.30 (Pin_30); no longer J1.6 (Pin_6)
- net LED_K30: now also J2.16 (Pin_16); no longer J2.6 (Pin_6)
- net LED_K31: now also J2.22 (Pin_22); no longer J2.4 (Pin_4)
- net LED_K32: now also J2.26 (Pin_26); no longer J2.2 (Pin_2)
- net LED_K33: now also J3.18 (Pin_18); no longer J3.34 (Pin_34)
- net LED_K34: now also J3.24 (Pin_24); no longer J3.32 (Pin_32)
- net LED_K35: now also J3.28 (Pin_28); no longer J3.30 (Pin_30)
- net LED_K36: now also J3.32 (Pin_32); no longer J3.28 (Pin_28)
- net LED_K37: now also J3.2 (Pin_2); no longer J3.26 (Pin_26)
- net LED_K38: now also J3.4 (Pin_4); no longer J3.24 (Pin_24)
- net LED_K39: now also J3.6 (Pin_6); no longer J3.22 (Pin_22)
- net LED_K4: now also J1.28 (Pin_28); no longer J1.8 (Pin_8)
- net LED_K40: now also J3.8 (Pin_8); no longer J3.18 (Pin_18)
- net LED_K41: now also J3.10 (Pin_10); no longer J3.16 (Pin_16)
- net LED_K42: now also J3.12 (Pin_12); no longer J3.14 (Pin_14)
- net LED_K43: now also J3.14 (Pin_14); no longer J3.12 (Pin_12)
- net LED_K44: now also J3.16 (Pin_16); no longer J3.10 (Pin_10)
- net LED_K45: now also J3.22 (Pin_22); no longer J3.8 (Pin_8)
- net LED_K46: now also J3.26 (Pin_26); no longer J3.6 (Pin_6)
- net LED_K47: now also J3.30 (Pin_30); no longer J3.4 (Pin_4)
- net LED_K48: now also J3.34 (Pin_34); no longer J3.2 (Pin_2)
- net LED_K49: now also J4.34 (Pin_34); no longer J4.2 (Pin_2)
- net LED_K5: now also J1.26 (Pin_26); no longer J1.10 (Pin_10)
- net LED_K50: now also J4.32 (Pin_32); no longer J4.4 (Pin_4)
- net LED_K51: now also J4.30 (Pin_30); no longer J4.6 (Pin_6)
- net LED_K52: now also J4.28 (Pin_28); no longer J4.8 (Pin_8)
- net LED_K53: now also J4.26 (Pin_26); no longer J4.10 (Pin_10)
- net LED_K54: now also J4.24 (Pin_24); no longer J4.12 (Pin_12)
- net LED_K55: now also J4.22 (Pin_22); no longer J4.14 (Pin_14)
- net LED_K56: now also J4.18 (Pin_18); no longer J4.16 (Pin_16)
- net LED_K57: now also J4.16 (Pin_16); no longer J4.18 (Pin_18)
- net LED_K58: now also J4.14 (Pin_14); no longer J4.22 (Pin_22)
- net LED_K59: now also J4.12 (Pin_12); no longer J4.24 (Pin_24)
- net LED_K6: now also J1.24 (Pin_24); no longer J1.12 (Pin_12)
- net LED_K60: now also J4.10 (Pin_10); no longer J4.26 (Pin_26)
- net LED_K61: now also J4.8 (Pin_8); no longer J4.28 (Pin_28)
- net LED_K62: now also J4.6 (Pin_6); no longer J4.30 (Pin_30)
- net LED_K63: now also J4.4 (Pin_4); no longer J4.32 (Pin_32)
- net LED_K64: now also J4.2 (Pin_2); no longer J4.34 (Pin_34)
- net LED_K65: now also J5.10 (Pin_10); no longer J5.34 (Pin_34)
- net LED_K66: now also J5.14 (Pin_14); no longer J5.32 (Pin_32)
- net LED_K67: now also J5.18 (Pin_18); no longer J5.30 (Pin_30)
- net LED_K68: now also J5.24 (Pin_24); no longer J5.28 (Pin_28)
- net LED_K69: now also J5.28 (Pin_28); no longer J5.26 (Pin_26)
- net LED_K7: now also J1.22 (Pin_22); no longer J1.14 (Pin_14)
- net LED_K70: now also J5.30 (Pin_30); no longer J5.24 (Pin_24)
- net LED_K71: now also J5.32 (Pin_32); no longer J5.22 (Pin_22)
- net LED_K72: now also J5.34 (Pin_34); no longer J5.18 (Pin_18)
- net LED_K73: now also J5.2 (Pin_2); no longer J5.16 (Pin_16)
- net LED_K74: now also J5.4 (Pin_4); no longer J5.14 (Pin_14)
- net LED_K75: now also J5.6 (Pin_6); no longer J5.12 (Pin_12)
- net LED_K76: now also J5.8 (Pin_8); no longer J5.10 (Pin_10)
- net LED_K77: now also J5.12 (Pin_12); no longer J5.8 (Pin_8)
- net LED_K78: now also J5.16 (Pin_16); no longer J5.6 (Pin_6)
- net LED_K79: now also J5.22 (Pin_22); no longer J5.4 (Pin_4)
- net LED_K8: now also J1.18 (Pin_18); no longer J1.16 (Pin_16)
- net LED_K80: now also J5.26 (Pin_26); no longer J5.2 (Pin_2)
- net LED_K81: now also J6.18 (Pin_18); no longer J6.34 (Pin_34)
- net LED_K82: now also J6.24 (Pin_24); no longer J6.32 (Pin_32)
- net LED_K83: now also J6.28 (Pin_28); no longer J6.30 (Pin_30)
- net LED_K84: now also J6.32 (Pin_32); no longer J6.28 (Pin_28)
- net LED_K85: now also J6.2 (Pin_2); no longer J6.26 (Pin_26)
- net LED_K86: now also J6.4 (Pin_4); no longer J6.24 (Pin_24)
- net LED_K87: now also J6.6 (Pin_6); no longer J6.22 (Pin_22)
- net LED_K88: now also J6.8 (Pin_8); no longer J6.18 (Pin_18)
- net LED_K89: now also J6.10 (Pin_10); no longer J6.16 (Pin_16)
- net LED_K9: now also J1.16 (Pin_16); no longer J1.18 (Pin_18)
- net LED_K90: now also J6.12 (Pin_12); no longer J6.14 (Pin_14)
- net LED_K91: now also J6.14 (Pin_14); no longer J6.12 (Pin_12)
- net LED_K92: now also J6.16 (Pin_16); no longer J6.10 (Pin_10)
- net LED_K93: now also J6.22 (Pin_22); no longer J6.8 (Pin_8)
- net LED_K94: now also J6.26 (Pin_26); no longer J6.6 (Pin_6)
- net LED_K95: now also J6.30 (Pin_30); no longer J6.4 (Pin_4)
- net LED_K96: now also J6.34 (Pin_34); no longer J6.2 (Pin_2)
- net NTC1: now also U1.2 (I7); no longer U1.23 (I8)
- net NTC10: now also U1.19 (I12); no longer U5.22 (I9)
- net NTC11: now also U1.7 (I2); no longer U6.23 (I8)
- net NTC12: now also U1.18 (I13); no longer U6.22 (I9)
- net NTC13: now also U1.8 (I1); no longer U1.21 (I10)
- net NTC14: now also U1.17 (I14); no longer U1.20 (I11)
- net NTC15: now also U1.9 (I0); no longer U2.21 (I10)
- net NTC16: now also U1.16 (I15); no longer U2.20 (I11)
- net NTC17: now also U2.2 (I7); no longer U3.21 (I10)
- net NTC18: now also U2.23 (I8); no longer U3.20 (I11)
- net NTC19: now also U2.3 (I6); no longer U4.21 (I10)
- net NTC2: now also U1.23 (I8); no longer U1.22 (I9)
- net NTC20: now also U2.22 (I9); no longer U4.20 (I11)
- net NTC21: now also U2.4 (I5); no longer U5.21 (I10)
- net NTC22: now also U2.21 (I10); no longer U5.20 (I11)
- net NTC23: now also U2.5 (I4); no longer U6.21 (I10)
- net NTC24: now also U2.20 (I11); no longer U6.20 (I11)
- net NTC25: now also U2.6 (I3); no longer U1.19 (I12)
- net NTC26: now also U2.19 (I12); no longer U1.18 (I13)
- net NTC27: now also U2.7 (I2); no longer U2.19 (I12)
- net NTC29: now also U2.8 (I1); no longer U3.19 (I12)
- net NTC3: now also U1.3 (I6); no longer U2.23 (I8)
- net NTC30: now also U2.17 (I14); no longer U3.18 (I13)
- net NTC31: now also U2.9 (I0); no longer U4.19 (I12)
- net NTC32: now also U2.16 (I15); no longer U4.18 (I13)
- net NTC33: now also U3.2 (I7); no longer U5.19 (I12)
- net NTC34: now also U3.23 (I8); no longer U5.18 (I13)
- net NTC35: now also U3.3 (I6); no longer U6.19 (I12)
- net NTC36: now also U3.22 (I9); no longer U6.18 (I13)
- net NTC37: now also U3.4 (I5); no longer U1.17 (I14)
- net NTC38: now also U3.21 (I10); no longer U1.16 (I15)
- net NTC39: now also U3.5 (I4); no longer U2.17 (I14)
- net NTC4: now also U1.22 (I9); no longer U2.22 (I9)
- net NTC40: now also U3.20 (I11); no longer U2.16 (I15)
- net NTC41: now also U3.6 (I3); no longer U3.17 (I14)
- net NTC42: now also U3.19 (I12); no longer U3.16 (I15)
- net NTC43: now also U3.7 (I2); no longer U4.17 (I14)
- net NTC44: now also U3.18 (I13); no longer U4.16 (I15)
- net NTC45: now also U3.8 (I1); no longer U5.17 (I14)
- net NTC46: now also U3.17 (I14); no longer U5.16 (I15)
- net NTC47: now also U3.9 (I0); no longer U6.17 (I14)
- net NTC48: now also U3.16 (I15); no longer U6.16 (I15)
- net NTC49: now also U4.2 (I7); no longer U1.2 (I7)
- net NTC5: now also U1.4 (I5); no longer U3.23 (I8)
- net NTC50: now also U4.23 (I8); no longer U1.3 (I6)
- net NTC51: now also U4.3 (I6); no longer U2.2 (I7)
- net NTC52: now also U4.22 (I9); no longer U2.3 (I6)
- net NTC53: now also U4.4 (I5); no longer U3.2 (I7)
- net NTC54: now also U4.21 (I10); no longer U3.3 (I6)
- net NTC55: now also U4.5 (I4); no longer U4.2 (I7)
- net NTC56: now also U4.20 (I11); no longer U4.3 (I6)
- net NTC57: now also U4.6 (I3); no longer U5.2 (I7)
- net NTC58: now also U4.19 (I12); no longer U5.3 (I6)
- net NTC59: now also U4.7 (I2); no longer U6.2 (I7)
- net NTC6: now also U1.21 (I10); no longer U3.22 (I9)
- net NTC60: now also U4.18 (I13); no longer U6.3 (I6)
- net NTC61: now also U4.8 (I1); no longer U1.4 (I5)
- net NTC62: now also U4.17 (I14); no longer U1.5 (I4)
- net NTC63: now also U4.9 (I0); no longer U2.4 (I5)
- net NTC64: now also U4.16 (I15); no longer U2.5 (I4)
- net NTC65: now also U5.2 (I7); no longer U3.4 (I5)
- net NTC66: now also U5.23 (I8); no longer U3.5 (I4)
- net NTC67: now also U5.3 (I6); no longer U4.4 (I5)
- net NTC68: now also U5.22 (I9); no longer U4.5 (I4)
- net NTC7: now also U1.5 (I4); no longer U4.23 (I8)
- net NTC70: now also U5.21 (I10); no longer U5.5 (I4)
- net NTC71: now also U5.5 (I4); no longer U6.4 (I5)
- net NTC72: now also U5.20 (I11); no longer U6.5 (I4)
- net NTC73: now also U5.6 (I3); no longer U1.6 (I3)
- net NTC74: now also U5.19 (I12); no longer U1.7 (I2)
- net NTC75: now also U5.7 (I2); no longer U2.6 (I3)
- net NTC76: now also U5.18 (I13); no longer U2.7 (I2)
- net NTC77: now also U5.8 (I1); no longer U3.6 (I3)
- net NTC78: now also U5.17 (I14); no longer U3.7 (I2)
- net NTC79: now also U5.9 (I0); no longer U4.6 (I3)
- net NTC8: now also U1.20 (I11); no longer U4.22 (I9)
- net NTC80: now also U5.16 (I15); no longer U4.7 (I2)
- net NTC81: now also U6.2 (I7); no longer U5.6 (I3)
- net NTC82: now also U6.23 (I8); no longer U5.7 (I2)
- net NTC83: now also U6.3 (I6); no longer U6.6 (I3)
- net NTC84: now also U6.22 (I9); no longer U6.7 (I2)
- net NTC85: now also U6.4 (I5); no longer U1.8 (I1)
- net NTC86: now also U6.21 (I10); no longer U1.9 (I0)
- net NTC87: now also U6.5 (I4); no longer U2.8 (I1)
- net NTC88: now also U6.20 (I11); no longer U2.9 (I0)
- net NTC89: now also U6.6 (I3); no longer U3.8 (I1)
- net NTC9: now also U1.6 (I3); no longer U5.23 (I8)
- net NTC90: now also U6.19 (I12); no longer U3.9 (I0)
- net NTC91: now also U6.7 (I2); no longer U4.8 (I1)
- net NTC92: now also U6.18 (I13); no longer U4.9 (I0)
- net NTC93: now also U6.8 (I1); no longer U5.8 (I1)
- net NTC94: now also U6.17 (I14); no longer U5.9 (I0)
- net NTC95: now also U6.9 (I0); no longer U6.8 (I1)
- net NTC96: now also U6.16 (I15); no longer U6.9 (I0)

Commit message: Decouple driver<->well mapping to slash ribbon crossings (461 -> 126/130)
Key insight (user): the driver serving a well need not share its index.
A ribbon SLOT (connector + IDE-safe pin-pair) is now the logical channel;
wells and drivers are assigned to slots INDEPENDENTLY, each board optimized
on its own geometry, cable wires slot-for-slot.

optimize_decoupled.py: per board, balanced min-distance grouping (0 crossings
BETWEEN ribbons) + angle order + 2-opt on the true anode/cathode-pad
ratsnest. Real crossings: LED 461->126, control ->130 (short local A/K
wires only; the board-spanning tangle is gone).

design_data.py: nets keyed by logical channel via slot2ch(); wells indexed
by grid (LED/TH/R{w}, NTC_MAP[w]), drivers by placement (U/R/L/D/C{d},
DIM{d}, PCA_MAP[d]). gen_schematics_hier instance labels remapped.
CONNECTIONS.md gains the well<->channel<->driver<->PWM firmware map.
pin_maps v10. New durable tool apply_netlist.py used for PCB re-net.
Netlists ALL MATCH both boards; cross-board ribbon consistency OK (192).

Co-Authored-By: Claude Fable 5 <noreply@anthropic.com>
Claude-Session: https://claude.ai/code/session_017oD54uh7Tvu54u9NPQNcZB
Parts:
- J1: value LED ch 1-16 -> LED ribbon 1 (16 ch)
- J2: value LED ch 17-32 -> LED ribbon 2 (16 ch)
- J3: value LED ch 33-48 -> LED ribbon 3 (16 ch)
- J4: value LED ch 49-64 -> LED ribbon 4 (16 ch)
- J5: value LED ch 65-80 -> LED ribbon 5 (16 ch)
- J6: value LED ch 81-96 -> LED ribbon 6 (16 ch)
Connections:
- net LED_A1: now also J1.1 (Pin_1); no longer J1.33 (Pin_33)
- net LED_A10: now also J1.21 (Pin_21); no longer J1.13 (Pin_13)
- net LED_A11: now also J1.23 (Pin_23); no longer J1.11 (Pin_11)
- net LED_A12: now also J1.25 (Pin_25); no longer J1.9 (Pin_9)
- net LED_A13: now also J1.27 (Pin_27); no longer J1.7 (Pin_7)
- net LED_A14: now also J1.29 (Pin_29); no longer J1.5 (Pin_5)
- net LED_A15: now also J1.31 (Pin_31); no longer J1.3 (Pin_3)
- net LED_A16: now also J1.33 (Pin_33); no longer J1.1 (Pin_1)
- net LED_A17: now also J2.1 (Pin_1); no longer J2.9 (Pin_9)
- net LED_A18: now also J2.3 (Pin_3); no longer J2.13 (Pin_13)
- net LED_A19: now also J2.5 (Pin_5); no longer J2.17 (Pin_17)
- net LED_A2: now also J1.3 (Pin_3); no longer J1.31 (Pin_31)
- net LED_A20: now also J2.7 (Pin_7); no longer J2.23 (Pin_23)
- net LED_A21: now also J2.9 (Pin_9); no longer J2.27 (Pin_27)
- net LED_A22: now also J2.11 (Pin_11); no longer J2.29 (Pin_29)
- net LED_A23: now also J2.13 (Pin_13); no longer J2.31 (Pin_31)
- net LED_A24: now also J2.15 (Pin_15); no longer J2.33 (Pin_33)
- net LED_A25: now also J2.17 (Pin_17); no longer J2.1 (Pin_1)
- net LED_A26: now also J2.21 (Pin_21); no longer J2.3 (Pin_3)
- net LED_A27: now also J2.23 (Pin_23); no longer J2.5 (Pin_5)
- net LED_A28: now also J2.25 (Pin_25); no longer J2.7 (Pin_7)
- net LED_A29: now also J2.27 (Pin_27); no longer J2.11 (Pin_11)
- net LED_A3: now also J1.5 (Pin_5); no longer J1.29 (Pin_29)
- net LED_A30: now also J2.29 (Pin_29); no longer J2.15 (Pin_15)
- net LED_A31: now also J2.31 (Pin_31); no longer J2.21 (Pin_21)
- net LED_A32: now also J2.33 (Pin_33); no longer J2.25 (Pin_25)
- net LED_A33: now also J3.1 (Pin_1); no longer J3.17 (Pin_17)
- net LED_A34: now also J3.3 (Pin_3); no longer J3.23 (Pin_23)
- net LED_A35: now also J3.5 (Pin_5); no longer J3.27 (Pin_27)
- net LED_A36: now also J3.7 (Pin_7); no longer J3.31 (Pin_31)
- net LED_A37: now also J3.9 (Pin_9); no longer J3.1 (Pin_1)
- net LED_A38: now also J3.11 (Pin_11); no longer J3.3 (Pin_3)
- net LED_A39: now also J3.13 (Pin_13); no longer J3.5 (Pin_5)
- net LED_A4: now also J1.7 (Pin_7); no longer J1.27 (Pin_27)
- net LED_A40: now also J3.15 (Pin_15); no longer J3.7 (Pin_7)
- net LED_A41: now also J3.17 (Pin_17); no longer J3.9 (Pin_9)
- net LED_A42: now also J3.21 (Pin_21); no longer J3.11 (Pin_11)
- net LED_A43: now also J3.23 (Pin_23); no longer J3.13 (Pin_13)
- net LED_A44: now also J3.25 (Pin_25); no longer J3.15 (Pin_15)
- net LED_A45: now also J3.27 (Pin_27); no longer J3.21 (Pin_21)
- net LED_A46: now also J3.29 (Pin_29); no longer J3.25 (Pin_25)
- net LED_A47: now also J3.31 (Pin_31); no longer J3.29 (Pin_29)
- net LED_A49: now also J4.1 (Pin_1); no longer J4.33 (Pin_33)
- net LED_A5: now also J1.9 (Pin_9); no longer J1.25 (Pin_25)
- net LED_A50: now also J4.3 (Pin_3); no longer J4.31 (Pin_31)
- net LED_A51: now also J4.5 (Pin_5); no longer J4.29 (Pin_29)
- net LED_A52: now also J4.7 (Pin_7); no longer J4.27 (Pin_27)
- net LED_A53: now also J4.9 (Pin_9); no longer J4.25 (Pin_25)
- net LED_A54: now also J4.11 (Pin_11); no longer J4.23 (Pin_23)
- net LED_A55: now also J4.13 (Pin_13); no longer J4.21 (Pin_21)
- net LED_A56: now also J4.15 (Pin_15); no longer J4.17 (Pin_17)
- net LED_A57: now also J4.17 (Pin_17); no longer J4.15 (Pin_15)
- net LED_A58: now also J4.21 (Pin_21); no longer J4.13 (Pin_13)
- net LED_A59: now also J4.23 (Pin_23); no longer J4.11 (Pin_11)
- net LED_A6: now also J1.11 (Pin_11); no longer J1.23 (Pin_23)
- net LED_A60: now also J4.25 (Pin_25); no longer J4.9 (Pin_9)
- net LED_A61: now also J4.27 (Pin_27); no longer J4.7 (Pin_7)
- net LED_A62: now also J4.29 (Pin_29); no longer J4.5 (Pin_5)
- net LED_A63: now also J4.31 (Pin_31); no longer J4.3 (Pin_3)
- net LED_A64: now also J4.33 (Pin_33); no longer J4.1 (Pin_1)
- net LED_A65: now also J5.1 (Pin_1); no longer J5.9 (Pin_9)
- net LED_A66: now also J5.3 (Pin_3); no longer J5.13 (Pin_13)
- net LED_A67: now also J5.5 (Pin_5); no longer J5.17 (Pin_17)
- net LED_A68: now also J5.7 (Pin_7); no longer J5.23 (Pin_23)
- net LED_A69: now also J5.9 (Pin_9); no longer J5.27 (Pin_27)
- net LED_A7: now also J1.13 (Pin_13); no longer J1.21 (Pin_21)
- net LED_A70: now also J5.11 (Pin_11); no longer J5.29 (Pin_29)
- net LED_A71: now also J5.13 (Pin_13); no longer J5.31 (Pin_31)
- net LED_A72: now also J5.15 (Pin_15); no longer J5.33 (Pin_33)
- net LED_A73: now also J5.17 (Pin_17); no longer J5.1 (Pin_1)
- net LED_A74: now also J5.21 (Pin_21); no longer J5.3 (Pin_3)
- net LED_A75: now also J5.23 (Pin_23); no longer J5.5 (Pin_5)
- net LED_A76: now also J5.25 (Pin_25); no longer J5.7 (Pin_7)
- net LED_A77: now also J5.27 (Pin_27); no longer J5.11 (Pin_11)
- net LED_A78: now also J5.29 (Pin_29); no longer J5.15 (Pin_15)
- net LED_A79: now also J5.31 (Pin_31); no longer J5.21 (Pin_21)
- net LED_A8: now also J1.15 (Pin_15); no longer J1.17 (Pin_17)
- net LED_A80: now also J5.33 (Pin_33); no longer J5.25 (Pin_25)
- net LED_A81: now also J6.1 (Pin_1); no longer J6.17 (Pin_17)
- net LED_A82: now also J6.3 (Pin_3); no longer J6.23 (Pin_23)
- net LED_A83: now also J6.5 (Pin_5); no longer J6.27 (Pin_27)
- net LED_A84: now also J6.7 (Pin_7); no longer J6.31 (Pin_31)
- net LED_A85: now also J6.9 (Pin_9); no longer J6.1 (Pin_1)
- net LED_A86: now also J6.11 (Pin_11); no longer J6.3 (Pin_3)
- net LED_A87: now also J6.13 (Pin_13); no longer J6.5 (Pin_5)
- net LED_A88: now also J6.15 (Pin_15); no longer J6.7 (Pin_7)
- net LED_A89: now also J6.17 (Pin_17); no longer J6.9 (Pin_9)
- net LED_A9: now also J1.17 (Pin_17); no longer J1.15 (Pin_15)
- net LED_A90: now also J6.21 (Pin_21); no longer J6.11 (Pin_11)
- net LED_A91: now also J6.23 (Pin_23); no longer J6.13 (Pin_13)
- net LED_A92: now also J6.25 (Pin_25); no longer J6.15 (Pin_15)
- net LED_A93: now also J6.27 (Pin_27); no longer J6.21 (Pin_21)
- net LED_A94: now also J6.29 (Pin_29); no longer J6.25 (Pin_25)
- net LED_A95: now also J6.31 (Pin_31); no longer J6.29 (Pin_29)
- net LED_K1: now also J1.2 (Pin_2); no longer J1.34 (Pin_34)
- net LED_K10: now also J1.22 (Pin_22); no longer J1.14 (Pin_14)
- net LED_K11: now also J1.24 (Pin_24); no longer J1.12 (Pin_12)
- net LED_K12: now also J1.26 (Pin_26); no longer J1.10 (Pin_10)
- net LED_K13: now also J1.28 (Pin_28); no longer J1.8 (Pin_8)
- net LED_K14: now also J1.30 (Pin_30); no longer J1.6 (Pin_6)
- net LED_K15: now also J1.32 (Pin_32); no longer J1.4 (Pin_4)
- net LED_K16: now also J1.34 (Pin_34); no longer J1.2 (Pin_2)
- net LED_K17: now also J2.2 (Pin_2); no longer J2.10 (Pin_10)
- net LED_K18: now also J2.4 (Pin_4); no longer J2.14 (Pin_14)
- net LED_K19: now also J2.6 (Pin_6); no longer J2.18 (Pin_18)
- net LED_K2: now also J1.4 (Pin_4); no longer J1.32 (Pin_32)
- net LED_K20: now also J2.8 (Pin_8); no longer J2.24 (Pin_24)
- net LED_K21: now also J2.10 (Pin_10); no longer J2.28 (Pin_28)
- net LED_K22: now also J2.12 (Pin_12); no longer J2.30 (Pin_30)
- net LED_K23: now also J2.14 (Pin_14); no longer J2.32 (Pin_32)
- net LED_K24: now also J2.16 (Pin_16); no longer J2.34 (Pin_34)
- net LED_K25: now also J2.18 (Pin_18); no longer J2.2 (Pin_2)
- net LED_K26: now also J2.22 (Pin_22); no longer J2.4 (Pin_4)
- net LED_K27: now also J2.24 (Pin_24); no longer J2.6 (Pin_6)
- net LED_K28: now also J2.26 (Pin_26); no longer J2.8 (Pin_8)
- net LED_K29: now also J2.28 (Pin_28); no longer J2.12 (Pin_12)
- net LED_K3: now also J1.6 (Pin_6); no longer J1.30 (Pin_30)
- net LED_K30: now also J2.30 (Pin_30); no longer J2.16 (Pin_16)
- net LED_K31: now also J2.32 (Pin_32); no longer J2.22 (Pin_22)
- net LED_K32: now also J2.34 (Pin_34); no longer J2.26 (Pin_26)
- net LED_K33: now also J3.2 (Pin_2); no longer J3.18 (Pin_18)
- net LED_K34: now also J3.4 (Pin_4); no longer J3.24 (Pin_24)
- net LED_K35: now also J3.6 (Pin_6); no longer J3.28 (Pin_28)
- net LED_K36: now also J3.8 (Pin_8); no longer J3.32 (Pin_32)
- net LED_K37: now also J3.10 (Pin_10); no longer J3.2 (Pin_2)
- net LED_K38: now also J3.12 (Pin_12); no longer J3.4 (Pin_4)
- net LED_K39: now also J3.14 (Pin_14); no longer J3.6 (Pin_6)
- net LED_K4: now also J1.8 (Pin_8); no longer J1.28 (Pin_28)
- net LED_K40: now also J3.16 (Pin_16); no longer J3.8 (Pin_8)
- net LED_K41: now also J3.18 (Pin_18); no longer J3.10 (Pin_10)
- net LED_K42: now also J3.22 (Pin_22); no longer J3.12 (Pin_12)
- net LED_K43: now also J3.24 (Pin_24); no longer J3.14 (Pin_14)
- net LED_K44: now also J3.26 (Pin_26); no longer J3.16 (Pin_16)
- net LED_K45: now also J3.28 (Pin_28); no longer J3.22 (Pin_22)
- net LED_K46: now also J3.30 (Pin_30); no longer J3.26 (Pin_26)
- net LED_K47: now also J3.32 (Pin_32); no longer J3.30 (Pin_30)
- net LED_K49: now also J4.2 (Pin_2); no longer J4.34 (Pin_34)
- net LED_K5: now also J1.10 (Pin_10); no longer J1.26 (Pin_26)
- net LED_K50: now also J4.4 (Pin_4); no longer J4.32 (Pin_32)
- net LED_K51: now also J4.6 (Pin_6); no longer J4.30 (Pin_30)
- net LED_K52: now also J4.8 (Pin_8); no longer J4.28 (Pin_28)
- net LED_K53: now also J4.10 (Pin_10); no longer J4.26 (Pin_26)
- net LED_K54: now also J4.12 (Pin_12); no longer J4.24 (Pin_24)
- net LED_K55: now also J4.14 (Pin_14); no longer J4.22 (Pin_22)
- net LED_K56: now also J4.16 (Pin_16); no longer J4.18 (Pin_18)
- net LED_K57: now also J4.18 (Pin_18); no longer J4.16 (Pin_16)
- net LED_K58: now also J4.22 (Pin_22); no longer J4.14 (Pin_14)
- net LED_K59: now also J4.24 (Pin_24); no longer J4.12 (Pin_12)
- net LED_K6: now also J1.12 (Pin_12); no longer J1.24 (Pin_24)
- net LED_K60: now also J4.26 (Pin_26); no longer J4.10 (Pin_10)
- net LED_K61: now also J4.28 (Pin_28); no longer J4.8 (Pin_8)
- net LED_K62: now also J4.30 (Pin_30); no longer J4.6 (Pin_6)
- net LED_K63: now also J4.32 (Pin_32); no longer J4.4 (Pin_4)
- net LED_K64: now also J4.34 (Pin_34); no longer J4.2 (Pin_2)
- net LED_K65: now also J5.2 (Pin_2); no longer J5.10 (Pin_10)
- net LED_K66: now also J5.4 (Pin_4); no longer J5.14 (Pin_14)
- net LED_K67: now also J5.6 (Pin_6); no longer J5.18 (Pin_18)
- net LED_K68: now also J5.8 (Pin_8); no longer J5.24 (Pin_24)
- net LED_K69: now also J5.10 (Pin_10); no longer J5.28 (Pin_28)
- net LED_K7: now also J1.14 (Pin_14); no longer J1.22 (Pin_22)
- net LED_K70: now also J5.12 (Pin_12); no longer J5.30 (Pin_30)
- net LED_K71: now also J5.14 (Pin_14); no longer J5.32 (Pin_32)
- net LED_K72: now also J5.16 (Pin_16); no longer J5.34 (Pin_34)
- net LED_K73: now also J5.18 (Pin_18); no longer J5.2 (Pin_2)
- net LED_K74: now also J5.22 (Pin_22); no longer J5.4 (Pin_4)
- net LED_K75: now also J5.24 (Pin_24); no longer J5.6 (Pin_6)
- net LED_K76: now also J5.26 (Pin_26); no longer J5.8 (Pin_8)
- net LED_K77: now also J5.28 (Pin_28); no longer J5.12 (Pin_12)
- net LED_K78: now also J5.30 (Pin_30); no longer J5.16 (Pin_16)
- net LED_K79: now also J5.32 (Pin_32); no longer J5.22 (Pin_22)
- net LED_K8: now also J1.16 (Pin_16); no longer J1.18 (Pin_18)
- net LED_K80: now also J5.34 (Pin_34); no longer J5.26 (Pin_26)
- net LED_K81: now also J6.2 (Pin_2); no longer J6.18 (Pin_18)
- net LED_K82: now also J6.4 (Pin_4); no longer J6.24 (Pin_24)
- net LED_K83: now also J6.6 (Pin_6); no longer J6.28 (Pin_28)
- net LED_K84: now also J6.8 (Pin_8); no longer J6.32 (Pin_32)
- net LED_K85: now also J6.10 (Pin_10); no longer J6.2 (Pin_2)
- net LED_K86: now also J6.12 (Pin_12); no longer J6.4 (Pin_4)
- net LED_K87: now also J6.14 (Pin_14); no longer J6.6 (Pin_6)
- net LED_K88: now also J6.16 (Pin_16); no longer J6.8 (Pin_8)
- net LED_K89: now also J6.18 (Pin_18); no longer J6.10 (Pin_10)
- net LED_K9: now also J1.18 (Pin_18); no longer J1.16 (Pin_16)
- net LED_K90: now also J6.22 (Pin_22); no longer J6.12 (Pin_12)
- net LED_K91: now also J6.24 (Pin_24); no longer J6.14 (Pin_14)
- net LED_K92: now also J6.26 (Pin_26); no longer J6.16 (Pin_16)
- net LED_K93: now also J6.28 (Pin_28); no longer J6.22 (Pin_22)
- net LED_K94: now also J6.30 (Pin_30); no longer J6.26 (Pin_26)
- net LED_K95: now also J6.32 (Pin_32); no longer J6.30 (Pin_30)
Other:
- note added: "96 WELLS (by grid position) - see well.kicad_sch"
- note added: "NTC MUXES U1-U6 (each takes its 16 nearest wells)"
- note removed: "96 WELLS (CH01..CH96) - see well.kicad_sch"
- note removed: "NTC MUXES U1-U6 (ch 1-16 / 17-32 / 33-48 / 49-64 / 65-80 / 81-96)"
