File: control-board/control-board.kicad_pcb (KiCad board)
At the start: 2 copper layers, 218 x 137.7 mm, 639 parts, among them J1 LED ch 1-24, J10 ESP32 left (3V3 row), J11 ESP32 right (GND row), J2 LED ch 25-48, J3 LED ch 49-72, J4 LED ch 73-96, J5 logic/analog, J6 24V IN, J7 24V IN (5.5/2.5), J8 FAN 24V, Q1 AO3400A, SW1 MODE, SW2 UP, SW3 DOWN, U1 PT4115, U10 PT4115, U101 PCA9685PW (0x40), U102 PCA9685PW (0x41), U103 PCA9685PW (0x42), U104 PCA9685PW (0x43), U105 PCA9685PW (0x44), U106 PCA9685PW (0x45), U11 PT4115, U110 XL1509-5.0E1, U111 ADS1115IDGS (DNP), U12 PT4115, U13 PT4115, U14 PT4115, U15 PT4115, U16 PT4115, U17 PT4115, U18 PT4115, U19 PT4115, U2 PT4115, U20 PT4115, U21 PT4115, U22 PT4115, U23 PT4115, U24 PT4115, U25 PT4115, U26 PT4115, U27 PT4115, U28 PT4115, U29 PT4115, U3 PT4115, U30 PT4115, U31 PT4115, U32 PT4115, U33 PT4115, U34 PT4115, U35 PT4115, U36 PT4115, U37 PT4115, U38 PT4115, U39 PT4115, U4 PT4115, U40 PT4115, U41 PT4115, U42 PT4115, U43 PT4115, U44 PT4115, U45 PT4115, U46 PT4115, U47 PT4115, U48 PT4115, U49 PT4115, U5 PT4115, U50 PT4115, U51 PT4115, U52 PT4115, U53 PT4115, U54 PT4115, U55 PT4115, U56 PT4115, U57 PT4115, U58 PT4115, U59 PT4115, U6 PT4115, U60 PT4115, U61 PT4115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

Commit message: Control board refinement: headers rotated 180 (ribbon-fold correct, crossing-free fan-out), PCA stacks aligned to channel bands, right column shifted clear of connector shroud lips; placement DRC clean
Co-Authored-By: Claude Fable 5 <noreply@anthropic.com>
Claude-Session: https://claude.ai/code/session_017oD54uh7Tvu54u9NPQNcZB
Parts:
- moved J1 66.0 mm to (182.0, 26.5), turned to -90 degrees
- moved J2 66.0 mm to (96.0, 26.5), turned to -90 degrees
- moved J3 66.0 mm to (103.2, 136.8), turned to -90 degrees
- moved J4 66.0 mm to (176.0, 136.8), turned to -90 degrees
- moved C123 13.0 mm to (32.0, 82.0)
- moved U103 13.0 mm to (24.0, 82.0)
- moved C124 12.5 mm to (195.5, 100.0)
- moved U104 12.5 mm to (187.5, 100.0)
- moved C125 9.19 mm to (195.5, 115.5)
- moved U105 9.19 mm to (187.5, 115.5)
- moved C122 7.00 mm to (32.0, 64.0)
- moved U102 7.00 mm to (24.0, 64.0)
- moved U111 6.71 mm to (203.0, 106.0)
- moved C126 6.52 mm to (195.5, 130.5)
- moved U106 6.52 mm to (187.5, 130.5)
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
Commit message: Control board fill/coupling pass: field rows spread to 12.25mm pitch, bulk caps split input/load side, XL group tight column, I2C parts at ESP32 SDA/SCL end, TP grid fills right-middle, fan header on edge
Co-Authored-By: Claude Fable 5 <noreply@anthropic.com>
Claude-Session: https://claude.ai/code/session_017oD54uh7Tvu54u9NPQNcZB
Parts:
- moved C103 204.7 mm to (197.0, 109.0)
- moved C104 203.7 mm to (206.0, 109.0)
- moved C102 97.1 mm to (7.00, 114.0)
- moved C101 85.5 mm to (7.00, 103.0)
- moved TP4 50.3 mm to (196.0, 66.0)
- moved TP7 49.5 mm to (196.0, 71.0)
- moved TP8 49.4 mm to (201.5, 71.0)
- moved TP10 49.3 mm to (196.0, 76.0)
- moved TP11 49.2 mm to (201.5, 76.0)
- moved TP12 49.2 mm to (207.0, 76.0)
- moved TP9 45.4 mm to (207.0, 71.0)
- moved TP6 43.9 mm to (207.0, 66.0)
- moved TP5 43.8 mm to (201.5, 66.0)
- moved TP3 43.0 mm to (207.0, 61.0)
- moved TP2 43.0 mm to (201.5, 61.0)
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