File: control-board/control-board.kicad_pcb (KiCad board)
At the start: 4 copper layers, 218 x 137.7 mm, 639 parts, among them J1 LED ch 1-24, J10 ESP32 left (3V3 row), J11 ESP32 right (GND row), J2 LED ch 25-48, J3 LED ch 49-72, J4 LED ch 73-96, J5 logic/analog, J6 24V IN, J7 24V IN (5.5/2.5), J8 FAN 24V, Q1 AO3400A, SW1 MODE, SW2 UP, SW3 DOWN, U1 PT4115, U10 PT4115, U101 PCA9685PW (0x40), U102 PCA9685PW (0x41), U103 PCA9685PW (0x42), U104 PCA9685PW (0x43), U105 PCA9685PW (0x44), U106 PCA9685PW (0x45), U11 PT4115, U110 XL1509-5.0E1, U111 ADS1115IDGS (DNP), U12 PT4115, U13 PT4115, U14 PT4115, U15 PT4115, U16 PT4115, U17 PT4115, U18 PT4115, U19 PT4115, U2 PT4115, U20 PT4115, U21 PT4115, U22 PT4115, U23 PT4115, U24 PT4115, U25 PT4115, U26 PT4115, U27 PT4115, U28 PT4115, U29 PT4115, U3 PT4115, U30 PT4115, U31 PT4115, U32 PT4115, U33 PT4115, U34 PT4115, U35 PT4115, U36 PT4115, U37 PT4115, U38 PT4115, U39 PT4115, U4 PT4115, U40 PT4115, U41 PT4115, U42 PT4115, U43 PT4115, U44 PT4115, U45 PT4115, U46 PT4115, U47 PT4115, U48 PT4115, U49 PT4115, U5 PT4115, U50 PT4115, U51 PT4115, U52 PT4115, U53 PT4115, U54 PT4115, U55 PT4115, U56 PT4115, U57 PT4115, U58 PT4115, U59 PT4115, U6 PT4115, U60 PT4115, U61 PT4115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

Commit message: Swap to 6x 40-pin IDC ribbons (IDE-safe pinout), clear routing for rearrange
- J1-J6 both boards: 16 channels each = one PCA9685 bank per cable;
  pairs on pins 1-18/21-34, pin 20 NC (IDE key), GND 19+35-40
- Logic ribbon renamed J9; control screw terminal now J12
- Schematics regenerated (netlists verified 300+412), CONNECTIONS
  updated; connectors placed at nominal spots for user rearrangement
- All routing cleared except LED thermal via farms per user request
- New vault note: What Every Part Does

Co-Authored-By: Claude Fable 5 <noreply@anthropic.com>
Claude-Session: https://claude.ai/code/session_017oD54uh7Tvu54u9NPQNcZB
Parts:
- added J5: 40-pin ribbon, Connector_IDC:IDC-Header_2x20_P2.54mm_Vertical, F.Cu at (96.0, 136.8)
- added J6: 40-pin ribbon, Connector_IDC:IDC-Header_2x20_P2.54mm_Vertical, F.Cu at (156.0, 136.8)
- J1: value LED ch 1-24 -> 40-pin ribbon; footprint Connector_IDC:IDC-Header_2x25_P2.54mm_Vertical -> Connector_IDC:IDC-Header_2x20_P2.54mm_Vertical
- J2: value LED ch 25-48 -> 40-pin ribbon; footprint Connector_IDC:IDC-Header_2x25_P2.54mm_Vertical -> Connector_IDC:IDC-Header_2x20_P2.54mm_Vertical
- J3: value LED ch 49-72 -> 40-pin ribbon; footprint Connector_IDC:IDC-Header_2x25_P2.54mm_Vertical -> Connector_IDC:IDC-Header_2x20_P2.54mm_Vertical
- J4: value LED ch 73-96 -> 40-pin ribbon; footprint Connector_IDC:IDC-Header_2x25_P2.54mm_Vertical -> Connector_IDC:IDC-Header_2x20_P2.54mm_Vertical
- moved J1 146.0 mm to (36.0, 26.5)
- moved J4 140.0 mm to (36.0, 136.8)
- moved J3 122.3 mm to (156.0, 26.5)
- renumbered J6 to J12, J5 to J9
Connections:
- J1 pad 10: /LED_K2 -> /LED_K5
- J1 pad 11: /LED_A14 -> /LED_A6
- J1 pad 12: /LED_K14 -> /LED_K6
- J1 pad 13: /LED_A26 -> /LED_A7
- J1 pad 14: /LED_K26 -> /LED_K7
- J1 pad 15: /LED_A38 -> /LED_A8
- J1 pad 16: /LED_K38 -> /LED_K8
- J1 pad 17: /LED_A3 -> /LED_A9
- J1 pad 18: /LED_K3 -> /LED_K9
- J1 pad 19: /LED_A15 -> GND
- J1 pad 20: /LED_K15 -> unconnected-(J1-Pin_20-Pad20)
- J1 pad 21: /LED_A27 -> /LED_A10
- J1 pad 22: /LED_K27 -> /LED_K10
- J1 pad 23: /LED_A39 -> /LED_A11
- J1 pad 24: /LED_K39 -> /LED_K11
- J1 pad 25: /LED_A4 -> /LED_A12
- J1 pad 26: /LED_K4 -> /LED_K12
- J1 pad 27: /LED_A16 -> /LED_A13
- J1 pad 28: /LED_K16 -> /LED_K13
- J1 pad 29: /LED_A28 -> /LED_A14
- J1 pad 3: /LED_A13 -> /LED_A2
- J1 pad 30: /LED_K28 -> /LED_K14
- J1 pad 31: /LED_A40 -> /LED_A15
- J1 pad 32: /LED_K40 -> /LED_K15
- J1 pad 33: /LED_A5 -> /LED_A16
- J1 pad 34: /LED_K5 -> /LED_K16
- J1 pad 35: /LED_A17 -> GND
- J1 pad 36: /LED_K17 -> GND
- J1 pad 37: /LED_A29 -> GND
- J1 pad 38: /LED_K29 -> GND
- J1 pad 39: /LED_A41 -> GND
- J1 pad 4: /LED_K13 -> /LED_K2
- J1 pad 40: /LED_K41 -> GND
- J1 pad 5: /LED_A25 -> /LED_A3
- J1 pad 6: /LED_K25 -> /LED_K3
- J1 pad 7: /LED_A37 -> /LED_A4
- J1 pad 8: /LED_K37 -> /LED_K4
- J1 pad 9: /LED_A2 -> /LED_A5
- J2 pad 1: /LED_A7 -> /LED_A17
- J2 pad 10: /LED_K8 -> /LED_K21
- J2 pad 11: /LED_A20 -> /LED_A22
- J2 pad 12: /LED_K20 -> /LED_K22
- J2 pad 13: /LED_A32 -> /LED_A23
- J2 pad 14: /LED_K32 -> /LED_K23
- J2 pad 15: /LED_A44 -> /LED_A24
- J2 pad 16: /LED_K44 -> /LED_K24
- J2 pad 17: /LED_A9 -> /LED_A25
- J2 pad 18: /LED_K9 -> /LED_K25
- J2 pad 19: /LED_A21 -> GND
- J2 pad 2: /LED_K7 -> /LED_K17
- J2 pad 20: /LED_K21 -> unconnected-(J2-Pin_20-Pad20)
- J2 pad 21: /LED_A33 -> /LED_A26
- J2 pad 22: /LED_K33 -> /LED_K26
- J2 pad 23: /LED_A45 -> /LED_A27
- J2 pad 24: /LED_K45 -> /LED_K27
- J2 pad 25: /LED_A10 -> /LED_A28
- J2 pad 26: /LED_K10 -> /LED_K28
- J2 pad 27: /LED_A22 -> /LED_A29
- J2 pad 28: /LED_K22 -> /LED_K29
- J2 pad 29: /LED_A34 -> /LED_A30
- J2 pad 3: /LED_A19 -> /LED_A18
- J2 pad 30: /LED_K34 -> /LED_K30
- J2 pad 31: /LED_A46 -> /LED_A31
- J2 pad 32: /LED_K46 -> /LED_K31
- J2 pad 33: /LED_A11 -> /LED_A32
- J2 pad 34: /LED_K11 -> /LED_K32
- J2 pad 35: /LED_A23 -> GND
- J2 pad 36: /LED_K23 -> GND
- J2 pad 37: /LED_A35 -> GND
- J2 pad 38: /LED_K35 -> GND
- J2 pad 39: /LED_A47 -> GND
- J2 pad 4: /LED_K19 -> /LED_K18
- J2 pad 40: /LED_K47 -> GND
- J2 pad 5: /LED_A31 -> /LED_A19
- J2 pad 6: /LED_K31 -> /LED_K19
- J2 pad 7: /LED_A43 -> /LED_A20
- J2 pad 8: /LED_K43 -> /LED_K20
- J2 pad 9: /LED_A8 -> /LED_A21
- J3 pad 1: /LED_A55 -> /LED_A33
- J3 pad 10: /LED_K56 -> /LED_K37
- J3 pad 11: /LED_A68 -> /LED_A38
- J3 pad 12: /LED_K68 -> /LED_K38
- J3 pad 13: /LED_A80 -> /LED_A39
- J3 pad 14: /LED_K80 -> /LED_K39
- J3 pad 15: /LED_A92 -> /LED_A40
- J3 pad 16: /LED_K92 -> /LED_K40
- J3 pad 17: /LED_A57 -> /LED_A41
- J3 pad 18: /LED_K57 -> /LED_K41
- J3 pad 19: /LED_A69 -> GND
- J3 pad 2: /LED_K55 -> /LED_K33
- J3 pad 20: /LED_K69 -> unconnected-(J3-Pin_20-Pad20)
- J3 pad 21: /LED_A81 -> /LED_A42
- J3 pad 22: /LED_K81 -> /LED_K42
- J3 pad 23: /LED_A93 -> /LED_A43
- J3 pad 24: /LED_K93 -> /LED_K43
- J3 pad 25: /LED_A58 -> /LED_A44
- J3 pad 26: /LED_K58 -> /LED_K44
- J3 pad 27: /LED_A70 -> /LED_A45
- J3 pad 28: /LED_K70 -> /LED_K45
- J3 pad 29: /LED_A82 -> /LED_A46
- J3 pad 3: /LED_A67 -> /LED_A34
- J3 pad 30: /LED_K82 -> /LED_K46
- J3 pad 31: /LED_A94 -> /LED_A47
- J3 pad 32: /LED_K94 -> /LED_K47
- J3 pad 33: /LED_A59 -> /LED_A48
- J3 pad 34: /LED_K59 -> /LED_K48
- J3 pad 35: /LED_A71 -> GND
- J3 pad 36: /LED_K71 -> GND
- J3 pad 37: /LED_A83 -> GND
- J3 pad 38: /LED_K83 -> GND
- J3 pad 39: /LED_A95 -> GND
- J3 pad 4: /LED_K67 -> /LED_K34
- J3 pad 40: /LED_K95 -> GND
- J3 pad 5: /LED_A79 -> /LED_A35
- J3 pad 6: /LED_K79 -> /LED_K35
- J3 pad 7: /LED_A91 -> /LED_A36
- J3 pad 8: /LED_K91 -> /LED_K36
- J3 pad 9: /LED_A56 -> /LED_A37
- J4 pad 10: /LED_K50 -> /LED_K53
- J4 pad 11: /LED_A62 -> /LED_A54
- J4 pad 12: /LED_K62 -> /LED_K54
- J4 pad 13: /LED_A74 -> /LED_A55
- J4 pad 14: /LED_K74 -> /LED_K55
- J4 pad 15: /LED_A86 -> /LED_A56
- J4 pad 16: /LED_K86 -> /LED_K56
- J4 pad 17: /LED_A51 -> /LED_A57
- J4 pad 18: /LED_K51 -> /LED_K57
- J4 pad 19: /LED_A63 -> GND
- J4 pad 20: /LED_K63 -> unconnected-(J4-Pin_20-Pad20)
- J4 pad 21: /LED_A75 -> /LED_A58
- J4 pad 22: /LED_K75 -> /LED_K58
- J4 pad 23: /LED_A87 -> /LED_A59
- J4 pad 24: /LED_K87 -> /LED_K59
- J4 pad 25: /LED_A52 -> /LED_A60
- J4 pad 26: /LED_K52 -> /LED_K60
- J4 pad 27: /LED_A64 -> /LED_A61
- J4 pad 28: /LED_K64 -> /LED_K61
- J4 pad 29: /LED_A76 -> /LED_A62
- J4 pad 3: /LED_A61 -> /LED_A50
- J4 pad 30: /LED_K76 -> /LED_K62
- J4 pad 31: /LED_A88 -> /LED_A63
- J4 pad 32: /LED_K88 -> /LED_K63
- J4 pad 33: /LED_A53 -> /LED_A64
- J4 pad 34: /LED_K53 -> /LED_K64
- J4 pad 35: /LED_A65 -> GND
- J4 pad 36: /LED_K65 -> GND
- J4 pad 37: /LED_A77 -> GND
- J4 pad 38: /LED_K77 -> GND
- J4 pad 39: /LED_A89 -> GND
- J4 pad 4: /LED_K61 -> /LED_K50
- J4 pad 40: /LED_K89 -> GND
- J4 pad 5: /LED_A73 -> /LED_A51
- J4 pad 6: /LED_K73 -> /LED_K51
- J4 pad 7: /LED_A85 -> /LED_A52
- J4 pad 8: /LED_K85 -> /LED_K52
- J4 pad 9: /LED_A50 -> /LED_A53
Routing:
- net GND: track 650.2 -> 0.00 mm, vias 464 -> 0
- net +24V: track 548.8 -> 0.00 mm, vias 392 -> 0

Commit message: Driver-board pinout optimization from user's rearranged placement
- CONN_MAP: per-ribbon pair order jointly optimized against BOTH
  boards' geometry (pads projected on connector axes, combined rank)
- PCA_MAP: each PCA9685's 16 outputs assigned to its bank's DIM
  lines by physical order (crossing-free fan-out)
- design_data table-driven; schematics regenerated; netlists verify
  (300+412); pads re-netted on both boards; CONNECTIONS updated

Co-Authored-By: Claude Fable 5 <noreply@anthropic.com>
Claude-Session: https://claude.ai/code/session_017oD54uh7Tvu54u9NPQNcZB
Parts:
- moved H2 252.5 mm to (279.4, 124.2)
- moved H1 246.4 mm to (272.8, 42.5)
- moved J9 211.2 mm to (222.3, 114.9)
- moved C110 203.1 mm to (218.3, 28.8), turned to 0 degrees
- moved J7 199.7 mm to (209.7, 127.5)
- moved J12 182.4 mm to (192.3, 137.1), turned to 0 degrees
- moved L101 182.4 mm to (202.2, 124.0), turned to 90 degrees
- moved U110 176.9 mm to (194.8, 124.6), turned to 180 degrees
- moved D101 173.2 mm to (193.2, 129.7), turned to 180 degrees
- moved C111 169.0 mm to (197.4, 117.0)
- moved TP4 167.3 mm to (46.5, 141.1)
- moved U102 167.0 mm to (184.9, 108.8), turned to 0 degrees
- moved U103 166.8 mm to (184.9, 126.2), turned to 0 degrees
- moved U101 161.2 mm to (184.9, 56.5), turned to 0 degrees
- moved C122 160.0 mm to (187.3, 102.8), turned to 180 degrees
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Connections:
- J1 pad 11: /LED_A6 -> /LED_A13
- J1 pad 12: /LED_K6 -> /LED_K13
- J1 pad 13: /LED_A7 -> /LED_A6
- J1 pad 14: /LED_K7 -> /LED_K6
- J1 pad 15: /LED_A8 -> /LED_A7
- J1 pad 16: /LED_K8 -> /LED_K7
- J1 pad 17: /LED_A9 -> /LED_A14
- J1 pad 18: /LED_K9 -> /LED_K14
- J1 pad 21: /LED_A10 -> /LED_A8
- J1 pad 22: /LED_K10 -> /LED_K8
- J1 pad 23: /LED_A11 -> /LED_A15
- J1 pad 24: /LED_K11 -> /LED_K15
- J1 pad 25: /LED_A12 -> /LED_A9
- J1 pad 26: /LED_K12 -> /LED_K9
- J1 pad 27: /LED_A13 -> /LED_A10
- J1 pad 28: /LED_K13 -> /LED_K10
- J1 pad 29: /LED_A14 -> /LED_A16
- J1 pad 30: /LED_K14 -> /LED_K16
- J1 pad 31: /LED_A15 -> /LED_A11
- J1 pad 32: /LED_K15 -> /LED_K11
- J1 pad 33: /LED_A16 -> /LED_A12
- J1 pad 34: /LED_K16 -> /LED_K12
- J2 pad 1: /LED_A17 -> /LED_A32
- J2 pad 10: /LED_K21 -> /LED_K28
- J2 pad 11: /LED_A22 -> /LED_A27
- J2 pad 12: /LED_K22 -> /LED_K27
- J2 pad 13: /LED_A23 -> /LED_A26
- J2 pad 14: /LED_K23 -> /LED_K26
- J2 pad 15: /LED_A24 -> /LED_A25
- J2 pad 16: /LED_K24 -> /LED_K25
- J2 pad 17: /LED_A25 -> /LED_A24
- J2 pad 18: /LED_K25 -> /LED_K24
- J2 pad 2: /LED_K17 -> /LED_K32
- J2 pad 21: /LED_A26 -> /LED_A23
- J2 pad 22: /LED_K26 -> /LED_K23
- J2 pad 23: /LED_A27 -> /LED_A22
- J2 pad 24: /LED_K27 -> /LED_K22
- J2 pad 25: /LED_A28 -> /LED_A21
- J2 pad 26: /LED_K28 -> /LED_K21
- J2 pad 27: /LED_A29 -> /LED_A20
- J2 pad 28: /LED_K29 -> /LED_K20
- J2 pad 29: /LED_A30 -> /LED_A19
- J2 pad 3: /LED_A18 -> /LED_A31
- J2 pad 30: /LED_K30 -> /LED_K19
- J2 pad 31: /LED_A31 -> /LED_A18
- J2 pad 32: /LED_K31 -> /LED_K18
- J2 pad 33: /LED_A32 -> /LED_A17
- J2 pad 34: /LED_K32 -> /LED_K17
- J2 pad 4: /LED_K18 -> /LED_K31
- J2 pad 5: /LED_A19 -> /LED_A30
- J2 pad 6: /LED_K19 -> /LED_K30
- J2 pad 7: /LED_A20 -> /LED_A29
- J2 pad 8: /LED_K20 -> /LED_K29
- J2 pad 9: /LED_A21 -> /LED_A28
- J3 pad 1: /LED_A33 -> /LED_A48
- J3 pad 10: /LED_K37 -> /LED_K44
- J3 pad 11: /LED_A38 -> /LED_A43
- J3 pad 12: /LED_K38 -> /LED_K43
- J3 pad 13: /LED_A39 -> /LED_A42
- J3 pad 14: /LED_K39 -> /LED_K42
- J3 pad 15: /LED_A40 -> /LED_A41
- J3 pad 16: /LED_K40 -> /LED_K41
- J3 pad 17: /LED_A41 -> /LED_A40
- J3 pad 18: /LED_K41 -> /LED_K40
- J3 pad 2: /LED_K33 -> /LED_K48
- J3 pad 21: /LED_A42 -> /LED_A39
- J3 pad 22: /LED_K42 -> /LED_K39
- J3 pad 23: /LED_A43 -> /LED_A38
- J3 pad 24: /LED_K43 -> /LED_K38
- J3 pad 25: /LED_A44 -> /LED_A37
- J3 pad 26: /LED_K44 -> /LED_K37
- J3 pad 27: /LED_A45 -> /LED_A36
- J3 pad 28: /LED_K45 -> /LED_K36
- J3 pad 29: /LED_A46 -> /LED_A35
- J3 pad 3: /LED_A34 -> /LED_A47
- J3 pad 30: /LED_K46 -> /LED_K35
- J3 pad 31: /LED_A47 -> /LED_A34
- J3 pad 32: /LED_K47 -> /LED_K34
- J3 pad 33: /LED_A48 -> /LED_A33
- J3 pad 34: /LED_K48 -> /LED_K33
- J3 pad 4: /LED_K34 -> /LED_K47
- J3 pad 5: /LED_A35 -> /LED_A46
- J3 pad 6: /LED_K35 -> /LED_K46
- J3 pad 7: /LED_A36 -> /LED_A45
- J3 pad 8: /LED_K36 -> /LED_K45
- J3 pad 9: /LED_A37 -> /LED_A44
- J4 pad 11: /LED_A54 -> /LED_A61
- J4 pad 12: /LED_K54 -> /LED_K61
- J4 pad 13: /LED_A55 -> /LED_A54
- J4 pad 14: /LED_K55 -> /LED_K54
- J4 pad 15: /LED_A56 -> /LED_A55
- J4 pad 16: /LED_K56 -> /LED_K55
- J4 pad 17: /LED_A57 -> /LED_A62
- J4 pad 18: /LED_K57 -> /LED_K62
- J4 pad 21: /LED_A58 -> /LED_A56
- J4 pad 22: /LED_K58 -> /LED_K56
- J4 pad 23: /LED_A59 -> /LED_A63
- J4 pad 24: /LED_K59 -> /LED_K63
- J4 pad 25: /LED_A60 -> /LED_A57
- J4 pad 26: /LED_K60 -> /LED_K57
- J4 pad 27: /LED_A61 -> /LED_A58
- J4 pad 28: /LED_K61 -> /LED_K58
- J4 pad 29: /LED_A62 -> /LED_A64
- J4 pad 30: /LED_K62 -> /LED_K64
- J4 pad 31: /LED_A63 -> /LED_A59
- J4 pad 32: /LED_K63 -> /LED_K59
- J4 pad 33: /LED_A64 -> /LED_A60
- J4 pad 34: /LED_K64 -> /LED_K60
- J5 pad 1: /LED_A65 -> /LED_A80
- J5 pad 10: /LED_K69 -> /LED_K76
- J5 pad 11: /LED_A70 -> /LED_A75
- J5 pad 12: /LED_K70 -> /LED_K75
- J5 pad 13: /LED_A71 -> /LED_A74
- J5 pad 14: /LED_K71 -> /LED_K74
- J5 pad 15: /LED_A72 -> /LED_A73
- J5 pad 16: /LED_K72 -> /LED_K73
- J5 pad 17: /LED_A73 -> /LED_A72
- J5 pad 18: /LED_K73 -> /LED_K72
- J5 pad 2: /LED_K65 -> /LED_K80
- J5 pad 21: /LED_A74 -> /LED_A71
- J5 pad 22: /LED_K74 -> /LED_K71
- J5 pad 23: /LED_A75 -> /LED_A70
- J5 pad 24: /LED_K75 -> /LED_K70
- J5 pad 25: /LED_A76 -> /LED_A69
- J5 pad 26: /LED_K76 -> /LED_K69
- J5 pad 27: /LED_A77 -> /LED_A68
- J5 pad 28: /LED_K77 -> /LED_K68
- J5 pad 29: /LED_A78 -> /LED_A67
- J5 pad 3: /LED_A66 -> /LED_A79
- J5 pad 30: /LED_K78 -> /LED_K67
- J5 pad 31: /LED_A79 -> /LED_A66
- J5 pad 32: /LED_K79 -> /LED_K66
- J5 pad 33: /LED_A80 -> /LED_A65
- J5 pad 34: /LED_K80 -> /LED_K65
- J5 pad 4: /LED_K66 -> /LED_K79
- J5 pad 5: /LED_A67 -> /LED_A78
- J5 pad 6: /LED_K67 -> /LED_K78
- J5 pad 7: /LED_A68 -> /LED_A77
- J5 pad 8: /LED_K68 -> /LED_K77
- J5 pad 9: /LED_A69 -> /LED_A76
- J6 pad 1: /LED_A81 -> /LED_A96
- J6 pad 10: /LED_K85 -> /LED_K92
- J6 pad 11: /LED_A86 -> /LED_A91
- J6 pad 12: /LED_K86 -> /LED_K91
- J6 pad 13: /LED_A87 -> /LED_A90
- J6 pad 14: /LED_K87 -> /LED_K90
- J6 pad 15: /LED_A88 -> /LED_A89
- J6 pad 16: /LED_K88 -> /LED_K89
- J6 pad 17: /LED_A89 -> /LED_A88
- J6 pad 18: /LED_K89 -> /LED_K88
- J6 pad 2: /LED_K81 -> /LED_K96
- J6 pad 21: /LED_A90 -> /LED_A87
- J6 pad 22: /LED_K90 -> /LED_K87
- J6 pad 23: /LED_A91 -> /LED_A86
- J6 pad 24: /LED_K91 -> /LED_K86
- J6 pad 25: /LED_A92 -> /LED_A85
- J6 pad 26: /LED_K92 -> /LED_K85
- J6 pad 27: /LED_A93 -> /LED_A84
- J6 pad 28: /LED_K93 -> /LED_K84
- J6 pad 29: /LED_A94 -> /LED_A83
- J6 pad 3: /LED_A82 -> /LED_A95
- J6 pad 30: /LED_K94 -> /LED_K83
- J6 pad 31: /LED_A95 -> /LED_A82
- J6 pad 32: /LED_K95 -> /LED_K82
- J6 pad 33: /LED_A96 -> /LED_A81
- J6 pad 34: /LED_K96 -> /LED_K81
- J6 pad 4: /LED_K82 -> /LED_K95
- J6 pad 5: /LED_A83 -> /LED_A94
- J6 pad 6: /LED_K83 -> /LED_K94
- J6 pad 7: /LED_A84 -> /LED_A93
- J6 pad 8: /LED_K84 -> /LED_K93
- J6 pad 9: /LED_A85 -> /LED_A92
- U101 pad 10: /DIM5 -> /DIM8
- U101 pad 11: /DIM6 -> /DIM7
- U101 pad 12: /DIM7 -> /DIM6
- U101 pad 13: /DIM8 -> /DIM5
- U101 pad 15: /DIM9 -> /DIM4
- U101 pad 16: /DIM10 -> /DIM3
- U101 pad 17: /DIM11 -> /DIM2
- U101 pad 18: /DIM12 -> /DIM1
- U101 pad 19: /DIM13 -> /DIM16
- U101 pad 20: /DIM14 -> /DIM15
- U101 pad 21: /DIM15 -> /DIM14
- U101 pad 22: /DIM16 -> /DIM13
- U101 pad 6: /DIM1 -> /DIM12
- U101 pad 7: /DIM2 -> /DIM11
- U101 pad 8: /DIM3 -> /DIM10
- U101 pad 9: /DIM4 -> /DIM9
- U102 pad 10: /DIM21 -> /DIM20
- U102 pad 11: /DIM22 -> /DIM19
- U102 pad 12: /DIM23 -> /DIM18
- U102 pad 13: /DIM24 -> /DIM17
- U102 pad 15: /DIM25 -> /DIM32
- U102 pad 16: /DIM26 -> /DIM31
- U102 pad 17: /DIM27 -> /DIM30
- U102 pad 18: /DIM28 -> /DIM29
- U102 pad 19: /DIM29 -> /DIM28
- U102 pad 20: /DIM30 -> /DIM27
- U102 pad 21: /DIM31 -> /DIM26
- U102 pad 22: /DIM32 -> /DIM25
- U102 pad 6: /DIM17 -> /DIM24
- U102 pad 7: /DIM18 -> /DIM23
- U102 pad 8: /DIM19 -> /DIM22
- U102 pad 9: /DIM20 -> /DIM21
- U103 pad 10: /DIM37 -> /DIM48
- U103 pad 11: /DIM38 -> /DIM47
- U103 pad 12: /DIM39 -> /DIM46
- U103 pad 13: /DIM40 -> /DIM45
- U103 pad 15: /DIM41 -> /DIM44
- U103 pad 16: /DIM42 -> /DIM43
- U103 pad 17: /DIM43 -> /DIM42
- U103 pad 18: /DIM44 -> /DIM41
- U103 pad 19: /DIM45 -> /DIM40
- U103 pad 20: /DIM46 -> /DIM39
- U103 pad 21: /DIM47 -> /DIM38
- U103 pad 22: /DIM48 -> /DIM37
- U103 pad 6: /DIM33 -> /DIM36
- U103 pad 7: /DIM34 -> /DIM35
- U103 pad 8: /DIM35 -> /DIM34
- U103 pad 9: /DIM36 -> /DIM33
- U104 pad 10: /DIM53 -> /DIM56
- U104 pad 11: /DIM54 -> /DIM55
- U104 pad 12: /DIM55 -> /DIM54
- U104 pad 13: /DIM56 -> /DIM53
- U104 pad 15: /DIM57 -> /DIM52
- U104 pad 16: /DIM58 -> /DIM51
- U104 pad 17: /DIM59 -> /DIM50
- U104 pad 18: /DIM60 -> /DIM49
- U104 pad 19: /DIM61 -> /DIM64
- U104 pad 20: /DIM62 -> /DIM63
- U104 pad 21: /DIM63 -> /DIM62
- U104 pad 22: /DIM64 -> /DIM61
- U104 pad 6: /DIM49 -> /DIM60
- U104 pad 7: /DIM50 -> /DIM59
- U104 pad 8: /DIM51 -> /DIM58
- U104 pad 9: /DIM52 -> /DIM57
- U105 pad 10: /DIM69 -> /DIM68
- U105 pad 11: /DIM70 -> /DIM67
- U105 pad 12: /DIM71 -> /DIM66
- U105 pad 13: /DIM72 -> /DIM65
- U105 pad 15: /DIM73 -> /DIM80
- U105 pad 16: /DIM74 -> /DIM79
- U105 pad 17: /DIM75 -> /DIM78
- U105 pad 18: /DIM76 -> /DIM77
- U105 pad 19: /DIM77 -> /DIM76
- U105 pad 20: /DIM78 -> /DIM75
- U105 pad 21: /DIM79 -> /DIM74
- U105 pad 22: /DIM80 -> /DIM73
- U105 pad 6: /DIM65 -> /DIM72
- U105 pad 7: /DIM66 -> /DIM71
- U105 pad 8: /DIM67 -> /DIM70
- U105 pad 9: /DIM68 -> /DIM69
- U106 pad 10: /DIM85 -> /DIM96
- U106 pad 11: /DIM86 -> /DIM95
- U106 pad 12: /DIM87 -> /DIM94
- U106 pad 13: /DIM88 -> /DIM93
- U106 pad 15: /DIM89 -> /DIM92
- U106 pad 16: /DIM90 -> /DIM91
- U106 pad 17: /DIM91 -> /DIM90
- U106 pad 18: /DIM92 -> /DIM89
- U106 pad 19: /DIM93 -> /DIM88
- U106 pad 20: /DIM94 -> /DIM87
- U106 pad 21: /DIM95 -> /DIM86
- U106 pad 22: /DIM96 -> /DIM85
- U106 pad 6: /DIM81 -> /DIM84
- U106 pad 7: /DIM82 -> /DIM83
- U106 pad 8: /DIM83 -> /DIM82
- U106 pad 9: /DIM84 -> /DIM81
Other:
- board size 218 x 137.7 mm -> 3 x 3 mm

Commit message: LED board support parts copied to control-board topology (15mm border kept)
J1/J4 vertical on left edge, J2/J3 top, J5/J6 bottom, mux stack +
J9 on right strip; pin_maps v6 (CONN_MAP re-optimized, NTC_MAP
re-derived for right-strip muxes); schematics regenerated, netlists
verified, pads re-netted, zones refilled. New scripts:
layout_led_support.py, apply_netlist.py.

Co-Authored-By: Claude Fable 5 <noreply@anthropic.com>
Claude-Session: https://claude.ai/code/session_017oD54uh7Tvu54u9NPQNcZB
Connections:
- J1 pad 11: /LED_A13 -> /LED_A6
- J1 pad 12: /LED_K13 -> /LED_K6
- J1 pad 13: /LED_A6 -> /LED_A7
- J1 pad 14: /LED_K6 -> /LED_K7
- J1 pad 15: /LED_A7 -> /LED_A8
- J1 pad 16: /LED_K7 -> /LED_K8
- J1 pad 17: /LED_A14 -> /LED_A9
- J1 pad 18: /LED_K14 -> /LED_K9
- J1 pad 21: /LED_A8 -> /LED_A10
- J1 pad 22: /LED_K8 -> /LED_K10
- J1 pad 23: /LED_A15 -> /LED_A11
- J1 pad 24: /LED_K15 -> /LED_K11
- J1 pad 25: /LED_A9 -> /LED_A12
- J1 pad 26: /LED_K9 -> /LED_K12
- J1 pad 27: /LED_A10 -> /LED_A13
- J1 pad 28: /LED_K10 -> /LED_K13
- J1 pad 29: /LED_A16 -> /LED_A14
- J1 pad 30: /LED_K16 -> /LED_K14
- J1 pad 31: /LED_A11 -> /LED_A15
- J1 pad 32: /LED_K11 -> /LED_K15
- J1 pad 33: /LED_A12 -> /LED_A16
- J1 pad 34: /LED_K12 -> /LED_K16
- J4 pad 11: /LED_A61 -> /LED_A54
- J4 pad 12: /LED_K61 -> /LED_K54
- J4 pad 13: /LED_A54 -> /LED_A55
- J4 pad 14: /LED_K54 -> /LED_K55
- J4 pad 15: /LED_A55 -> /LED_A56
- J4 pad 16: /LED_K55 -> /LED_K56
- J4 pad 17: /LED_A62 -> /LED_A57
- J4 pad 18: /LED_K62 -> /LED_K57
- J4 pad 21: /LED_A56 -> /LED_A58
- J4 pad 22: /LED_K56 -> /LED_K58
- J4 pad 23: /LED_A63 -> /LED_A59
- J4 pad 24: /LED_K63 -> /LED_K59
- J4 pad 25: /LED_A57 -> /LED_A60
- J4 pad 26: /LED_K57 -> /LED_K60
- J4 pad 27: /LED_A58 -> /LED_A61
- J4 pad 28: /LED_K58 -> /LED_K61
- J4 pad 29: /LED_A64 -> /LED_A62
- J4 pad 30: /LED_K64 -> /LED_K62
- J4 pad 31: /LED_A59 -> /LED_A63
- J4 pad 32: /LED_K59 -> /LED_K63
- J4 pad 33: /LED_A60 -> /LED_A64
- J4 pad 34: /LED_K60 -> /LED_K64
Changed lines of the file:
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@@
 			(layers "*.Cu" "*.Mask")
 			(remove_unused_layers no)
-			(net "/LED_A61")
+			(net "/LED_A54")
 		)
 		(pad "12" thru_hole circle
@@
 			(layers "*.Cu" "*.Mask")
 			(remove_unused_layers no)
-			(net "/LED_K61")
+			(net "/LED_K54")
 		)
 		(pad "13" thru_hole circle
@@
 			(layers "*.Cu" "*.Mask")
 			(remove_unused_layers no)
-			(net "/LED_A54")
+			(net "/LED_A55")
 		)
 		(pad "14" thru_hole circle
@@
 			(layers "*.Cu" "*.Mask")
 			(remove_unused_layers no)
-			(net "/LED_K54")
+			(net "/LED_K55")
 		)
 		(pad "15" thru_hole circle
@@
 			(layers "*.Cu" "*.Mask")
 			(remove_unused_layers no)
-			(net "/LED_A55")
+			(net "/LED_A56")
 		)
 		(pad "16" thru_hole circle
@@
 			(layers "*.Cu" "*.Mask")
 			(remove_unused_layers no)
-			(net "/LED_K55")
+			(net "/LED_K56")
 		)
 		(pad "17" thru_hole circle
@@
 			(layers "*.Cu" "*.Mask")
 			(remove_unused_layers no)
-			(net "/LED_A62")
+			(net "/LED_A57")
 		)
 		(pad "18" thru_hole circle
@@
 			(layers "*.Cu" "*.Mask")
 			(remove_unused_layers no)
-			(net "/LED_K62")
+			(net "/LED_K57")
 		)
 		(pad "19" thru_hole circle
@@
 			(layers "*.Cu" "*.Mask")
 			(remove_unused_layers no)
-			(net "/LED_A56")
+			(net "/LED_A58")
 		)
 		(pad "22" thru_hole circle
@@
 			(layers "*.Cu" "*.Mask")
 			(remove_unused_layers no)
-			(net "/LED_K56")
+			(net "/LED_K58")
 		)
 		(pad "23" thru_hole circle
@@
 			(layers "*.Cu" "*.Mask")
 			(remove_unused_layers no)
-			(net "/LED_A63")
+			(net "/LED_A59")
 		)
 		(pad "24" thru_hole circle
@@
 			(layers "*.Cu" "*.Mask")
 			(remove_unused_layers no)
-			(net "/LED_K63")
+			(net "/LED_K59")
 		)
 		(pad "25" thru_hole circle
@@
 			(layers "*.Cu" "*.Mask")
 			(remove_unused_layers no)
-			(net "/LED_A57")
+			(net "/LED_A60")
 		)
 		(pad "26" thru_hole circle
@@
 			(layers "*.Cu" "*.Mask")
 			(remove_unused_layers no)
-			(net "/LED_K57")
+			(net "/LED_K60")
 		)
 		(pad "27" thru_hole circle
@@
 			(layers "*.Cu" "*.Mask")
 			(remove_unused_layers no)
-			(net "/LED_A58")
+			(net "/LED_A61")
 		)
 		(pad "28" thru_hole circle
@@
 			(layers "*.Cu" "*.Mask")
 			(remove_unused_layers no)
-			(net "/LED_K58")
+			(net "/LED_K61")
 		)
 		(pad "29" thru_hole circle
@@
 			(layers "*.Cu" "*.Mask")
 			(remove_unused_layers no)
-			(net "/LED_A64")
+			(net "/LED_A62")
 		)
 		(pad "30" thru_hole circle
@@
 			(layers "*.Cu" "*.Mask")
 			(remove_unused_layers no)
-			(net "/LED_K64")
+			(net "/LED_K62")
 		)
 		(pad "31" thru_hole circle
@@
 			(layers "*.Cu" "*.Mask")
 			(remove_unused_layers no)
-			(net "/LED_A59")
+			(net "/LED_A63")
 		)
 		(pad "32" thru_hole circle
@@
 			(layers "*.Cu" "*.Mask")
 			(remove_unused_layers no)
-			(net "/LED_K59")
+			(net "/LED_K63")
 		)
 		(pad "33" thru_hole circle
@@
 			(layers "*.Cu" "*.Mask")
 			(remove_unused_layers no)
-			(net "/LED_A60")
+			(net "/LED_A64")
 		)
 		(pad "34" thru_hole circle
@@
 			(layers "*.Cu" "*.Mask")
 			(remove_unused_layers no)
-			(net "/LED_K60")
+			(net "/LED_K64")
 		)
 		(pad "35" thru_hole circle
@@
 			(layers "*.Cu" "*.Mask")
 			(remove_unused_layers no)
-			(net "/LED_A13")
+			(net "/LED_A6")
 		)
 		(pad "12" thru_hole circle
@@
 			(layers "*.Cu" "*.Mask")
 			(remove_unused_layers no)
-			(net "/LED_K13")
+			(net "/LED_K6")
 		)
 		(pad "13" thru_hole circle
@@
 			(layers "*.Cu" "*.Mask")
 			(remove_unused_layers no)
-			(net "/LED_A6")
+			(net "/LED_A7")
 		)
 		(pad "14" thru_hole circle
@@
 			(layers "*.Cu" "*.Mask")
 			(remove_unused_layers no)
-			(net "/LED_K6")
+			(net "/LED_K7")
 		)
 		(pad "15" thru_hole circle
@@
 			(layers "*.Cu" "*.Mask")
 			(remove_unused_layers no)
-			(net "/LED_A7")
+			(net "/LED_A8")
 		)
 		(pad "16" thru_hole circle
@@
 			(layers "*.Cu" "*.Mask")
 			(remove_unused_layers no)
-			(net "/LED_K7")
+			(net "/LED_K8")
 		)
 		(pad "17" thru_hole circle
@@
 			(layers "*.Cu" "*.Mask")
 			(remove_unused_layers no)
-			(net "/LED_A14")
+			(net "/LED_A9")
 		)
 		(pad "18" thru_hole circle
@@
 			(layers "*.Cu" "*.Mask")
 			(remove_unused_layers no)
-			(net "/LED_K14")
+			(net "/LED_K9")
 		)
 		(pad "19" thru_hole circle
@@
 			(layers "*.Cu" "*.Mask")
 			(remove_unused_layers no)
-			(net "/LED_A8")
+			(net "/LED_A10")
 		)
 		(pad "22" thru_hole circle
@@
 			(layers "*.Cu" "*.Mask")
 			(remove_unused_layers no)
-			(net "/LED_K8")
+			(net "/LED_K10")
 		)
 		(pad "23" thru_hole circle
@@
 			(layers "*.Cu" "*.Mask")
 			(remove_unused_layers no)
-			(net "/LED_A15")
+			(net "/LED_A11")
 		)
 		(pad "24" thru_hole circle
@@
 			(layers "*.Cu" "*.Mask")
 			(remove_unused_layers no)
-			(net "/LED_K15")
+			(net "/LED_K11")
 		)
 		(pad "25" thru_hole circle
@@
 			(layers "*.Cu" "*.Mask")
 			(remove_unused_layers no)
-			(net "/LED_A9")
+			(net "/LED_A12")
 		)
 		(pad "26" thru_hole circle
@@
 			(layers "*.Cu" "*.Mask")
 			(remove_unused_layers no)
-			(net "/LED_K9")
+			(net "/LED_K12")
 		)
 		(pad "27" thru_hole circle
@@
 			(layers "*.Cu" "*.Mask")
 			(remove_unused_layers no)
-			(net "/LED_A10")
+			(net "/LED_A13")
 		)
 		(pad "28" thru_hole circle
@@
 			(layers "*.Cu" "*.Mask")
 			(remove_unused_layers no)
-			(net "/LED_K10")
+			(net "/LED_K13")
 		)
 		(pad "29" thru_hole circle
@@
 			(layers "*.Cu" "*.Mask")
 			(remove_unused_layers no)
-			(net "/LED_A16")
+			(net "/LED_A14")
 		)
 		(pad "30" thru_hole circle
@@
 			(layers "*.Cu" "*.Mask")
 			(remove_unused_layers no)
-			(net "/LED_K16")
+			(net "/LED_K14")
 		)
 		(pad "31" thru_hole circle
@@
 			(layers "*.Cu" "*.Mask")
 			(remove_unused_layers no)
-			(net "/LED_A11")
+			(net "/LED_A15")
 		)
 		(pad "32" thru_hole circle
@@
 			(layers "*.Cu" "*.Mask")
 			(remove_unused_layers no)
-			(net "/LED_K11")
+			(net "/LED_K15")
 		)
 		(pad "33" thru_hole circle
@@
 			(layers "*.Cu" "*.Mask")
 			(remove_unused_layers no)
-			(net "/LED_A12")
+			(net "/LED_A16")
 		)
 		(pad "34" thru_hole circle
@@
 			(layers "*.Cu" "*.Mask")
 			(remove_unused_layers no)
-			(net "/LED_K12")
+			(net "/LED_K16")
 		)
 		(pad "35" thru_hole circle
