File: control-board/control-board.kicad_sch (KiCad schematic)
At the start: 65 parts, among them J1 LED ch 1-16, J10 ESP32 left (3V3 row), J11 ESP32 right (GND row), J12 24V IN, J2 LED ch 17-32, J3 LED ch 33-48, J4 LED ch 49-64, J5 LED ch 65-80, J6 LED ch 81-96, J7 24V IN (5.5/2.5), J8 FAN 24V, J9 logic/analog, Q1 AO3400A, SW1 MODE, SW2 UP, SW3 DOWN, U101 PCA9685PW (0x40), U102 PCA9685PW (0x41), U103 PCA9685PW (0x42), U104 PCA9685PW (0x43), U105 PCA9685PW (0x44), U106 PCA9685PW (0x45), U110 XL1509-5.0E1, U111 ADS1115IDGS (DNP)

Commit message: Decouple driver<->well mapping to slash ribbon crossings (461 -> 126/130)
Key insight (user): the driver serving a well need not share its index.
A ribbon SLOT (connector + IDE-safe pin-pair) is now the logical channel;
wells and drivers are assigned to slots INDEPENDENTLY, each board optimized
on its own geometry, cable wires slot-for-slot.

optimize_decoupled.py: per board, balanced min-distance grouping (0 crossings
BETWEEN ribbons) + angle order + 2-opt on the true anode/cathode-pad
ratsnest. Real crossings: LED 461->126, control ->130 (short local A/K
wires only; the board-spanning tangle is gone).

design_data.py: nets keyed by logical channel via slot2ch(); wells indexed
by grid (LED/TH/R{w}, NTC_MAP[w]), drivers by placement (U/R/L/D/C{d},
DIM{d}, PCA_MAP[d]). gen_schematics_hier instance labels remapped.
CONNECTIONS.md gains the well<->channel<->driver<->PWM firmware map.
pin_maps v10. New durable tool apply_netlist.py used for PCB re-net.
Netlists ALL MATCH both boards; cross-board ribbon consistency OK (192).

Co-Authored-By: Claude Fable 5 <noreply@anthropic.com>
Claude-Session: https://claude.ai/code/session_017oD54uh7Tvu54u9NPQNcZB
Parts:
- J1: value LED ch 1-16 -> LED ribbon 1 (16 ch)
- J2: value LED ch 17-32 -> LED ribbon 2 (16 ch)
- J3: value LED ch 33-48 -> LED ribbon 3 (16 ch)
- J4: value LED ch 49-64 -> LED ribbon 4 (16 ch)
- J5: value LED ch 65-80 -> LED ribbon 5 (16 ch)
- J6: value LED ch 81-96 -> LED ribbon 6 (16 ch)
- TP11: value LED_A1 -> LED_A33
- TP12: value LED_K1 -> LED_K33
Connections:
- net DIM1: now also U101.9 (LED3); no longer U101.18 (LED11)
- net DIM10: now also U105.8 (LED2); no longer U101.8 (LED2)
- net DIM11: now also U105.7 (LED1); no longer U101.7 (LED1)
- net DIM12: now also U105.6 (LED0); no longer U101.6 (LED0)
- net DIM13: now also U101.13 (LED7); no longer U101.22 (LED15)
- net DIM14: now also U101.12 (LED6); no longer U101.21 (LED14)
- net DIM15: now also U101.11 (LED5); no longer U101.20 (LED13)
- net DIM16: now also U101.10 (LED4); no longer U101.19 (LED12)
- net DIM17: now also U104.15 (LED8); no longer U102.13 (LED7)
- net DIM18: now also U104.13 (LED7); no longer U102.12 (LED6)
- net DIM19: now also U104.12 (LED6); no longer U102.11 (LED5)
- net DIM2: now also U101.8 (LED2); no longer U101.17 (LED10)
- net DIM20: now also U104.11 (LED5); no longer U102.10 (LED4)
- net DIM21: now also U105.12 (LED6); no longer U102.9 (LED3)
- net DIM22: now also U105.11 (LED5); no longer U102.8 (LED2)
- net DIM23: now also U105.10 (LED4); no longer U102.7 (LED1)
- net DIM24: now also U105.9 (LED3); no longer U102.6 (LED0)
- net DIM25: now also U101.18 (LED11); no longer U102.22 (LED15)
- net DIM26: now also U101.17 (LED10); no longer U102.21 (LED14)
- net DIM27: now also U101.16 (LED9); no longer U102.20 (LED13)
- net DIM28: now also U101.15 (LED8); no longer U102.19 (LED12)
- net DIM29: now also U104.19 (LED12); no longer U102.18 (LED11)
- net DIM3: now also U101.7 (LED1); no longer U101.16 (LED9)
- net DIM30: now also U104.18 (LED11); no longer U102.17 (LED10)
- net DIM31: now also U104.17 (LED10); no longer U102.16 (LED9)
- net DIM32: now also U104.16 (LED9); no longer U102.15 (LED8)
- net DIM33: now also U105.17 (LED10); no longer U103.9 (LED3)
- net DIM34: now also U105.16 (LED9); no longer U103.8 (LED2)
- net DIM35: now also U105.15 (LED8); no longer U103.7 (LED1)
- net DIM36: now also U105.13 (LED7); no longer U103.6 (LED0)
- net DIM37: now also U101.22 (LED15); no longer U103.22 (LED15)
- net DIM38: now also U101.21 (LED14); no longer U103.21 (LED14)
- net DIM39: now also U101.20 (LED13); no longer U103.20 (LED13)
- net DIM4: now also U101.6 (LED0); no longer U101.15 (LED8)
- net DIM40: now also U101.19 (LED12); no longer U103.19 (LED12)
- net DIM41: now also U104.22 (LED15); no longer U103.18 (LED11)
- net DIM42: now also U104.21 (LED14); no longer U103.17 (LED10)
- net DIM43: now also U104.20 (LED13); no longer U103.16 (LED9)
- net DIM44: now also U105.22 (LED15); no longer U103.15 (LED8)
- net DIM45: now also U105.21 (LED14); no longer U103.13 (LED7)
- net DIM46: now also U105.20 (LED13); no longer U103.12 (LED6)
- net DIM47: now also U105.19 (LED12); no longer U103.11 (LED5)
- net DIM48: now also U105.18 (LED11); no longer U103.10 (LED4)
- net DIM49: now also U102.9 (LED3); no longer U104.18 (LED11)
- net DIM5: now also U104.10 (LED4); no longer U101.13 (LED7)
- net DIM50: now also U102.8 (LED2); no longer U104.17 (LED10)
- net DIM51: now also U102.7 (LED1); no longer U104.16 (LED9)
- net DIM52: now also U102.6 (LED0); no longer U104.15 (LED8)
- net DIM53: now also U103.8 (LED2); no longer U104.13 (LED7)
- net DIM54: now also U103.7 (LED1); no longer U104.12 (LED6)
- net DIM55: now also U103.6 (LED0); no longer U104.11 (LED5)
- net DIM56: now also U106.10 (LED4); no longer U104.10 (LED4)
- net DIM57: now also U106.9 (LED3); no longer U104.9 (LED3)
- net DIM58: now also U106.8 (LED2); no longer U104.8 (LED2)
- net DIM59: now also U106.7 (LED1); no longer U104.7 (LED1)
- net DIM6: now also U104.9 (LED3); no longer U101.12 (LED6)
- net DIM60: now also U106.6 (LED0); no longer U104.6 (LED0)
- net DIM61: now also U102.13 (LED7); no longer U104.22 (LED15)
- net DIM62: now also U102.12 (LED6); no longer U104.21 (LED14)
- net DIM63: now also U102.11 (LED5); no longer U104.20 (LED13)
- net DIM64: now also U102.10 (LED4); no longer U104.19 (LED12)
- net DIM65: now also U103.12 (LED6); no longer U105.13 (LED7)
- net DIM66: now also U103.11 (LED5); no longer U105.12 (LED6)
- net DIM67: now also U103.10 (LED4); no longer U105.11 (LED5)
- net DIM68: now also U103.9 (LED3); no longer U105.10 (LED4)
- net DIM69: now also U106.15 (LED8); no longer U105.9 (LED3)
- net DIM7: now also U104.8 (LED2); no longer U101.11 (LED5)
- net DIM70: now also U106.13 (LED7); no longer U105.8 (LED2)
- net DIM71: now also U106.12 (LED6); no longer U105.7 (LED1)
- net DIM72: now also U106.11 (LED5); no longer U105.6 (LED0)
- net DIM73: now also U102.18 (LED11); no longer U105.22 (LED15)
- net DIM74: now also U102.17 (LED10); no longer U105.21 (LED14)
- net DIM75: now also U102.16 (LED9); no longer U105.20 (LED13)
- net DIM76: now also U102.15 (LED8); no longer U105.19 (LED12)
- net DIM77: now also U103.17 (LED10); no longer U105.18 (LED11)
- net DIM78: now also U103.16 (LED9); no longer U105.17 (LED10)
- net DIM79: now also U103.15 (LED8); no longer U105.16 (LED9)
- net DIM8: now also U104.7 (LED1); no longer U101.10 (LED4)
- net DIM80: now also U103.13 (LED7); no longer U105.15 (LED8)
- net DIM81: now also U106.19 (LED12); no longer U106.9 (LED3)
- net DIM82: now also U106.18 (LED11); no longer U106.8 (LED2)
- net DIM83: now also U106.17 (LED10); no longer U106.7 (LED1)
- net DIM84: now also U106.16 (LED9); no longer U106.6 (LED0)
- net DIM85: now also U102.22 (LED15); no longer U106.22 (LED15)
- net DIM86: now also U102.21 (LED14); no longer U106.21 (LED14)
- net DIM87: now also U102.20 (LED13); no longer U106.20 (LED13)
- net DIM88: now also U102.19 (LED12); no longer U106.19 (LED12)
- net DIM89: now also U103.22 (LED15); no longer U106.18 (LED11)
- net DIM9: now also U104.6 (LED0); no longer U101.9 (LED3)
- net DIM90: now also U103.21 (LED14); no longer U106.17 (LED10)
- net DIM91: now also U103.20 (LED13); no longer U106.16 (LED9)
- net DIM92: now also U103.19 (LED12); no longer U106.15 (LED8)
- net DIM93: now also U103.18 (LED11); no longer U106.13 (LED7)
- net DIM94: now also U106.22 (LED15); no longer U106.12 (LED6)
- net DIM95: now also U106.21 (LED14); no longer U106.11 (LED5)
- net DIM96: now also U106.20 (LED13); no longer U106.10 (LED4)
- net LED_A1: now also J1.1 (Pin_1); no longer J1.33 (Pin_33), TP11.1
- net LED_A10: now also J1.21 (Pin_21); no longer J1.13 (Pin_13)
- net LED_A11: now also J1.23 (Pin_23); no longer J1.11 (Pin_11)
- net LED_A12: now also J1.25 (Pin_25); no longer J1.9 (Pin_9)
- net LED_A13: now also J1.27 (Pin_27); no longer J1.7 (Pin_7)
- net LED_A14: now also J1.29 (Pin_29); no longer J1.5 (Pin_5)
- net LED_A15: now also J1.31 (Pin_31); no longer J1.3 (Pin_3)
- net LED_A16: now also J1.33 (Pin_33); no longer J1.1 (Pin_1)
- net LED_A17: now also J2.1 (Pin_1); no longer J2.9 (Pin_9)
- net LED_A18: now also J2.3 (Pin_3); no longer J2.13 (Pin_13)
- net LED_A19: now also J2.5 (Pin_5); no longer J2.17 (Pin_17)
- net LED_A2: now also J1.3 (Pin_3); no longer J1.31 (Pin_31)
- net LED_A20: now also J2.7 (Pin_7); no longer J2.23 (Pin_23)
- net LED_A21: now also J2.9 (Pin_9); no longer J2.27 (Pin_27)
- net LED_A22: now also J2.11 (Pin_11); no longer J2.29 (Pin_29)
- net LED_A23: now also J2.13 (Pin_13); no longer J2.31 (Pin_31)
- net LED_A24: now also J2.15 (Pin_15); no longer J2.33 (Pin_33)
- net LED_A25: now also J2.17 (Pin_17); no longer J2.1 (Pin_1)
- net LED_A26: now also J2.21 (Pin_21); no longer J2.3 (Pin_3)
- net LED_A27: now also J2.23 (Pin_23); no longer J2.5 (Pin_5)
- net LED_A28: now also J2.25 (Pin_25); no longer J2.7 (Pin_7)
- net LED_A29: now also J2.27 (Pin_27); no longer J2.11 (Pin_11)
- net LED_A3: now also J1.5 (Pin_5); no longer J1.29 (Pin_29)
- net LED_A30: now also J2.29 (Pin_29); no longer J2.15 (Pin_15)
- net LED_A31: now also J2.31 (Pin_31); no longer J2.21 (Pin_21)
- net LED_A32: now also J2.33 (Pin_33); no longer J2.25 (Pin_25)
- net LED_A33: now also J3.1 (Pin_1), TP11.1; no longer J3.17 (Pin_17)
- net LED_A34: now also J3.3 (Pin_3); no longer J3.23 (Pin_23)
- net LED_A35: now also J3.5 (Pin_5); no longer J3.27 (Pin_27)
- net LED_A36: now also J3.7 (Pin_7); no longer J3.31 (Pin_31)
- net LED_A37: now also J3.9 (Pin_9); no longer J3.1 (Pin_1)
- net LED_A38: now also J3.11 (Pin_11); no longer J3.3 (Pin_3)
- net LED_A39: now also J3.13 (Pin_13); no longer J3.5 (Pin_5)
- net LED_A4: now also J1.7 (Pin_7); no longer J1.27 (Pin_27)
- net LED_A40: now also J3.15 (Pin_15); no longer J3.7 (Pin_7)
- net LED_A41: now also J3.17 (Pin_17); no longer J3.9 (Pin_9)
- net LED_A42: now also J3.21 (Pin_21); no longer J3.11 (Pin_11)
- net LED_A43: now also J3.23 (Pin_23); no longer J3.13 (Pin_13)
- net LED_A44: now also J3.25 (Pin_25); no longer J3.15 (Pin_15)
- net LED_A45: now also J3.27 (Pin_27); no longer J3.21 (Pin_21)
- net LED_A46: now also J3.29 (Pin_29); no longer J3.25 (Pin_25)
- net LED_A47: now also J3.31 (Pin_31); no longer J3.29 (Pin_29)
- net LED_A49: now also J4.1 (Pin_1); no longer J4.33 (Pin_33)
- net LED_A5: now also J1.9 (Pin_9); no longer J1.25 (Pin_25)
- net LED_A50: now also J4.3 (Pin_3); no longer J4.31 (Pin_31)
- net LED_A51: now also J4.5 (Pin_5); no longer J4.29 (Pin_29)
- net LED_A52: now also J4.7 (Pin_7); no longer J4.27 (Pin_27)
- net LED_A53: now also J4.9 (Pin_9); no longer J4.25 (Pin_25)
- net LED_A54: now also J4.11 (Pin_11); no longer J4.23 (Pin_23)
- net LED_A55: now also J4.13 (Pin_13); no longer J4.21 (Pin_21)
- net LED_A56: now also J4.15 (Pin_15); no longer J4.17 (Pin_17)
- net LED_A57: now also J4.17 (Pin_17); no longer J4.15 (Pin_15)
- net LED_A58: now also J4.21 (Pin_21); no longer J4.13 (Pin_13)
- net LED_A59: now also J4.23 (Pin_23); no longer J4.11 (Pin_11)
- net LED_A6: now also J1.11 (Pin_11); no longer J1.23 (Pin_23)
- net LED_A60: now also J4.25 (Pin_25); no longer J4.9 (Pin_9)
- net LED_A61: now also J4.27 (Pin_27); no longer J4.7 (Pin_7)
- net LED_A62: now also J4.29 (Pin_29); no longer J4.5 (Pin_5)
- net LED_A63: now also J4.31 (Pin_31); no longer J4.3 (Pin_3)
- net LED_A64: now also J4.33 (Pin_33); no longer J4.1 (Pin_1)
- net LED_A65: now also J5.1 (Pin_1); no longer J5.9 (Pin_9)
- net LED_A66: now also J5.3 (Pin_3); no longer J5.13 (Pin_13)
- net LED_A67: now also J5.5 (Pin_5); no longer J5.17 (Pin_17)
- net LED_A68: now also J5.7 (Pin_7); no longer J5.23 (Pin_23)
- net LED_A69: now also J5.9 (Pin_9); no longer J5.27 (Pin_27)
- net LED_A7: now also J1.13 (Pin_13); no longer J1.21 (Pin_21)
- net LED_A70: now also J5.11 (Pin_11); no longer J5.29 (Pin_29)
- net LED_A71: now also J5.13 (Pin_13); no longer J5.31 (Pin_31)
- net LED_A72: now also J5.15 (Pin_15); no longer J5.33 (Pin_33)
- net LED_A73: now also J5.17 (Pin_17); no longer J5.1 (Pin_1)
- net LED_A74: now also J5.21 (Pin_21); no longer J5.3 (Pin_3)
- net LED_A75: now also J5.23 (Pin_23); no longer J5.5 (Pin_5)
- net LED_A76: now also J5.25 (Pin_25); no longer J5.7 (Pin_7)
- net LED_A77: now also J5.27 (Pin_27); no longer J5.11 (Pin_11)
- net LED_A78: now also J5.29 (Pin_29); no longer J5.15 (Pin_15)
- net LED_A79: now also J5.31 (Pin_31); no longer J5.21 (Pin_21)
- net LED_A8: now also J1.15 (Pin_15); no longer J1.17 (Pin_17)
- net LED_A80: now also J5.33 (Pin_33); no longer J5.25 (Pin_25)
- net LED_A81: now also J6.1 (Pin_1); no longer J6.17 (Pin_17)
- net LED_A82: now also J6.3 (Pin_3); no longer J6.23 (Pin_23)
- net LED_A83: now also J6.5 (Pin_5); no longer J6.27 (Pin_27)
- net LED_A84: now also J6.7 (Pin_7); no longer J6.31 (Pin_31)
- net LED_A85: now also J6.9 (Pin_9); no longer J6.1 (Pin_1)
- net LED_A86: now also J6.11 (Pin_11); no longer J6.3 (Pin_3)
- net LED_A87: now also J6.13 (Pin_13); no longer J6.5 (Pin_5)
- net LED_A88: now also J6.15 (Pin_15); no longer J6.7 (Pin_7)
- net LED_A89: now also J6.17 (Pin_17); no longer J6.9 (Pin_9)
- net LED_A9: now also J1.17 (Pin_17); no longer J1.15 (Pin_15)
- net LED_A90: now also J6.21 (Pin_21); no longer J6.11 (Pin_11)
- net LED_A91: now also J6.23 (Pin_23); no longer J6.13 (Pin_13)
- net LED_A92: now also J6.25 (Pin_25); no longer J6.15 (Pin_15)
- net LED_A93: now also J6.27 (Pin_27); no longer J6.21 (Pin_21)
- net LED_A94: now also J6.29 (Pin_29); no longer J6.25 (Pin_25)
- net LED_A95: now also J6.31 (Pin_31); no longer J6.29 (Pin_29)
- net LED_K1: now also J1.2 (Pin_2); no longer J1.34 (Pin_34), TP12.1
- net LED_K10: now also J1.22 (Pin_22); no longer J1.14 (Pin_14)
- net LED_K11: now also J1.24 (Pin_24); no longer J1.12 (Pin_12)
- net LED_K12: now also J1.26 (Pin_26); no longer J1.10 (Pin_10)
- net LED_K13: now also J1.28 (Pin_28); no longer J1.8 (Pin_8)
- net LED_K14: now also J1.30 (Pin_30); no longer J1.6 (Pin_6)
- net LED_K15: now also J1.32 (Pin_32); no longer J1.4 (Pin_4)
- net LED_K16: now also J1.34 (Pin_34); no longer J1.2 (Pin_2)
- net LED_K17: now also J2.2 (Pin_2); no longer J2.10 (Pin_10)
- net LED_K18: now also J2.4 (Pin_4); no longer J2.14 (Pin_14)
- net LED_K19: now also J2.6 (Pin_6); no longer J2.18 (Pin_18)
- net LED_K2: now also J1.4 (Pin_4); no longer J1.32 (Pin_32)
- net LED_K20: now also J2.8 (Pin_8); no longer J2.24 (Pin_24)
- net LED_K21: now also J2.10 (Pin_10); no longer J2.28 (Pin_28)
- net LED_K22: now also J2.12 (Pin_12); no longer J2.30 (Pin_30)
- net LED_K23: now also J2.14 (Pin_14); no longer J2.32 (Pin_32)
- net LED_K24: now also J2.16 (Pin_16); no longer J2.34 (Pin_34)
- net LED_K25: now also J2.18 (Pin_18); no longer J2.2 (Pin_2)
- net LED_K26: now also J2.22 (Pin_22); no longer J2.4 (Pin_4)
- net LED_K27: now also J2.24 (Pin_24); no longer J2.6 (Pin_6)
- net LED_K28: now also J2.26 (Pin_26); no longer J2.8 (Pin_8)
- net LED_K29: now also J2.28 (Pin_28); no longer J2.12 (Pin_12)
- net LED_K3: now also J1.6 (Pin_6); no longer J1.30 (Pin_30)
- net LED_K30: now also J2.30 (Pin_30); no longer J2.16 (Pin_16)
- net LED_K31: now also J2.32 (Pin_32); no longer J2.22 (Pin_22)
- net LED_K32: now also J2.34 (Pin_34); no longer J2.26 (Pin_26)
- net LED_K33: now also J3.2 (Pin_2), TP12.1; no longer J3.18 (Pin_18)
- net LED_K34: now also J3.4 (Pin_4); no longer J3.24 (Pin_24)
- net LED_K35: now also J3.6 (Pin_6); no longer J3.28 (Pin_28)
- net LED_K36: now also J3.8 (Pin_8); no longer J3.32 (Pin_32)
- net LED_K37: now also J3.10 (Pin_10); no longer J3.2 (Pin_2)
- net LED_K38: now also J3.12 (Pin_12); no longer J3.4 (Pin_4)
- net LED_K39: now also J3.14 (Pin_14); no longer J3.6 (Pin_6)
- net LED_K4: now also J1.8 (Pin_8); no longer J1.28 (Pin_28)
- net LED_K40: now also J3.16 (Pin_16); no longer J3.8 (Pin_8)
- net LED_K41: now also J3.18 (Pin_18); no longer J3.10 (Pin_10)
- net LED_K42: now also J3.22 (Pin_22); no longer J3.12 (Pin_12)
- net LED_K43: now also J3.24 (Pin_24); no longer J3.14 (Pin_14)
- net LED_K44: now also J3.26 (Pin_26); no longer J3.16 (Pin_16)
- net LED_K45: now also J3.28 (Pin_28); no longer J3.22 (Pin_22)
- net LED_K46: now also J3.30 (Pin_30); no longer J3.26 (Pin_26)
- net LED_K47: now also J3.32 (Pin_32); no longer J3.30 (Pin_30)
- net LED_K49: now also J4.2 (Pin_2); no longer J4.34 (Pin_34)
- net LED_K5: now also J1.10 (Pin_10); no longer J1.26 (Pin_26)
- net LED_K50: now also J4.4 (Pin_4); no longer J4.32 (Pin_32)
- net LED_K51: now also J4.6 (Pin_6); no longer J4.30 (Pin_30)
- net LED_K52: now also J4.8 (Pin_8); no longer J4.28 (Pin_28)
- net LED_K53: now also J4.10 (Pin_10); no longer J4.26 (Pin_26)
- net LED_K54: now also J4.12 (Pin_12); no longer J4.24 (Pin_24)
- net LED_K55: now also J4.14 (Pin_14); no longer J4.22 (Pin_22)
- net LED_K56: now also J4.16 (Pin_16); no longer J4.18 (Pin_18)
- net LED_K57: now also J4.18 (Pin_18); no longer J4.16 (Pin_16)
- net LED_K58: now also J4.22 (Pin_22); no longer J4.14 (Pin_14)
- net LED_K59: now also J4.24 (Pin_24); no longer J4.12 (Pin_12)
- net LED_K6: now also J1.12 (Pin_12); no longer J1.24 (Pin_24)
- net LED_K60: now also J4.26 (Pin_26); no longer J4.10 (Pin_10)
- net LED_K61: now also J4.28 (Pin_28); no longer J4.8 (Pin_8)
- net LED_K62: now also J4.30 (Pin_30); no longer J4.6 (Pin_6)
- net LED_K63: now also J4.32 (Pin_32); no longer J4.4 (Pin_4)
- net LED_K64: now also J4.34 (Pin_34); no longer J4.2 (Pin_2)
- net LED_K65: now also J5.2 (Pin_2); no longer J5.10 (Pin_10)
- net LED_K66: now also J5.4 (Pin_4); no longer J5.14 (Pin_14)
- net LED_K67: now also J5.6 (Pin_6); no longer J5.18 (Pin_18)
- net LED_K68: now also J5.8 (Pin_8); no longer J5.24 (Pin_24)
- net LED_K69: now also J5.10 (Pin_10); no longer J5.28 (Pin_28)
- net LED_K7: now also J1.14 (Pin_14); no longer J1.22 (Pin_22)
- net LED_K70: now also J5.12 (Pin_12); no longer J5.30 (Pin_30)
- net LED_K71: now also J5.14 (Pin_14); no longer J5.32 (Pin_32)
- net LED_K72: now also J5.16 (Pin_16); no longer J5.34 (Pin_34)
- net LED_K73: now also J5.18 (Pin_18); no longer J5.2 (Pin_2)
- net LED_K74: now also J5.22 (Pin_22); no longer J5.4 (Pin_4)
- net LED_K75: now also J5.24 (Pin_24); no longer J5.6 (Pin_6)
- net LED_K76: now also J5.26 (Pin_26); no longer J5.8 (Pin_8)
- net LED_K77: now also J5.28 (Pin_28); no longer J5.12 (Pin_12)
- net LED_K78: now also J5.30 (Pin_30); no longer J5.16 (Pin_16)
- net LED_K79: now also J5.32 (Pin_32); no longer J5.22 (Pin_22)
- net LED_K8: now also J1.16 (Pin_16); no longer J1.18 (Pin_18)
- net LED_K80: now also J5.34 (Pin_34); no longer J5.26 (Pin_26)
- net LED_K81: now also J6.2 (Pin_2); no longer J6.18 (Pin_18)
- net LED_K82: now also J6.4 (Pin_4); no longer J6.24 (Pin_24)
- net LED_K83: now also J6.6 (Pin_6); no longer J6.28 (Pin_28)
- net LED_K84: now also J6.8 (Pin_8); no longer J6.32 (Pin_32)
- net LED_K85: now also J6.10 (Pin_10); no longer J6.2 (Pin_2)
- net LED_K86: now also J6.12 (Pin_12); no longer J6.4 (Pin_4)
- net LED_K87: now also J6.14 (Pin_14); no longer J6.6 (Pin_6)
- net LED_K88: now also J6.16 (Pin_16); no longer J6.8 (Pin_8)
- net LED_K89: now also J6.18 (Pin_18); no longer J6.10 (Pin_10)
- net LED_K9: now also J1.18 (Pin_18); no longer J1.16 (Pin_16)
- net LED_K90: now also J6.22 (Pin_22); no longer J6.12 (Pin_12)
- net LED_K91: now also J6.24 (Pin_24); no longer J6.14 (Pin_14)
- net LED_K92: now also J6.26 (Pin_26); no longer J6.16 (Pin_16)
- net LED_K93: now also J6.28 (Pin_28); no longer J6.22 (Pin_22)
- net LED_K94: now also J6.30 (Pin_30); no longer J6.26 (Pin_26)
- net LED_K95: now also J6.32 (Pin_32); no longer J6.30 (Pin_30)
Other:
- note added: "96 DRIVER CHANNELS - see channel.kicad_sch"
- note removed: "96 DRIVER CHANNELS (CH01..CH96) - see channel.kicad_sch"
